File: can.kicad_sch (KiCad schematic)
At the start: 17 parts, among them Q301 2N7002K, U301 TJA1051T-3, U302 MCP2510-x/SO, U303 MAX3485CSA, Y301 16MHz

Commit message: started routing
Parts:
- R7: renamed from R301; value 10k -> 1k
- R8: renamed from R302; value 10k -> 1k
- U5: renamed from U303; footprint (none) -> Package_SO:SOIC-8_3.9x4.9mm_P1.27mm
- renumbered C302 to C16, C303 to C17, C301 to C18, C304 to C19, D301 to D1, JP301 to JP1, JP302 to JP2, Q301 to Q1, R304 to R10, R305 to R11, R303 to R9, U301 to U3, U302 to U4, Y301 to Y2
Other:
- title: (none) -> [canbrd] CAN/RS485 IO board

Commit message: Done?
Parts:
- removed JP1: Pin5, Jumper:SolderJumper-3_P1.3mm_Bridged2Bar12_Pad1.0x1.5mm, symbol Jumper:Jumper_3_Bridged12
- removed JP2: Pin8, Jumper:SolderJumper-3_P1.3mm_Bridged2Bar12_Pad1.0x1.5mm, symbol Jumper:Jumper_3_Bridged12
- added C20: 100n, Capacitor_SMD:C_0603_1608Metric, symbol Device:C
- added D1, D2: TBU-CA, TBU-CA:DIOC650X400X100N, symbol TBU-CA065-200-WH:TBU-CA065-200-WH
- added JP1: Pin5H, Jumper:SolderJumper-2_P1.3mm_Bridged_Pad1.0x1.5mm, symbol Jumper:Jumper_2_Bridged
- added JP2: Pin8H, Jumper:SolderJumper-2_P1.3mm_Open_TrianglePad1.0x1.5mm, symbol Jumper:Jumper_2_Open
- added JP3: Pin5L, Jumper:SolderJumper-2_P1.3mm_Open_TrianglePad1.0x1.5mm, symbol Jumper:Jumper_2_Open
- added JP4: Pin8L, Jumper:SolderJumper-2_P1.3mm_Bridged_Pad1.0x1.5mm, symbol Jumper:Jumper_2_Bridged
- renumbered D1 to D3
Connections:
- net +3V3: now also C20.1
- net +5V: now also JP1.2 (B), JP2.1 (A)
- net CANH: now also D1.3; no longer D3.2 (K), U3.7 (CANH), U5.6 (A)
- net CANL: now also D2.3; no longer D3.1 (K), U3.6 (CANL), U5.7 (B)
- net GND: now also C20.2, JP3.1 (A), JP4.2 (B)
- net Pin5: now also JP1.1 (A), JP3.2 (B)
- net Pin8: now also JP2.2 (B), JP4.1 (A)
- new net: D2.1, D3.1 (K), U3.6 (CANL), U5.7 (B)
- new net: D1.1, D3.2 (K), U3.7 (CANH), U5.6 (A)
Other:
- moved on the sheet: C18, C19
