File: conn.kicad_sch (KiCad schematic)
At the start: 6 parts, among them J701 Out, J702 PwrOut, J703 RJ45_Shielded, J704 In, J705 RawIO, J706 RJ45_Shielded

Commit message: started routing
Parts:
- removed J701: Out, canbrd_conn:NR1212x1xxxxG, symbol Connector_Generic:Conn_02x06_Odd_Even
- removed J702: PwrOut, canbrd_conn:NR1212x1xxxxG, symbol Connector_Generic:Conn_02x06_Odd_Even
- removed J704: In, canbrd_conn:NR1212x1xxxxG, symbol Connector_Generic:Conn_02x06_Odd_Even
- removed J705: RawIO, canbrd_conn:NR1212x1xxxxG, symbol Connector_Generic:Conn_02x06_Odd_Even
- added J10: IO2, canbrd_conn:NH0810x0xxxxG, symbol Connector:Screw_Terminal_01x08
- added J11: I^{2}C, Connector_PinHeader_2.54mm:PinHeader_2x04_P2.54mm_Vertical_SMD, symbol Connector_Generic:Conn_02x04_Odd_Even
- added J12: PwrOut, canbrd_conn:NH0810x0xxxxG, symbol Connector:Screw_Terminal_01x08
- added J13: USB_C_Receptacle_USB2.0, Connector_USB:USB_C_Receptacle_GCT_USB4085, symbol Connector:USB_C_Receptacle_USB2.0
- added J14: IO1, canbrd_conn:NH0810x0xxxxG, symbol Connector:Screw_Terminal_01x08
- added J15: IO0, canbrd_conn:NH0810x0xxxxG, symbol Connector:Screw_Terminal_01x08
- added J4: GND, canbrd_conn:NH0210x0xxxxG, symbol Connector:Screw_Terminal_01x02
- added J5: Field24V, canbrd_conn:NH0210x0xxxxG, symbol Connector:Screw_Terminal_01x02
- added J8, J9: CAN, canbrd_conn:NH0210x0xxxxG, symbol Connector:Screw_Terminal_01x02
- renumbered J703 to J6, J706 to J7
Connections:
- net GND: now reaches J6.1
- net GND: now also J6.3, J6.5, J6.SH, J7.1, J7.3, J7.5, J7.SH, J11.1 (Pin_1), J11.8 (Pin_8), J12.1 (Pin_1), J12.2 (Pin_2), J4.1 (Pin_1), J4.2 (Pin_2)
- net Field24V: now reaches J6.2
- net Field24V: now also J6.4, J6.6, J7.2, J7.4, J7.6, J5.1 (Pin_1), J5.2 (Pin_2)
- net CANH: now reaches J6.7
- net CANH: now also J7.7, J8.2 (Pin_2), J9.2 (Pin_2)
- net CANL: now reaches J6.8
- net CANL: now also J7.8, J8.1 (Pin_1), J9.1 (Pin_1)
- new net: J13.A1 (GND), J13.A12 (GND), J13.B1 (GND), J13.B12 (GND)
- new net: J13.A4 (VBUS), J13.A9 (VBUS), J13.B4 (VBUS), J13.B9 (VBUS)
- new net +24V: J12.7 (Pin_7), J12.8 (Pin_8)
- new net +3V3: J11.2 (Pin_2), J11.7 (Pin_7), J12.3 (Pin_3), J12.4 (Pin_4)
- new net +5V: J12.5 (Pin_5), J12.6 (Pin_6)
- new net EXT.0: J11.6 (Pin_6)
- new net EXT.1: J11.4 (Pin_4)
- new net IO0.0: J15.1 (Pin_1)
- new net IO0.1: J15.2 (Pin_2)
- new net IO0.2: J15.3 (Pin_3)
- new net IO0.3: J15.4 (Pin_4)
- new net IO0.4: J15.5 (Pin_5)
- new net IO0.5: J15.6 (Pin_6)
- new net IO0.6: J15.7 (Pin_7)
- new net IO0.7: J15.8 (Pin_8)
- new net SCL: J11.5 (Pin_5)
- new net SDA: J11.3 (Pin_3)
Other:
- title: (none) -> [canbrd] CAN/RS485 IO board
- moved on the sheet: J6, J7

Commit message: Done?
Parts:
- removed J13: USB_C_Receptacle_USB2.0, Connector_USB:USB_C_Receptacle_GCT_USB4085, symbol Connector:USB_C_Receptacle_USB2.0
- added J13: USB_C_Receptacle, 10132328:10132328, symbol Connector:USB_C_Receptacle
- added R21, R22: 5.1k, Resistor_SMD:R_0603_1608Metric, symbol Device:R
- J6, J7: value RJ45_Shielded -> Amphenol RJHSE5380
- renumbered J12 to J10, J10 to J11, J11 to J12
Connections:
- net +3V3: no longer J12.2 (Pin_2), J12.7 (Pin_7)
- net CANH: now also J6.1, J7.1, J8.1 (Pin_1), J9.1 (Pin_1); no longer J6.7, J7.7, J8.2 (Pin_2), J9.2 (Pin_2)
- net CANL: now also J6.2, J7.2, J8.2 (Pin_2), J9.2 (Pin_2); no longer J6.8, J7.8, J8.1 (Pin_1), J9.1 (Pin_1)
- net Field24V: now also J6.8, J7.8; no longer J6.2, J6.4, J6.6, J7.2, J7.4, J7.6
- net GND: now also J12.2 (Pin_2), J12.7 (Pin_7), J6.6, J6.7, J7.6, J7.7, J13.A1 (GND), J13.A12 (GND), J13.B1 (GND), J13.B12 (GND), J13.S1 (SHIELD), R21.2, R22.2; no longer J6.1, J6.5, J7.1, J7.5
- net IO1.0: now reaches J14.1 (Pin_1)
- net IO1.1: now reaches J14.2 (Pin_2)
- net IO1.2: now reaches J14.3 (Pin_3)
- net IO1.3: now reaches J14.4 (Pin_4)
- net IO1.4: now reaches J14.5 (Pin_5)
- net IO1.5: now reaches J14.6 (Pin_6)
- net IO1.6: now reaches J14.7 (Pin_7)
- net IO1.7: now reaches J14.8 (Pin_8)
- net IO2.0: now reaches J11.1 (Pin_1)
- net IO2.1: now reaches J11.2 (Pin_2)
- net IO2.2: now reaches J11.3 (Pin_3)
- net IO2.3: now reaches J11.4 (Pin_4)
- net IO2.4: now reaches J11.5 (Pin_5)
- net IO2.5: now reaches J11.6 (Pin_6)
- net IO2.6: now reaches J11.7 (Pin_7)
- net IO2.7: now reaches J11.8 (Pin_8)
- new net: J13.A5 (CC1), R21.1
- new net: J13.B5 (CC2), R22.1
- new net USB+: J13.A6 (D+), J13.B6 (D+)
- new net USB-: J13.A7 (D-), J13.B7 (D-)
- new net VBUS: J13.A4 (VBUS), J13.A9 (VBUS), J13.B4 (VBUS), J13.B9 (VBUS)
- no-connect marks 0 -> 14
Other:
- moved on the sheet: J10, J8, J9
