File: hardware.kicad_pcb (KiCad board)
At the start: 2 copper layers, 100 x 100 mm, 95 parts, among them J1 PowerIn, J201 RP_DEBUG, J203 RJ45_LED_Shielded_x2, J7 PowerThru, J701 Out, J702 PwrOut, J703 RJ45_Shielded, J704 In, J705 RawIO, J706 RJ45_Shielded, Q301 2N7002K, Q401 2N7002K, Q601 Q_PMOS_GDS, SW101 SW_DIP_x08, SW201 BOOTSEL, SW202 RESET, SW401 SW_DIP_x08, SW402 User, U201 W25Q16JVSNIQ, U202 RP2040, U301 TJA1051T-3, U302 MCP2510-x/SO, Y201 12MHz, Y301 16MHz

Commit message: started routing
Parts:
- removed C201, C204: 1u, Capacitor_SMD:C_0603_1608Metric
- removed C202, C203, C205, C206, C207, C208, C209, C210, C211, C213, C214, C301, C304: 100n, Capacitor_SMD:C_0603_1608Metric
- removed C212: 2.2u, Capacitor_SMD:C_0603_1608Metric
- removed C215, C216, C302, C303: ???, Capacitor_SMD:C_0603_1608Metric
- removed C601, C604: 100n, Capacitor_SMD:C_0805_2012Metric
- removed C602, C603: 100u, Capacitor_THT:CP_Radial_D10.0mm_P5.00mm
- removed D301: NUP2105L, Package_TO_SOT_SMD:SOT-23
- removed D401: User, LED_SMD:LED_0805_2012Metric
- removed D402: Heartbeat, LED_SMD:LED_0805_2012Metric
- removed D601: 10V, Diode_SMD:D_SOD-123
- removed D602: 33V, Diode_SMD:D_SMB
- removed F601: 500mA, Littelfuse-154:Littelfuse-154
- removed H101, H102, H103, H104: MountingHole, MountingHole:MountingHole_3.2mm_M3
- removed J201: RP_DEBUG, Connector_PinHeader_1.27mm:PinHeader_2x05_P1.27mm_Vertical_SMD
- removed J203: RJ45_LED_Shielded_x2, Connector_RJ:RJ45_Amphenol_RJHSE538X-02
- removed J701: Out, canbrd_conn:NR1212x1xxxxG
- removed J702: PwrOut, canbrd_conn:NR1212x1xxxxG
- removed J703, J706: RJ45_Shielded, Connector_RJ:RJ45_Amphenol_RJHSE5380
- removed J704: In, canbrd_conn:NR1212x1xxxxG
- removed J705: RawIO, canbrd_conn:NR1212x1xxxxG
- removed JP301: Pin5, Jumper:SolderJumper-3_P1.3mm_Bridged2Bar12_Pad1.0x1.5mm
- removed JP302: Pin8, Jumper:SolderJumper-3_P1.3mm_Bridged2Bar12_Pad1.0x1.5mm
- removed L601: 3.3u, Inductor_SMD:L_1008_2520Metric
- removed LD101, LD401: LTD4708G, LTD-470:LED_LTD-4708G
- removed Q301, Q401: 2N7002K, Package_TO_SOT_SMD:SOT-23
- removed Q601: Q_PMOS_GDS, Package_TO_SOT_SMD:TO-252-2
- removed R201: 200, Resistor_SMD:R_0603_1608Metric
- removed R202, R203: 27, Resistor_SMD:R_0603_1608Metric
- removed R204, R301, R302, R304, R402, R404, R406, R408, R410, R412, R414, R416, R419, R601: 10k, Resistor_SMD:R_0603_1608Metric
- removed R205, R401, R403, R405, R407, R409, R411, R413, R415, R417, R418: 1k, Resistor_SMD:R_0603_1608Metric
- removed R206, R305: ???, Resistor_SMD:R_0603_1608Metric
- removed R303: 4k7, Resistor_SMD:R_0603_1608Metric
- removed RV601: 20V, Resistor_SMD:R_1206_3216Metric
- removed SW101, SW401: SW_DIP_x08, Button_Switch_SMD:SW_DIP_SPSTx08_Slide_Omron_A6H-8101_W6.15mm_P1.27mm
- removed SW201: BOOTSEL, PTS815-SJ:PTS815-SJ
- removed SW202: RESET, PTS815-SJ:PTS815-SJ
- removed SW402: User, PTS815-SJ:PTS815-SJ
- removed U201: W25Q16JVSNIQ, Package_SO:SOIC-8_3.9x4.9mm_P1.27mm
- removed U202: RP2040, Package_DFN_QFN:QFN-56-1EP_7x7mm_P0.4mm_EP5.6x5.6mm_ThermalVias
- removed U301: TJA1051T-3, Package_SO:SOIC-8_3.9x4.9mm_P1.27mm
- removed U302: MCP2510-x/SO, Package_SO:SOIC-18W_7.5x11.6mm_P1.27mm
- removed Y201: 12MHz, Crystal:Crystal_SMD_3225-4Pin_3.2x2.5mm
- removed Y301: 16MHz, Crystal:Crystal_SMD_3225-4Pin_3.2x2.5mm
- added C1: 1u, Capacitor_SMD:C_0603_1608Metric, F.Cu at (177.6, 113.2)
- added C10: 100n, Capacitor_SMD:C_0603_1608Metric, F.Cu at (173.4, 105.3)
- added C11: 1u, Capacitor_SMD:C_0603_1608Metric, F.Cu at (176.0, 117.0)
- added C12: 100n, Capacitor_SMD:C_0603_1608Metric, F.Cu at (174.5, 117.0)
- added C13: 100n, Capacitor_SMD:C_0603_1608Metric, F.Cu at (184.5, 99.8)
- added C14: ???, Capacitor_SMD:C_0603_1608Metric, F.Cu at (157.2, 105.8)
- added C15: ???, Capacitor_SMD:C_0603_1608Metric, F.Cu at (157.2, 111.5)
- added C16: ???, Capacitor_SMD:C_0603_1608Metric, F.Cu at (466.8, 129.0)
- added C17: ???, Capacitor_SMD:C_0603_1608Metric, F.Cu at (459.2, 137.4)
- added C18: 100n, Capacitor_SMD:C_0603_1608Metric, F.Cu at (466.8, 126.5)
- added C19: 100n, Capacitor_SMD:C_0603_1608Metric, F.Cu at (151.1, 81.1)
- added C2: 100n, Capacitor_SMD:C_0603_1608Metric, F.Cu at (177.6, 109.7)
- added C20: 1u, Capacitor_SMD:C_0603_1608Metric, F.Cu at (232.0, 132.7)
- added C21: 100n, Capacitor_SMD:C_0603_1608Metric, F.Cu at (233.5, 132.7)
- added C22: 1u, Capacitor_SMD:C_0603_1608Metric, F.Cu at (232.0, 135.8)
- added C23: 100n, Capacitor_SMD:C_0603_1608Metric, F.Cu at (233.5, 135.8)
- added C24: 100n, Capacitor_SMD:C_0603_1608Metric, F.Cu at (364.6, 59.0)
- added C25: 100n, Capacitor_SMD:C_0805_2012Metric, F.Cu at (190.0, 62.0)
- added C26: 47u, Capacitor_SMD:CP_Elec_8x6.5, F.Cu at (192.5, 71.0)
- added C27: 47u, Capacitor_SMD:CP_Elec_8x6.5, F.Cu at (192.5, 80.0)
- added C28: 100n, Capacitor_SMD:C_0805_2012Metric, F.Cu at (180.5, 75.5)
- added C3: 100n, Capacitor_SMD:C_0603_1608Metric, F.Cu at (161.5, 112.7)
- added C4: 1u, Capacitor_SMD:C_0603_1608Metric, F.Cu at (177.6, 114.7)
- added C5: 100n, Capacitor_SMD:C_0603_1608Metric, F.Cu at (177.6, 111.2)
- added C6: 100n, Capacitor_SMD:C_0603_1608Metric, F.Cu at (173.0, 117.0)
- added C7: 100n, Capacitor_SMD:C_0603_1608Metric, F.Cu at (168.6, 117.0)
- added C8: 100n, Capacitor_SMD:C_0603_1608Metric, F.Cu at (161.5, 111.2)
- added C9: 100n, Capacitor_SMD:C_0603_1608Metric, F.Cu at (169.0, 104.0)
- added D1: NUP2105L, Package_TO_SOT_SMD:SOT-23, F.Cu at (149.5, 70.0)
- added D10: 3.3V, Diode_SMD:D_SOD-123, F.Cu at (168.2, 129.8)
- added D11: 3.3V, Diode_SMD:D_SOD-123, F.Cu at (182.2, 129.8)
- added D12: 3.3V, Diode_SMD:D_SOD-123, F.Cu at (327.7, 5.60)
- added D13: 3.3V, Diode_SMD:D_SOD-123, F.Cu at (316.2, 15.7)
- added D14: 3.3V, Diode_SMD:D_SOD-123, F.Cu at (316.2, 22.4)
- added D15: 3.3V, Diode_SMD:D_SOD-123, F.Cu at (322.0, 8.95)
- added D16: 3.3V, Diode_SMD:D_SOD-123, F.Cu at (322.0, 12.3)
- added D17: 3.3V, Diode_SMD:D_SOD-123, F.Cu at (316.2, 5.60)
- added D18: 3.3V, Diode_SMD:D_SOD-123, F.Cu at (316.2, 12.3)
- added D19: 3.3V, Diode_SMD:D_SOD-123, F.Cu at (316.2, 8.95)
- added D2: User, LED_SMD:LED_0805_2012Metric, F.Cu at (249.5, 119.5)
- added D20: 3.3V, Diode_SMD:D_SOD-123, F.Cu at (322.0, 5.60)
- added D21: 3.3V, Diode_SMD:D_SOD-123, F.Cu at (327.7, 8.95)
- added D22: 3.3V, Diode_SMD:D_SOD-123, F.Cu at (333.5, 5.60)
- added D23: 3.3V, Diode_SMD:D_SOD-123, F.Cu at (316.2, 19.0)
- added D24: D_Schottky, Diode_SMD:D_SOD-123, F.Cu at (463.4, 94.0)
- added D25: 33V, Diode_SMD:D_SMB, F.Cu at (447.1, 87.2)
- added D26: D_Schottky, Diode_SMD:D_SOD-123, F.Cu at (463.4, 97.4)
- added D27: 33V, Diode_SMD:D_SMB, F.Cu at (455.5, 81.7)
- added D28: D_Schottky, Diode_SMD:D_SOD-123, F.Cu at (463.4, 90.7)
- added D29: 33V, Diode_SMD:D_SMB, F.Cu at (447.1, 81.7)
- added D3: Heartbeat, LED_SMD:LED_0805_2012Metric, F.Cu at (245.0, 119.5)
- added D30: D_Schottky, Diode_SMD:D_SOD-123, F.Cu at (469.1, 90.7)
- added D31: 33V, Diode_SMD:D_SMB, F.Cu at (447.1, 92.8)
- added D32: 10V, Diode_SMD:D_SOD-123, F.Cu at (178.0, 70.0)
- added D33: 33V, Diode_SMD:D_SMB, F.Cu at (183.0, 58.5)
- added D4: 3.3V, Diode_SMD:D_SOD-123, F.Cu at (157.8, 129.8)
- added D5: 3.3V, Diode_SMD:D_SOD-123, F.Cu at (171.8, 129.8)
- added D6: 3.3V, Diode_SMD:D_SOD-123, F.Cu at (161.2, 129.8)
- added D7: 3.3V, Diode_SMD:D_SOD-123, F.Cu at (175.2, 129.8)
- added D8: 3.3V, Diode_SMD:D_SOD-123, F.Cu at (164.8, 129.8)
- added D9: 3.3V, Diode_SMD:D_SOD-123, F.Cu at (178.8, 129.8)
- added F1: 1A, Fuse:Fuse_1206_3216Metric, F.Cu at (454.1, 86.1)
- added F2: 1A, Fuse:Fuse_1206_3216Metric, F.Cu at (437.3, 93.5)
- added F3: 1A, Fuse:Fuse_1206_3216Metric, F.Cu at (454.1, 89.4)
- added F4: 1A, Fuse:Fuse_1206_3216Metric, F.Cu at (459.7, 86.1)
- added F5: 1A, Littelfuse-154:Littelfuse-154, F.Cu at (185.0, 53.0)
- added H1: M3, MountingHole:MountingHole_3.2mm_M3_Pad_Via, F.Cu at (105.0, 55.0)
- added H2: M3, MountingHole:MountingHole_3.2mm_M3_Pad_Via, F.Cu at (195.0, 55.0)
- added H3: M3, MountingHole:MountingHole_3.2mm_M3_Pad_Via, F.Cu at (105.0, 145.0)
- added H4: M3, MountingHole:MountingHole_3.2mm_M3_Pad_Via, F.Cu at (195.0, 145.0)
- added J10: IO2, canbrd_conn:NH0810x0xxxxG, F.Cu at (106.0, 120.0)
- added J11: I^{2}C, Connector_PinHeader_2.54mm:PinHeader_2x04_P2.54mm_Vertical_SMD, F.Cu at (320.8, 133.6)
- added J12: PwrOut, canbrd_conn:NH0810x0xxxxG, F.Cu at (194.0, 100.0)
- added J13: USB_C_Receptacle_USB2.0, Connector_USB:USB_C_Receptacle_GCT_USB4085, F.Cu at (191.1, 129.8)
- added J14: IO1, canbrd_conn:NH0810x0xxxxG, F.Cu at (130.0, 144.0)
- added J15: IO0, canbrd_conn:NH0810x0xxxxG, F.Cu at (170.0, 144.0)
- added J2: UPDI, Connector_PinHeader_1.27mm:PinHeader_2x03_P1.27mm_Vertical_SMD, F.Cu at (232.0, 127.0)
- added J3: Micro_SD_Card, GTFH081x1YHR:GTFH081x1YHR, F.Cu at (83.0, 68.0)
- added J4: GND, canbrd_conn:NH0210x0xxxxG, F.Cu at (165.0, 56.0)
- added J5: Field24V, canbrd_conn:NH0210x0xxxxG, F.Cu at (175.0, 56.0)
- added J6: RJ45_Shielded, Connector_RJ:RJ45_Amphenol_RJHSE5380, F.Cu at (126.4, 59.1)
- added J8: CAN, canbrd_conn:NH0210x0xxxxG, F.Cu at (150.0, 56.0)
- added J9: CAN, canbrd_conn:NH0210x0xxxxG, F.Cu at (130.0, 56.0)
- added JP1: Pin5, Jumper:SolderJumper-3_P1.3mm_Bridged2Bar12_Pad1.0x1.5mm, B.Cu at (153.4, 75.1)
- added JP10: LowZ, Jumper:SolderJumper-2_P1.3mm_Open_TrianglePad1.0x1.5mm, B.Cu at (175.2, 137.2)
- added JP11: Vdiv, Jumper:SolderJumper-2_P1.3mm_Open_TrianglePad1.0x1.5mm, B.Cu at (164.8, 133.8)
- added JP12: Vdiv, Jumper:SolderJumper-2_P1.3mm_Open_TrianglePad1.0x1.5mm, B.Cu at (178.8, 133.8)
- added JP13: LowZ, Jumper:SolderJumper-2_P1.3mm_Open_TrianglePad1.0x1.5mm, B.Cu at (164.8, 137.2)
- added JP14: LowZ, Jumper:SolderJumper-2_P1.3mm_Open_TrianglePad1.0x1.5mm, B.Cu at (178.8, 137.2)
- added JP15: Vdiv, Jumper:SolderJumper-2_P1.3mm_Open_TrianglePad1.0x1.5mm, B.Cu at (168.2, 133.8)
- added JP16: Vdiv, Jumper:SolderJumper-2_P1.3mm_Open_TrianglePad1.0x1.5mm, B.Cu at (182.2, 133.8)
- added JP17: LowZ, Jumper:SolderJumper-2_P1.3mm_Open_TrianglePad1.0x1.5mm, B.Cu at (168.2, 137.2)
- added JP18: LowZ, Jumper:SolderJumper-2_P1.3mm_Open_TrianglePad1.0x1.5mm, B.Cu at (182.2, 137.2)
- added JP19: Addr, Jumper:SolderJumper-2_P1.3mm_Open_TrianglePad1.0x1.5mm, B.Cu at (238.0, 130.0)
- added JP2: Pin8, Jumper:SolderJumper-3_P1.3mm_Bridged2Bar12_Pad1.0x1.5mm, B.Cu at (145.5, 75.1)
- added JP20: Vdiv, Jumper:SolderJumper-2_P1.3mm_Open_TrianglePad1.0x1.5mm, F.Cu at (329.8, 18.6)
- added JP21: Vdiv, Jumper:SolderJumper-2_P1.3mm_Open_TrianglePad1.0x1.5mm, F.Cu at (355.7, 5.70)
- added JP22: Vdiv, Jumper:SolderJumper-2_P1.3mm_Open_TrianglePad1.0x1.5mm, F.Cu at (339.7, 14.0)
- added JP23: LowZ, Jumper:SolderJumper-2_P1.3mm_Open_TrianglePad1.0x1.5mm, F.Cu at (348.4, 12.8)
- added JP24: LowZ, Jumper:SolderJumper-2_P1.3mm_Open_TrianglePad1.0x1.5mm, F.Cu at (325.4, 21.9)
- added JP25: LowZ, Jumper:SolderJumper-2_P1.3mm_Open_TrianglePad1.0x1.5mm, F.Cu at (336.9, 10.4)
- added JP26: Vdiv, Jumper:SolderJumper-2_P1.3mm_Open_TrianglePad1.0x1.5mm, F.Cu at (342.7, 5.70)
- added JP27: Vdiv, Jumper:SolderJumper-2_P1.3mm_Open_TrianglePad1.0x1.5mm, F.Cu at (335.3, 14.0)
- added JP28: Vdiv, Jumper:SolderJumper-2_P1.3mm_Open_TrianglePad1.0x1.5mm, F.Cu at (351.4, 5.70)
- added JP29: LowZ, Jumper:SolderJumper-2_P1.3mm_Open_TrianglePad1.0x1.5mm, F.Cu at (332.5, 25.6)
- added JP3: Vdiv, Jumper:SolderJumper-2_P1.3mm_Open_TrianglePad1.0x1.5mm, B.Cu at (157.8, 133.8)
- added JP30: LowZ, Jumper:SolderJumper-2_P1.3mm_Open_TrianglePad1.0x1.5mm, F.Cu at (334.1, 22.1)
- added JP31: LowZ, Jumper:SolderJumper-2_P1.3mm_Open_TrianglePad1.0x1.5mm, F.Cu at (338.5, 21.1)
- added JP32: Vdiv, Jumper:SolderJumper-2_P1.3mm_Open_TrianglePad1.0x1.5mm, F.Cu at (329.8, 22.1)
- added JP33: Vdiv, Jumper:SolderJumper-2_P1.3mm_Open_TrianglePad1.0x1.5mm, F.Cu at (342.8, 17.6)
- added JP34: Vdiv, Jumper:SolderJumper-2_P1.3mm_Open_TrianglePad1.0x1.5mm, F.Cu at (328.2, 25.6)
- added JP35: LowZ, Jumper:SolderJumper-2_P1.3mm_Open_TrianglePad1.0x1.5mm, F.Cu at (345.6, 9.25)
- added JP36: LowZ, Jumper:SolderJumper-2_P1.3mm_Open_TrianglePad1.0x1.5mm, F.Cu at (341.3, 10.4)
- added JP37: LowZ, Jumper:SolderJumper-2_P1.3mm_Open_TrianglePad1.0x1.5mm, F.Cu at (336.9, 25.6)
- added JP38: Vdiv, Jumper:SolderJumper-2_P1.3mm_Open_TrianglePad1.0x1.5mm, F.Cu at (344.0, 14.0)
- added JP39: Vdiv, Jumper:SolderJumper-2_P1.3mm_Open_TrianglePad1.0x1.5mm, F.Cu at (338.5, 17.6)
- added JP4: Vdiv, Jumper:SolderJumper-2_P1.3mm_Open_TrianglePad1.0x1.5mm, B.Cu at (171.8, 133.8)
- added JP40: Vdiv, Jumper:SolderJumper-2_P1.3mm_Open_TrianglePad1.0x1.5mm, F.Cu at (334.1, 18.6)
- added JP41: LowZ, Jumper:SolderJumper-2_P1.3mm_Open_TrianglePad1.0x1.5mm, F.Cu at (323.8, 25.4)
- added JP42: LowZ, Jumper:SolderJumper-2_P1.3mm_Open_TrianglePad1.0x1.5mm, F.Cu at (347.0, 5.70)
- added JP43: LowZ, Jumper:SolderJumper-2_P1.3mm_Open_TrianglePad1.0x1.5mm, F.Cu at (350.0, 9.25)
- added JP5: LowZ, Jumper:SolderJumper-2_P1.3mm_Open_TrianglePad1.0x1.5mm, B.Cu at (157.8, 137.2)
- added JP6: LowZ, Jumper:SolderJumper-2_P1.3mm_Open_TrianglePad1.0x1.5mm, B.Cu at (171.8, 137.2)
- added JP7: Vdiv, Jumper:SolderJumper-2_P1.3mm_Open_TrianglePad1.0x1.5mm, B.Cu at (161.2, 133.8)
- added JP8: Vdiv, Jumper:SolderJumper-2_P1.3mm_Open_TrianglePad1.0x1.5mm, B.Cu at (175.2, 133.8)
- added JP9: LowZ, Jumper:SolderJumper-2_P1.3mm_Open_TrianglePad1.0x1.5mm, B.Cu at (161.2, 137.2)
- added L1: 3.3u, Inductor_SMD:L_1008_2520Metric, F.Cu at (185.5, 75.5)
- added Q1: 2N7002K, Package_TO_SOT_SMD:SOT-23, F.Cu at (147.9, 83.9)
- added Q2: 2N7002K, Package_TO_SOT_SMD:SOT-23, F.Cu at (251.2, 111.0)
- added Q3: 2N7002, Package_TO_SOT_SMD:SOT-23, F.Cu at (277.9, 97.0)
- added Q4: AO4828, Package_SO:SOIC-8_3.9x4.9mm_P1.27mm, F.Cu at (438.7, 88.6)
- added Q5: AO4828, Package_SO:SOIC-8_3.9x4.9mm_P1.27mm, F.Cu at (438.7, 82.1)
- added Q6: Q_PMOS_GDS, Package_TO_SOT_SMD:TO-252-2, F.Cu at (183.0, 67.1)
- added R1: 220, Resistor_SMD:R_0603_1608Metric, F.Cu at (177.5, 117.0)
- added R10: 10k, Resistor_SMD:R_0603_1608Metric, F.Cu at (151.1, 86.7)
- added R11: 1k, Resistor_SMD:R_0603_1608Metric, F.Cu at (452.6, 143.4)
- added R12: 1k, Resistor_SMD:R_0603_1608Metric, F.Cu at (253.7, 114.8)
- added R13: 1k, Resistor_SMD:R_0603_1608Metric, F.Cu at (265.7, 110.0)
- added R14: 220, Resistor_SMD:R_0603_1608Metric, F.Cu at (261.7, 110.0)
- added R15: 10k, Resistor_SMD:R_0603_1608Metric, F.Cu at (257.7, 114.8)
- added R16: 220, Resistor_SMD:R_0603_1608Metric, F.Cu at (230.5, 134.2)
- added R17: 10k, Resistor_SMD:R_0603_1608Metric, F.Cu at (178.0, 75.5)
- added R2: 27, Resistor_SMD:R_0603_1608Metric, F.Cu at (182.5, 111.4)
- added R3: 27, Resistor_SMD:R_0603_1608Metric, F.Cu at (182.5, 112.9)
- added R4: 10k, Resistor_SMD:R_0603_1608Metric, F.Cu at (178.0, 99.0)
- added R5: 1k, Resistor_SMD:R_0603_1608Metric, F.Cu at (182.0, 99.0)
- added R6: 1k, Resistor_SMD:R_0603_1608Metric, F.Cu at (161.5, 109.7)
- added R7: 1k, Resistor_SMD:R_0603_1608Metric, F.Cu at (147.9, 86.7)
- added R8: 1k, Resistor_SMD:R_0603_1608Metric, F.Cu at (147.9, 81.1)
- added R9: 4k7, Resistor_SMD:R_0603_1608Metric, F.Cu at (151.1, 83.9)
- added RN1: 220, Resistor_SMD:R_Array_Convex_4x0603, F.Cu at (255.8, 111.2)
- added RN10: 1k, Resistor_SMD:R_Array_Convex_4x0603, F.Cu at (177.0, 133.8)
- added RN11: 68, Resistor_SMD:R_Array_Convex_4x0603, F.Cu at (321.2, 21.1)
- added RN12: 10k, Resistor_SMD:R_Array_Convex_4x0603, F.Cu at (315.4, 26.4)
- added RN13: 68, Resistor_SMD:R_Array_Convex_4x0603, F.Cu at (321.2, 16.4)
- added RN14: 10k, Resistor_SMD:R_Array_Convex_4x0603, F.Cu at (331.1, 14.4)
- added RN15: 68, Resistor_SMD:R_Array_Convex_4x0603, F.Cu at (319.6, 26.4)
- added RN16: 10k, Resistor_SMD:R_Array_Convex_4x0603, F.Cu at (325.3, 17.8)
- added RN17: 1k, Resistor_SMD:R_Array_Convex_4x0603, F.Cu at (326.9, 13.0)
- added RN18: 1k, Resistor_SMD:R_Array_Convex_4x0603, F.Cu at (332.7, 9.65)
- added RN19: 1k, Resistor_SMD:R_Array_Convex_4x0603, F.Cu at (338.4, 6.30)
- added RN2: 10k, Resistor_SMD:R_Array_Convex_4x0603, F.Cu at (244.9, 115.6)
- added RN3: 220, Resistor_SMD:R_Array_Convex_4x0603, F.Cu at (277.5, 101.5)
- added RN4: 10k, Resistor_SMD:R_Array_Convex_4x0603, F.Cu at (249.0, 115.6)
- added RN5: 330, Resistor_SMD:R_Array_Convex_4x0603, F.Cu at (163.0, 125.5)
- added RN6: 10k, Resistor_SMD:R_Array_Convex_4x0603, F.Cu at (163.0, 137.5)
- added RN7: 330, Resistor_SMD:R_Array_Convex_4x0603, F.Cu at (177.0, 125.5)
- added RN8: 10k, Resistor_SMD:R_Array_Convex_4x0603, F.Cu at (177.0, 137.5)
- added RN9: 1k, Resistor_SMD:R_Array_Convex_4x0603, F.Cu at (163.0, 133.8)
- added RV1: 20V, Resistor_SMD:R_1206_3216Metric, F.Cu at (190.0, 59.5)
- added SW1: BOOTSEL, PTS815-SJ:PTS815-SJ, F.Cu at (196.0, 118.0)
- added SW2: RESET, PTS815-SJ:PTS815-SJ, F.Cu at (150.0, 146.0)
- added SW3: SW_DIP_x08, Button_Switch_SMD:SW_DIP_SPSTx08_Slide_Omron_A6H-8101_W6.15mm_P1.27mm, F.Cu at (107.0, 89.5)
- added SW4: User, PTS815-SJ:PTS815-SJ, F.Cu at (245.8, 111.0)
- added U1: W25Q16JVSNIQ, Package_SO:SOIC-8_3.9x4.9mm_P1.27mm, F.Cu at (180.0, 102.5)
- added U2: RP2040, RP2040:RP2040-QFN-56, F.Cu at (170.0, 111.0)
- added U3: TJA1051T-3, Package_SO:SOIC-8_3.9x4.9mm_P1.27mm, F.Cu at (149.5, 76.5)
- added U4: MCP2510-x/SO, Package_SO:SOIC-18W_7.5x11.6mm_P1.27mm, F.Cu at (424.9, 129.3)
- added U5: MAX3485CSA, Package_SO:SOIC-8_3.9x4.9mm_P1.27mm, F.Cu at (143.0, 76.5)
- added U6: SA39-11EWA, Display_7Segment:Sx39-1xxxxx, F.Cu at (112.0, 64.3)
- added U7: SA39-11EWA, Display_7Segment:Sx39-1xxxxx, F.Cu at (112.0, 75.3)
- added U8: ATtiny427, Package_DFN_QFN:QFN-24-1EP_4x4mm_P0.5mm_EP2.6x2.6mm, F.Cu at (237.5, 133.5)
- added U9: M24C04-WMN, Package_SO:SOIC-8_3.9x4.9mm_P1.27mm, F.Cu at (366.8, 54.5)
- added Y1: 12MHz, Crystal:Crystal_SMD_3225-4Pin_3.2x2.5mm, F.Cu at (157.2, 108.7)
- added Y2: 16MHz, Crystal:Crystal_SMD_3225-4Pin_3.2x2.5mm, F.Cu at (462.1, 127.5)
- J1: value PowerIn -> RP_DEBUG; footprint canbrd_conn:10127819-04xxxPxLF -> Connector_PinHeader_1.27mm:PinHeader_2x05_P1.27mm_Vertical_SMD
- J7: value PowerThru -> RJ45_Shielded; footprint canbrd_conn:10127819-04xxxPxLF -> Connector_RJ:RJ45_Amphenol_RJHSE5380
- moved J1 46.2 mm to (148.0, 111.0), turned to -90 degrees
- moved J7 34.3 mm to (146.4, 59.1), turned to 0 degrees
Connections:
- J1 pad 1: unconnected-(J1-Pad1) -> +3V3
- J1 pad 2: unconnected-(J1-Pad2) -> /MCU/RP_SWDIO
- J1 pad 3: unconnected-(J1-Pad3) -> GND
- J1 pad 4: unconnected-(J1-Pad4) -> /MCU/RP_SWCLK
- J7 pad 1: unconnected-(J7-Pad1) -> GND
- J7 pad 2: unconnected-(J7-Pad2) -> /Connectors/Field24V
- J7 pad 3: unconnected-(J7-Pad3) -> GND
- J7 pad 4: unconnected-(J7-Pad4) -> /Connectors/Field24V
Routing:
- net /Connectors/Field24V: track 0.00 -> 97.1 mm
- net /CAN/CANL: track 0.00 -> 63.4 mm
- net /CAN/CANH: track 0.00 -> 60.3 mm, vias 0 -> 1
- net /MCU/~{BOOTSEL}: track 0.00 -> 28.1 mm
- net /MCU/RP_~{RESET}: track 0.00 -> 23.8 mm
- net +24V: track 0.00 -> 23.1 mm
- net /MCU/RP_SWCLK: track 0.00 -> 22.8 mm
- net +3V3: track 0.00 -> 22.4 mm, vias 0 -> 2
- net Net-(D5-Pad1): track 0.00 -> 21.8 mm, vias 0 -> 2
- net Net-(D4-Pad1): track 0.00 -> 21.8 mm, vias 0 -> 2
- net Net-(D11-Pad1): track 0.00 -> 20.3 mm, vias 0 -> 2
- net Net-(D10-Pad1): track 0.00 -> 20.3 mm, vias 0 -> 2
- net /MCU/QSPI_IO3: track 0.00 -> 19.4 mm
- net /MCU/RP_SWDIO: track 0.00 -> 18.7 mm
- net Net-(D8-Pad1): track 0.00 -> 18.0 mm, vias 0 -> 2
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- added copper zone on F.Cu, net +1V1
- added copper zone on F.Cu, net +3.3VA
- added copper zone on F.Cu, net +3.3VA2
- added copper zone on F.Cu, net +3V3
- added copper zone on F.Cu, net +5V
- added copper zone on F.Cu, net /Connectors/Field24V
- added copper zone on F.Cu, net /Power/Fused24V
- added copper zone on F.Cu, net /Power/RevProt24V
- added copper zone on F.Cu, net /Power/revprot_gate
- added copper zone on B.Cu, net GND
- added copper zone on F.Cu, net GND

Commit message: Done?
Parts:
- removed the C24 at (364.6, 59.0)
- removed the D12 at (327.7, 5.60)
- removed the D13 at (316.2, 15.7)
- removed the D22 at (333.5, 5.60)
- removed D27, D29, D31, D33: 33V, Diode_SMD:D_SMB
- removed D28, D30: D_Schottky, Diode_SMD:D_SOD-123
- removed D32: 10V, Diode_SMD:D_SOD-123
- removed the JP20 at (329.8, 18.6)
- removed the JP21 at (355.7, 5.70)
- removed JP40: Vdiv, Jumper:SolderJumper-2_P1.3mm_Open_TrianglePad1.0x1.5mm
- removed JP41, JP42, JP43: LowZ, Jumper:SolderJumper-2_P1.3mm_Open_TrianglePad1.0x1.5mm
- removed Q6: Q_PMOS_GDS, Package_TO_SOT_SMD:TO-252-2
- removed RN15: 68, Resistor_SMD:R_Array_Convex_4x0603
- removed RN16: 10k, Resistor_SMD:R_Array_Convex_4x0603
- removed RN17, RN18, RN19: 1k, Resistor_SMD:R_Array_Convex_4x0603
- removed the RN2 at (244.9, 115.6)
- added C20: 100n, Capacitor_SMD:C_0603_1608Metric, F.Cu at (139.4, 71.5)
- added C28: 100n, Capacitor_SMD:C_0805_2012Metric, F.Cu at (183.0, 77.0)
- added C30: 2.2u, Capacitor_SMD:C_1206_3216Metric, F.Cu at (169.0, 78.1)
- added C31: 2.2u, Capacitor_SMD:C_1206_3216Metric, F.Cu at (169.0, 87.9)
- added C32: 100n, Capacitor_SMD:C_0603_1608Metric, F.Cu at (170.5, 82.2)
- added C33: 22u, Capacitor_SMD:C_1206_3216Metric, F.Cu at (177.5, 87.9)
- added C34: 22u, Capacitor_SMD:C_1206_3216Metric, F.Cu at (177.5, 78.1)
- added C35: 5.6n, Capacitor_SMD:C_0603_1608Metric, F.Cu at (162.6, 83.8)
- added C36: 2.2u, Capacitor_SMD:C_0603_1608Metric, F.Cu at (163.5, 80.7)
- added C37: 100n, Capacitor_SMD:C_0603_1608Metric, F.Cu at (172.1, 94.8)
- added C38: 10u, Capacitor_SMD:C_0805_2012Metric, F.Cu at (178.2, 93.0)
- added C39: 22u, Capacitor_SMD:C_1206_3216Metric, F.Cu at (180.5, 96.0)
- added C40: 22u, Capacitor_SMD:C_1206_3216Metric, F.Cu at (183.0, 96.0)
- added D1: TBU-CA, TBU-CA:DIOC650X400X100N, F.Cu at (123.8, 72.0)
- added D2: TBU-CA, TBU-CA:DIOC650X400X100N, F.Cu at (129.0, 72.0)
- added D26: 30V, Diode_SMD:D_SOD-123, F.Cu at (176.0, 63.5)
- added F6: 1A, Fuse:Fuse_1206_3216Metric, F.Cu at (113.8, 114.8)
- added F7: 1A, Fuse:Fuse_1206_3216Metric, F.Cu at (113.8, 111.2)
- added F8: 500mA, Fuse:Fuse_1206_3216Metric, F.Cu at (113.8, 107.8)
- added F9: 1A, Littelfuse-154:Littelfuse-154, F.Cu at (184.8, 52.8)
- added H3: M3, MountingHole:MountingHole_3.2mm_M3_Pad_Via, F.Cu at (145.0, 95.0)
- added JP3: Pin5L, Jumper:SolderJumper-2_P1.3mm_Open_TrianglePad1.0x1.5mm, B.Cu at (139.7, 73.5)
- added JP4: Pin8L, Jumper:SolderJumper-2_P1.3mm_Bridged_Pad1.0x1.5mm, B.Cu at (130.7, 73.5)
- added L2: 2.2u, Inductor_SMD:L_Taiyo-Yuden_NR-50xx, F.Cu at (175.8, 97.7)
- added R18: 10k, Resistor_SMD:R_0603_1608Metric, F.Cu at (177.5, 74.0)
- added R19: 31.6k, Resistor_SMD:R_0603_1608Metric, F.Cu at (171.3, 92.5)
- added R20: 10k, Resistor_SMD:R_0603_1608Metric, F.Cu at (171.3, 90.9)
- added R21: 5.1k, Resistor_SMD:R_0603_1608Metric, F.Cu at (192.2, 131.8)
- added R22: 5.1k, Resistor_SMD:R_0603_1608Metric, F.Cu at (195.8, 131.8)
- added RN3: 330, Resistor_SMD:R_Array_Convex_4x0603, F.Cu at (163.0, 133.5)
- added U10: ULN2003A, Package_SO:SOIC-16_3.9x9.9mm_P1.27mm, F.Cu at (121.2, 112.5)
- added U11: MAX17634BATP+, MAX17634:TQFN20-EP, F.Cu at (167.0, 83.0)
- added U12: AP62250WU, TSOT26:TSOT26, F.Cu at (175.0, 93.0)
- added kibuzzard-621788DF: G***, kibuzzard-621788DF, F.Cu at (147.0, 105.7)
- D22: renamed from D24; value D_Schottky -> 33V; footprint Diode_SMD:D_SOD-123 -> Diode_SMD:D_SMB
- D23: value 3.3V -> 33V; footprint Diode_SMD:D_SOD-123 -> Diode_SMD:D_SMB
- D24: renamed from D26; value D_Schottky -> 10V
- F4: value 1A -> 500mA
- F5: footprint Littelfuse-154:Littelfuse-154 -> Fuse:Fuse_1206_3216Metric
- J13: value USB_C_Receptacle_USB2.0 -> USB_C_Receptacle; footprint Connector_USB:USB_C_Receptacle_GCT_USB4085 -> 10132328:10132328
- J6, J7: value RJ45_Shielded -> Amphenol RJHSE5380
- JP1: value Pin5 -> Pin5H; footprint Jumper:SolderJumper-3_P1.3mm_Bridged2Bar12_Pad1.0x1.5mm -> Jumper:SolderJumper-2_P1.3mm_Bridged_Pad1.0x1.5mm
- JP10: renamed from JP8; value Vdiv -> LowZ
- JP11: renamed from JP9; value LowZ -> Vdiv
- JP12: renamed from JP10; value LowZ -> Vdiv
- JP13: renamed from JP11; value Vdiv -> LowZ
- JP14: renamed from JP12; value Vdiv -> LowZ
- JP15: renamed from JP13; value LowZ -> Vdiv
- JP16: renamed from JP14; value LowZ -> Vdiv
- JP17: renamed from JP15; value Vdiv -> LowZ
- JP18: renamed from JP16; value Vdiv -> LowZ
- JP19: renamed from JP17; value LowZ -> Vdiv
- JP2: value Pin8 -> Pin8H; footprint Jumper:SolderJumper-3_P1.3mm_Bridged2Bar12_Pad1.0x1.5mm -> Jumper:SolderJumper-2_P1.3mm_Open_TrianglePad1.0x1.5mm
- JP20: renamed from JP18; value LowZ -> Vdiv
- JP22, JP26, JP27, JP34: value Vdiv -> LowZ; moved to B.Cu
- JP23, JP28, JP30, JP31, JP32, JP33, JP35: moved to B.Cu
- JP24, JP25, JP29, JP36, JP37: value LowZ -> Vdiv; moved to B.Cu
- JP38: value Vdiv -> DCM; moved to B.Cu
- JP39: value Vdiv -> PWM; moved to B.Cu
- JP5: renamed from JP3; value Vdiv -> LowZ
- JP6: renamed from JP4; value Vdiv -> LowZ
- JP7: renamed from JP5; value LowZ -> Vdiv
- JP8: renamed from JP6; value LowZ -> Vdiv
- JP9: renamed from JP7; value Vdiv -> LowZ
- L1: value 3.3u -> 6.8u; footprint Inductor_SMD:L_1008_2520Metric -> Inductor_SMD:L_Abracon_ASPI-0630LR
- Q2: value 2N7002K -> BSS83P
- Q3: value 2N7002 -> BSS83P
- Q4: value AO4828 -> Q_PMOS_GDS; footprint Package_SO:SOIC-8_3.9x4.9mm_P1.27mm -> Package_TO_SOT_SMD:TO-252-2
- Q5: value AO4828 -> BC856; footprint Package_SO:SOIC-8_3.9x4.9mm_P1.27mm -> Package_TO_SOT_SMD:SOT-23
- R12: renamed from R14; value 220 -> 470
- R15: value 10k -> 220
- R16: value 220 -> 1k
- RN1: value 220 -> 470
- RN10: value 1k -> 10k
- RN13: value 68 -> 1k; moved to B.Cu
- RN14, RN8: value 10k -> 1k; moved to B.Cu
- RN2: renamed from RN3; value 220 -> 470
- RN7: value 330 -> 1k; moved to B.Cu
- RN9: value 1k -> 68
- RV1: value 20V -> 30V
- U6, U7: value SA39-11EWA -> 157119S12801
- U9: value M24C04-WMN -> ULN2003A; footprint Package_SO:SOIC-8_3.9x4.9mm_P1.27mm -> Package_SO:SOIC-16_3.9x9.9mm_P1.27mm
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- renumbered C20 to C21, C21 to C22, C22 to C23, C23 to C24, C28 to C29, D8 to D10, D9 to D11, D10 to D12, D11 to D13, D1 to D3, D2 to D4, D3 to D5, D4 to D6, D5 to D7, D6 to D8, D7 to D9, H3 to H4, H4 to H5, J12 to J10, J10 to J11, J11 to J12, JP19 to JP21, R12 to R14
Connections:
- net Net-(J13-PadA4) renamed VBUS
- C26 pad 1: /Power/RevProt24V -> +24V
- D10 pad 1: Net-(D8-Pad1) -> /IO/RP2
- D11 pad 1: Net-(D9-Pad1) -> /IO/RP6
- D12 pad 1: Net-(D10-Pad1) -> /IO/RP3
- D13 pad 1: Net-(D11-Pad1) -> /IO/RP7
- D14 pad 1: Net-(D14-Pad1) -> /IO Expander/IO Expander Protection/AT1.0
- D15 pad 1: Net-(D15-Pad1) -> /IO Expander/IO Expander Protection/AT1.4
- D16 pad 1: Net-(D16-Pad1) -> /IO Expander/IO Expander Protection/AT1.1
- D17 pad 1: Net-(D17-Pad1) -> /IO Expander/IO Expander Protection/AT1.5
- D18 pad 1: Net-(D18-Pad1) -> /IO Expander/IO Expander Protection/AT1.2
- D19 pad 1: Net-(D19-Pad1) -> /IO Expander/IO Expander Protection/AT1.6
- D20 pad 1: Net-(D20-Pad1) -> /IO Expander/IO Expander Protection/AT1.3
- D21 pad 1: Net-(D21-Pad1) -> /IO Expander/IO Expander Protection/AT1.7
- D22 pad 1: Net-(D24-Pad1) -> /IO Expander/IO Expander Power IO/COM0
- D23 pad 1: Net-(D23-Pad1) -> /IO Expander/IO Expander Power IO/COM1
- D24 pad 1: Net-(D26-Pad1) -> +24V
- D24 pad 2: GND -> /Power/revprot_gate
- D25 pad 2: Net-(D24-Pad1) -> /Power/Fused24V
- D3 pad 1: /CAN/CANL -> Net-(D2-Pad1)
- D3 pad 2: /CAN/CANH -> Net-(D1-Pad1)
- D4 pad 1: unconnected-(D2-Pad1) -> /DISP+SW/SegR.8
- D4 pad 2: /DISP+SW/SegR.8 -> /DISP+SW/nDig
- D5 pad 1: unconnected-(D3-Pad1) -> /DISP+SW/SegR.8
- D5 pad 2: /DISP+SW/SegR.8 -> /DISP+SW/~{nDig}
- D6 pad 1: Net-(D4-Pad1) -> /IO/RP0
- D7 pad 1: Net-(D5-Pad1) -> /IO/RP4
- D8 pad 1: Net-(D6-Pad1) -> /IO/RP1
- D9 pad 1: Net-(D7-Pad1) -> /IO/RP5
- F1 pad 1: Net-(D24-Pad1) -> /IO Expander/IO Expander Power IO/HC0
- F1 pad 2: /Connectors/IO2.0 -> /Connectors/IO2.7
- F2 pad 1: Net-(D26-Pad1) -> /IO Expander/IO Expander Power IO/HC1
- F2 pad 2: /Connectors/IO2.1 -> /Connectors/IO2.6
- F3 pad 1: Net-(D28-Pad1) -> /IO Expander/IO Expander Power IO/HC2
- F3 pad 2: /Connectors/IO2.2 -> /Connectors/IO2.5
- F4 pad 1: Net-(D30-Pad1) -> /IO Expander/IO Expander Power IO/HC3
- F4 pad 2: /Connectors/IO2.3 -> /Connectors/IO2.4
- F5 pad 1: /Connectors/Field24V -> /IO Expander/IO Expander Power IO/HC4
- F5 pad 2: /Power/Fused24V -> /Connectors/IO2.3
- J11 pad 1: unconnected-(J10-Pad1) -> /Connectors/IO2.0
- J11 pad 2: unconnected-(J10-Pad2) -> /Connectors/IO2.1
- J11 pad 3: unconnected-(J10-Pad3) -> /Connectors/IO2.2
- J11 pad 4: unconnected-(J10-Pad4) -> /Connectors/IO2.3
- J11 pad 5: unconnected-(J10-Pad5) -> /Connectors/IO2.4
- J11 pad 6: unconnected-(J10-Pad6) -> /Connectors/IO2.5
- J11 pad 7: unconnected-(J10-Pad7) -> /Connectors/IO2.6
- J11 pad 8: unconnected-(J10-Pad8) -> /Connectors/IO2.7
- J12 pad 2: +3V3 -> GND
- J12 pad 7: +3V3 -> GND
- J13 pad A1: Net-(J13-PadA1) -> GND
- J13 pad A12: Net-(J13-PadA1) -> GND
- J13 pad A5: unconnected-(J13-PadA5) -> Net-(J13-PadA5)
- J13 pad A6: unconnected-(J13-PadA6) -> /Connectors/USB+
- J13 pad A7: unconnected-(J13-PadA7) -> /Connectors/USB-
- J13 pad B1: Net-(J13-PadA1) -> GND
- J13 pad B12: Net-(J13-PadA1) -> GND
- J13 pad B5: unconnected-(J13-PadB5) -> Net-(J13-PadB5)
- J13 pad B6: unconnected-(J13-PadB6) -> /Connectors/USB+
- J13 pad B7: unconnected-(J13-PadB7) -> /Connectors/USB-
- J13 pad S1: unconnected-(J13-PadS1) -> GND
- J14 pad 1: unconnected-(J14-Pad1) -> /Connectors/IO1.0
- J14 pad 2: unconnected-(J14-Pad2) -> /Connectors/IO1.1
- J14 pad 3: unconnected-(J14-Pad3) -> /Connectors/IO1.2
- J14 pad 4: unconnected-(J14-Pad4) -> /Connectors/IO1.3
- J14 pad 5: unconnected-(J14-Pad5) -> /Connectors/IO1.4
- J14 pad 6: unconnected-(J14-Pad6) -> /Connectors/IO1.5
- J14 pad 7: unconnected-(J14-Pad7) -> /Connectors/IO1.6
- J14 pad 8: unconnected-(J14-Pad8) -> /Connectors/IO1.7
- J6 pad 1: GND -> /CAN/CANH
- J6 pad 2: /Connectors/Field24V -> /CAN/CANL
- J6 pad 4: /Connectors/Field24V -> unconnected-(J6-Pad4)
- J6 pad 5: GND -> unconnected-(J6-Pad5)
- J6 pad 6: /Connectors/Field24V -> GND
- J6 pad 7: /CAN/CANH -> GND
- J6 pad 8: /CAN/CANL -> /Connectors/Field24V
- J7 pad 1: GND -> /CAN/CANH
- J7 pad 2: /Connectors/Field24V -> /CAN/CANL
- J7 pad 4: /Connectors/Field24V -> unconnected-(J7-Pad4)
- J7 pad 5: GND -> unconnected-(J7-Pad5)
- J7 pad 6: /Connectors/Field24V -> GND
- J7 pad 7: /CAN/CANH -> GND
- J7 pad 8: /CAN/CANL -> /Connectors/Field24V
- J8 pad 1: /CAN/CANL -> /CAN/CANH
- J8 pad 2: /CAN/CANH -> /CAN/CANL
- J9 pad 1: /CAN/CANL -> /CAN/CANH
- J9 pad 2: /CAN/CANH -> /CAN/CANL
- JP1 pad 1: +5V -> /CAN/Pin5
- JP1 pad 2: /CAN/Pin5 -> +5V
- JP10 pad 1: Net-(D7-Pad1) -> Net-(JP10-Pad1)
- JP10 pad 2: Net-(JP8-Pad2) -> /Connectors/IO0.5
- JP11 pad 1: Net-(D6-Pad1) -> Net-(JP11-Pad1)
- JP11 pad 2: /Connectors/IO0.1 -> GND
- JP12 pad 1: Net-(D7-Pad1) -> Net-(JP12-Pad1)
- JP12 pad 2: /Connectors/IO0.5 -> GND
- JP13 pad 1: Net-(D8-Pad1) -> Net-(JP13-Pad1)
- JP13 pad 2: Net-(JP11-Pad2) -> /Connectors/IO0.2
- JP14 pad 1: Net-(D9-Pad1) -> Net-(JP14-Pad1)
- JP14 pad 2: Net-(JP12-Pad2) -> /Connectors/IO0.6
- JP15 pad 1: Net-(D8-Pad1) -> Net-(JP15-Pad1)
- JP15 pad 2: /Connectors/IO0.2 -> GND
- JP16 pad 1: Net-(D9-Pad1) -> Net-(JP16-Pad1)
- JP16 pad 2: /Connectors/IO0.6 -> GND
- JP17 pad 1: Net-(D10-Pad1) -> Net-(JP17-Pad1)
- JP17 pad 2: Net-(JP15-Pad2) -> /Connectors/IO0.3
- JP18 pad 1: Net-(D11-Pad1) -> Net-(JP18-Pad1)
- JP18 pad 2: Net-(JP16-Pad2) -> /Connectors/IO0.7
- JP19 pad 1: Net-(D10-Pad1) -> Net-(JP19-Pad1)
- JP19 pad 2: /Connectors/IO0.3 -> GND
- JP2 pad 1: GND -> +5V
- JP20 pad 1: Net-(D11-Pad1) -> Net-(JP20-Pad1)
- JP20 pad 2: /Connectors/IO0.7 -> GND
- JP22 pad 1: Net-(D14-Pad1) -> Net-(JP22-Pad1)
- JP22 pad 2: Net-(JP22-Pad2) -> /Connectors/IO1.0
- JP23 pad 1: Net-(D12-Pad1) -> Net-(JP23-Pad1)
- JP23 pad 2: /Connectors/IO1.0 -> /Connectors/IO1.4
- JP24 pad 1: Net-(D13-Pad1) -> Net-(JP24-Pad1)
- JP24 pad 2: /Connectors/IO1.4 -> GND
- JP25 pad 1: Net-(D14-Pad1) -> Net-(JP25-Pad1)
- JP25 pad 2: /Connectors/IO2.0 -> GND
- JP26 pad 1: Net-(D15-Pad1) -> Net-(JP26-Pad1)
- JP26 pad 2: Net-(JP26-Pad2) -> /Connectors/IO1.1
- JP27 pad 1: Net-(D16-Pad1) -> Net-(JP27-Pad1)
- JP27 pad 2: Net-(JP27-Pad2) -> /Connectors/IO1.5
- JP28 pad 1: Net-(D17-Pad1) -> Net-(JP28-Pad1)
- JP28 pad 2: Net-(JP28-Pad2) -> GND
- JP29 pad 1: Net-(D15-Pad1) -> Net-(JP29-Pad1)
- JP29 pad 2: /Connectors/IO1.1 -> GND
- JP30 pad 1: Net-(D16-Pad1) -> Net-(JP30-Pad1)
- JP30 pad 2: /Connectors/IO1.5 -> /Connectors/IO1.2
- JP31 pad 1: Net-(D17-Pad1) -> Net-(JP31-Pad1)
- JP31 pad 2: /Connectors/IO2.1 -> /Connectors/IO1.6
- JP32 pad 1: Net-(D18-Pad1) -> Net-(JP32-Pad1)
- JP32 pad 2: Net-(JP32-Pad2) -> GND
- JP33 pad 1: Net-(D19-Pad1) -> Net-(JP33-Pad1)
- JP33 pad 2: Net-(JP33-Pad2) -> GND
- JP34 pad 1: Net-(D20-Pad1) -> Net-(JP34-Pad1)
- JP34 pad 2: Net-(JP34-Pad2) -> /Connectors/IO1.3
- JP35 pad 1: Net-(D18-Pad1) -> Net-(JP35-Pad1)
- JP35 pad 2: /Connectors/IO1.2 -> /Connectors/IO1.7
- JP36 pad 1: Net-(D19-Pad1) -> Net-(JP36-Pad1)
- JP36 pad 2: /Connectors/IO1.6 -> GND
- JP37 pad 1: Net-(D20-Pad1) -> Net-(JP37-Pad1)
- JP37 pad 2: /Connectors/IO2.2 -> GND
- JP38 pad 1: Net-(D21-Pad1) -> /Power/MAX_MODE
- JP38 pad 2: Net-(JP38-Pad2) -> /Power/MAX_INTVCC
- JP39 pad 1: Net-(D22-Pad1) -> GND
- JP39 pad 2: Net-(JP39-Pad2) -> /Power/MAX_MODE
- JP5 pad 1: Net-(D4-Pad1) -> Net-(JP5-Pad1)
- JP5 pad 2: Net-(JP3-Pad2) -> /Connectors/IO0.0
- JP6 pad 1: Net-(D5-Pad1) -> Net-(JP6-Pad1)
- JP6 pad 2: Net-(JP4-Pad2) -> /Connectors/IO0.4
- JP7 pad 1: Net-(D4-Pad1) -> Net-(JP7-Pad1)
- JP7 pad 2: /Connectors/IO0.0 -> GND
- JP8 pad 1: Net-(D5-Pad1) -> Net-(JP8-Pad1)
- JP8 pad 2: /Connectors/IO0.4 -> GND
- JP9 pad 1: Net-(D6-Pad1) -> Net-(JP9-Pad1)
- JP9 pad 2: Net-(JP7-Pad2) -> /Connectors/IO0.1
- L1 pad 1: /Power/RevProt24V -> /Power/MAX_LX
- L1 pad 2: +24V -> +5V
- Q2 pad 1: /DISP+SW/nDig -> /DISP+SW/Dig
- Q2 pad 2: GND -> /DISP+SW/nDig
- Q2 pad 3: /DISP+SW/~{nDig} -> +3V3
- Q3 pad 1: unconnected-(Q3-Pad1) -> /DISP+SW/nDig
- Q3 pad 2: GND -> /DISP+SW/~{nDig}
- Q3 pad 3: /DISP+SW/nDig -> +3V3
- Q4 pad 1: GND -> /Power/revprot_gate
- Q4 pad 2: /IO Expander/IO Expander Power IO/AT2.4 -> /Power/Fused24V
- Q4 pad 3: GND -> +24V
- Q5 pad 1: GND -> Net-(Q5-Pad1)
- Q5 pad 2: /IO Expander/IO Expander Power IO/AT2.6 -> /Power/Fused24V
- Q5 pad 3: GND -> /Power/revprot_gate
- R13 pad 1: +3V3 -> /DISP+SW/~{nDig}
- R13 pad 2: /DISP+SW/~{nDig} -> GND
- R14 pad 1: +3V3 -> /DISP+SW/nDig
- R14 pad 2: /DISP+SW/nDig -> GND
- R15 pad 1: Net-(R15-Pad1) -> +3V3
- R15 pad 2: unconnected-(R15-Pad2) -> +3.3VA2
- R16 pad 1: +3V3 -> Net-(D26-Pad1)
- R16 pad 2: +3.3VA2 -> Net-(Q5-Pad1)
- R17 pad 1: /Power/revprot_gate -> +24V
- RN10 pad 1: GND -> /Connectors/IO1.0
- RN10 pad 2: GND -> /Connectors/IO1.1
- RN10 pad 3: GND -> /Connectors/IO1.2
- RN10 pad 4: GND -> /Connectors/IO1.3
- RN10 pad 5: Net-(JP4-Pad2) -> Net-(JP34-Pad1)
- RN10 pad 6: Net-(JP8-Pad2) -> Net-(JP30-Pad1)
- RN10 pad 7: Net-(JP12-Pad2) -> Net-(JP26-Pad1)
- RN10 pad 8: Net-(JP16-Pad2) -> Net-(JP22-Pad1)
- RN11 pad 1: Net-(D12-Pad1) -> Net-(JP23-Pad1)
- RN11 pad 2: Net-(D15-Pad1) -> Net-(JP27-Pad1)
- RN11 pad 3: Net-(D18-Pad1) -> Net-(JP31-Pad1)
- RN11 pad 4: Net-(D21-Pad1) -> Net-(JP35-Pad1)
- RN11 pad 5: /IO Expander/IO Expander Protection/AT1.3 -> /IO Expander/IO Expander Protection/AT1.7
- RN11 pad 6: /IO Expander/IO Expander Protection/AT1.2 -> /IO Expander/IO Expander Protection/AT1.6
- RN11 pad 7: /IO Expander/IO Expander Protection/AT1.1 -> /IO Expander/IO Expander Protection/AT1.5
- RN11 pad 8: /IO Expander/IO Expander Protection/AT1.0 -> /IO Expander/IO Expander Protection/AT1.4
- RN12 pad 1: /Connectors/IO1.0 -> /Connectors/IO1.4
- RN12 pad 2: /Connectors/IO1.1 -> /Connectors/IO1.5
- RN12 pad 3: /Connectors/IO1.2 -> /Connectors/IO1.6
- RN12 pad 4: /Connectors/IO1.3 -> /Connectors/IO1.7
- RN12 pad 5: Net-(D21-Pad1) -> Net-(JP35-Pad1)
- RN12 pad 6: Net-(D18-Pad1) -> Net-(JP31-Pad1)
- RN12 pad 7: Net-(D15-Pad1) -> Net-(JP27-Pad1)
- RN12 pad 8: Net-(D12-Pad1) -> Net-(JP23-Pad1)
- RN13 pad 1: Net-(D13-Pad1) -> Net-(JP24-Pad1)
- RN13 pad 2: Net-(D16-Pad1) -> Net-(JP28-Pad1)
- RN13 pad 3: Net-(D19-Pad1) -> Net-(JP32-Pad1)
- RN13 pad 4: Net-(D22-Pad1) -> Net-(JP36-Pad1)
- RN13 pad 5: /IO Expander/IO Expander Protection/AT1.7 -> Net-(JP34-Pad1)
- RN13 pad 6: /IO Expander/IO Expander Protection/AT1.6 -> Net-(JP30-Pad1)
- RN13 pad 7: /IO Expander/IO Expander Protection/AT1.5 -> Net-(JP26-Pad1)
- RN13 pad 8: /IO Expander/IO Expander Protection/AT1.4 -> Net-(JP22-Pad1)
- RN14 pad 1: /Connectors/IO1.4 -> Net-(JP25-Pad1)
- RN14 pad 2: /Connectors/IO1.5 -> Net-(JP29-Pad1)
- RN14 pad 3: /Connectors/IO1.6 -> Net-(JP33-Pad1)
- RN14 pad 4: /Connectors/IO1.7 -> Net-(JP37-Pad1)
- RN14 pad 5: Net-(D22-Pad1) -> Net-(JP35-Pad1)
- RN14 pad 6: Net-(D19-Pad1) -> Net-(JP31-Pad1)
- RN14 pad 7: Net-(D16-Pad1) -> Net-(JP27-Pad1)
- RN14 pad 8: Net-(D13-Pad1) -> Net-(JP23-Pad1)
- RN4 pad 1: unconnected-(RN4-Pad1) -> /Connectors/IO0.0
- RN4 pad 2: unconnected-(RN4-Pad2) -> /Connectors/IO0.1
- RN4 pad 3: unconnected-(RN4-Pad3) -> /Connectors/IO0.2
- RN4 pad 4: unconnected-(RN4-Pad4) -> /Connectors/IO0.3
- RN4 pad 5: Net-(RN4-Pad5) -> Net-(JP17-Pad1)
- RN4 pad 6: Net-(RN4-Pad6) -> Net-(JP13-Pad1)
- RN4 pad 7: Net-(RN4-Pad7) -> Net-(JP9-Pad1)
- RN4 pad 8: Net-(RN4-Pad8) -> Net-(JP5-Pad1)
- RN5 pad 1: Net-(D4-Pad1) -> Net-(JP6-Pad1)
- RN5 pad 2: Net-(D6-Pad1) -> Net-(JP10-Pad1)
- RN5 pad 3: Net-(D8-Pad1) -> Net-(JP14-Pad1)
- RN5 pad 4: Net-(D10-Pad1) -> Net-(JP18-Pad1)
- RN5 pad 5: /IO/RP3 -> /IO/RP7
- RN5 pad 6: /IO/RP2 -> /IO/RP6
- RN5 pad 7: /IO/RP1 -> /IO/RP5
- RN5 pad 8: /IO/RP0 -> /IO/RP4
- RN6 pad 1: /Connectors/IO0.0 -> /Connectors/IO0.4
- RN6 pad 2: /Connectors/IO0.1 -> /Connectors/IO0.5
- RN6 pad 3: /Connectors/IO0.2 -> /Connectors/IO0.6
- RN6 pad 4: /Connectors/IO0.3 -> /Connectors/IO0.7
- RN6 pad 5: Net-(D10-Pad1) -> Net-(JP18-Pad1)
- RN6 pad 6: Net-(D8-Pad1) -> Net-(JP14-Pad1)
- RN6 pad 7: Net-(D6-Pad1) -> Net-(JP10-Pad1)
- RN6 pad 8: Net-(D4-Pad1) -> Net-(JP6-Pad1)
- RN7 pad 1: Net-(D5-Pad1) -> Net-(JP7-Pad1)
- RN7 pad 2: Net-(D7-Pad1) -> Net-(JP11-Pad1)
- RN7 pad 3: Net-(D9-Pad1) -> Net-(JP15-Pad1)
- RN7 pad 4: Net-(D11-Pad1) -> Net-(JP19-Pad1)
- RN7 pad 5: /IO/RP7 -> Net-(JP17-Pad1)
- RN7 pad 6: /IO/RP6 -> Net-(JP13-Pad1)
- RN7 pad 7: /IO/RP5 -> Net-(JP9-Pad1)
- RN7 pad 8: /IO/RP4 -> Net-(JP5-Pad1)
- RN8 pad 1: /Connectors/IO0.4 -> Net-(JP8-Pad1)
- RN8 pad 2: /Connectors/IO0.5 -> Net-(JP12-Pad1)
- RN8 pad 3: /Connectors/IO0.6 -> Net-(JP16-Pad1)
- RN8 pad 4: /Connectors/IO0.7 -> Net-(JP20-Pad1)
- RN8 pad 5: Net-(D11-Pad1) -> Net-(JP18-Pad1)
- RN8 pad 6: Net-(D9-Pad1) -> Net-(JP14-Pad1)
- RN8 pad 7: Net-(D7-Pad1) -> Net-(JP10-Pad1)
- RN8 pad 8: Net-(D5-Pad1) -> Net-(JP6-Pad1)
- RN9 pad 1: GND -> Net-(JP22-Pad1)
- RN9 pad 2: GND -> Net-(JP26-Pad1)
- RN9 pad 3: GND -> Net-(JP30-Pad1)
- RN9 pad 4: GND -> Net-(JP34-Pad1)
- RN9 pad 5: Net-(JP3-Pad2) -> /IO Expander/IO Expander Protection/AT1.3
- RN9 pad 6: Net-(JP7-Pad2) -> /IO Expander/IO Expander Protection/AT1.2
- RN9 pad 7: Net-(JP11-Pad2) -> /IO Expander/IO Expander Protection/AT1.1
- RN9 pad 8: Net-(JP15-Pad2) -> /IO Expander/IO Expander Protection/AT1.0
- SW3 pad 1: Net-(SW3-Pad1) -> /DISP+SW/Dig
- SW3 pad 10: Net-(RN4-Pad6) -> /DISP+SW/Seg.6
- SW3 pad 11: Net-(RN4-Pad7) -> /DISP+SW/Seg.5
- SW3 pad 12: Net-(RN4-Pad8) -> /DISP+SW/Seg.4
- SW3 pad 13: Net-(RN2-Pad5) -> /DISP+SW/Seg.3
- SW3 pad 14: Net-(RN2-Pad6) -> /DISP+SW/Seg.2
- SW3 pad 15: Net-(RN2-Pad7) -> /DISP+SW/Seg.1
- SW3 pad 16: Net-(RN2-Pad8) -> /DISP+SW/Seg.0
- SW3 pad 2: Net-(SW3-Pad1) -> /DISP+SW/Dig
- SW3 pad 3: Net-(SW3-Pad1) -> /DISP+SW/Dig
- SW3 pad 4: Net-(SW3-Pad1) -> /DISP+SW/Dig
- SW3 pad 5: Net-(SW3-Pad1) -> /DISP+SW/Dig
- SW3 pad 6: Net-(SW3-Pad1) -> /DISP+SW/Dig
- SW3 pad 7: Net-(SW3-Pad1) -> /DISP+SW/Dig
- SW3 pad 8: Net-(SW3-Pad1) -> /DISP+SW/Dig
- SW3 pad 9: Net-(RN4-Pad5) -> /DISP+SW/Seg.7
- SW4 pad 1: Net-(SW3-Pad1) -> /DISP+SW/Dig
- SW4 pad 2: Net-(R15-Pad1) -> /DISP+SW/Seg.8
- U2 pad 11: /DISP+SW/Seg.8 -> /DISP+SW/Seg.7
- U2 pad 12: /DISP+SW/Dig -> /DISP+SW/Seg.6
- U2 pad 13: /CAN/~{INT} -> /DISP+SW/Seg.5
- U2 pad 14: /CAN/~{RX1} -> /DISP+SW/Seg.4
- U2 pad 15: /CAN/MISO -> /DISP+SW/Seg.3
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Routing:
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- added copper zone on F.Cu, net +24V
- added copper zone on B.Cu, net +5V
- added copper zone on F.Cu, net /IO Expander/IO Expander Power IO/COM0
- added copper zone on F.Cu, net /IO Expander/IO Expander Power IO/COM1
- added copper zone on F.Cu, net /IO Expander/IO Expander Power IO/HC0
- added copper zone on F.Cu, net /IO Expander/IO Expander Power IO/HC1
- added copper zone on F.Cu, net /IO Expander/IO Expander Power IO/HC2
- added copper zone on F.Cu, net /IO Expander/IO Expander Power IO/HC3
- added copper zone on F.Cu, net /IO Expander/IO Expander Power IO/HC4
- added copper zone on F.Cu, net /IO Expander/IO Expander Power IO/HC5
- added copper zone on F.Cu, net /IO Expander/IO Expander Power IO/HC6
- added copper zone on F.Cu, net /IO Expander/IO Expander Power IO/HC7
- added copper zone on F.Cu, net /Power/AP_BST
- added copper zone on F.Cu, net /Power/MAX_LX
- added copper zone on F.Cu, net /Power/SW3v3
- removed copper zone on F.Cu, net /Power/RevProt24V
