File: hardware.kicad_pcb (KiCad board)
At the start: 2 copper layers, 100 x 100 mm, 197 parts, among them J1 RP_DEBUG, J10 PwrOut, J11 IO2, J12 I^{2}C, J13 USB_C_Receptacle, J14 IO1, J15 IO0, J2 UPDI, J3 Micro_SD_Card, J4 GND, J5 Field24V, J6 Amphenol RJHSE5380, J7 Amphenol RJHSE5380, J8 CAN, J9 CAN, Q1 2N7002K, Q2 BSS83P, Q3 BSS83P, Q4 Q_PMOS_GDS, Q5 BC856, SW1 BOOTSEL, SW2 RESET, SW3 SW_DIP_x08, SW4 User, U1 W25Q16JVSNIQ, U10 ULN2003A, U11 MAX17634BATP+, U12 AP62250WU, U2 RP2040, U3 TJA1051T-3, U4 MCP2510-x/SO, U5 MAX3485CSA, U6 157119S12801, U7 157119S12801, U8 ATtiny427, U9 ULN2003A, Y1 12MHz, Y2 16MHz

Commit message: WIP: display
Parts:
- added U7: DC56-11CGKWA, Display_7Segment:DA56-11CGKWA, F.Cu at (222.7, 106.1)
- added kibuzzard-62179C2A: G***, kibuzzard-62179C2A, F.Cu at (188.5, 89.5)
- added kibuzzard-62179C5E: G***, kibuzzard-62179C5E, F.Cu at (188.5, 96.5)
- added kibuzzard-62179C9D: G***, kibuzzard-62179C9D, F.Cu at (188.5, 103.5)
- added kibuzzard-62179CFC: G***, kibuzzard-62179CFC, F.Cu at (188.5, 110.5)
- added kibuzzard-62179D4A: G***, kibuzzard-62179D4A, F.Cu at (165.0, 61.5)
- added kibuzzard-62179E31: G***, kibuzzard-62179E31, F.Cu at (175.0, 61.5)
- added kibuzzard-62179E98: G***, kibuzzard-62179E98, F.Cu at (149.2, 63.0)
- added kibuzzard-62179EAF: G***, kibuzzard-62179EAF, F.Cu at (129.0, 63.0)
- added kibuzzard-62179F21: G***, kibuzzard-62179F21, F.Cu at (197.5, 118.0)
- added kibuzzard-62179F8F: G***, kibuzzard-62179F8F, F.Cu at (170.0, 138.2)
- added kibuzzard-62179F9F: G***, kibuzzard-62179F9F, F.Cu at (140.0, 138.2)
- added kibuzzard-62179FB2: G***, kibuzzard-62179FB2, F.Cu at (103.8, 135.5)
- added kibuzzard-6217A003: G***, kibuzzard-6217A003, F.Cu at (156.8, 138.2)
- added kibuzzard-6217A022: G***, kibuzzard-6217A022, F.Cu at (183.2, 138.2)
- added kibuzzard-6217A03E: G***, kibuzzard-6217A03E, F.Cu at (153.2, 138.2)
- added kibuzzard-6217A08D: G***, kibuzzard-6217A08D, F.Cu at (126.2, 138.2)
- added kibuzzard-6217A0B8: G***, kibuzzard-6217A0B8, F.Cu at (111.5, 105.2)
- added kibuzzard-6217A0C8: G***, kibuzzard-6217A0C8, F.Cu at (111.5, 134.8)
- added kibuzzard-6217A0EA: G***, kibuzzard-6217A0EA, F.Cu at (130.0, 116.5)
- added kibuzzard-621B6EAC: G***, kibuzzard-621B6EAC, F.Cu at (118.0, 52.5)
- added kibuzzard-621B6EB9: G***, kibuzzard-621B6EB9, F.Cu at (118.0, 55.5)
- added kibuzzard-621B6EDA: G***, kibuzzard-621B6EDA, F.Cu at (118.0, 58.0)
- SW3: footprint Button_Switch_SMD:SW_DIP_SPSTx08_Slide_Omron_A6H-8101_W6.15mm_P1.27mm -> Button_Switch_SMD:SW_DIP_SPSTx08_Slide_KingTek_DSHP08TS_W7.62mm_P1.27mm
- moved SW4 51.0 mm to (113.0, 52.5), turned to 0 degrees
- moved R12 2.00 mm to (116.0, 61.0)
- moved SW3 0.70 mm to (109.0, 97.7)
- moved D4 0.50 mm to (113.0, 55.5)
- renumbered U9 to U10, U10 to U11, U11 to U12, U12 to U13, U7 to U8, U8 to U9
Connections:
- Q2 pad 2: /DISP+SW/nDig -> +3V3
- Q2 pad 3: +3V3 -> /DISP+SW/nDig
- Q3 pad 2: /DISP+SW/~{nDig} -> +3V3
- Q3 pad 3: +3V3 -> /DISP+SW/~{nDig}
- SW4 pad 1: /DISP+SW/Dig -> /DISP+SW/~{nDig}
- U2 pad 3: /CAN/~{CS} -> /CAN/~{INT}
- U2 pad 7: /CAN/~{INT} -> /CAN/~{CS}
Routing:
- net /DISP+SW/~{nDig}: track 29.3 -> 39.7 mm
- net /CAN/~{INT}: track 51.8 -> 61.7 mm, vias 0 -> 2
- net /DISP+SW/Seg.8: track 118.6 -> 113.7 mm, vias 3 -> 2
- net /DISP+SW/Dig: track 92.3 -> 88.7 mm
- net /CAN/~{CS}: track 83.9 -> 80.4 mm, vias 0 -> 2
- net /DISP+SW/Seg.0: track 80.5 -> 82.4 mm
- net /DISP+SW/nDig: track 39.0 -> 40.4 mm
- net /DISP+SW/Seg.1: track 79.7 -> 80.9 mm
- net /CAN/SCK: track 92.2 -> 93.0 mm
- net /CAN/MOSI: track 95.8 -> 96.6 mm
- net /DISP+SW/Seg.2: track 78.8 -> 79.5 mm
- net /CAN/MISO: track 85.6 -> 86.2 mm
- net GND: vias 476 -> 469

Commit message: Should be final
Parts:
- removed U7: DC56-11CGKWA, Display_7Segment:DA56-11CGKWA
- C33, C34, C39, C40: footprint Capacitor_SMD:C_1206_3216Metric -> Capacitor_SMD:C_0805_2012Metric
- moved C40 0.50 mm to (182.6, 95.7)
- moved C39 0.30 mm to (180.5, 95.7)
