File: hardware.kicad_sch (KiCad schematic)
At the start: 4 parts

Commit message: started routing
Parts:
- removed H101, H102, H103, H104: MountingHole, MountingHole:MountingHole_3.2mm_M3, symbol Mechanical:MountingHole
- added H1, H2, H3, H4: M3, MountingHole:MountingHole_3.2mm_M3_Pad_Via, symbol Mechanical:MountingHole_Pad
Connections:
- new net GND: H1.1, H2.1, H3.1, H4.1
Other:
- sheet CAN ports: added {CAN}, {SPI}; removed {CANH CANL}, {MOSI MISO SCK}
- sheet Connectors ports: added EXT.[0..1], Field24V, IO0.[0..7], IO1.[0..7], IO2.[0..7], {CAN}, {I^{2}C}, {USB}; removed none
- sheet IO Expander ports: added {I^{2}C}; removed {SDA SCL
- sheet MCU ports: added EXT.[0..1], {I^{2}C}, {SPI}, {USB}; removed USB_DM, USB_DP, {MOSI MISO SCK}, {SDA SCL}
- sheet Power ports: added Field24V; removed none
- sheet SD+EEPROM ports: added {I^{2}C}, {SPI}; removed {MOSI MISO SCK}, {SDA SCL}
- title: (none) -> [canbrd] CAN/RS485 IO board

Commit message: Done?
Parts:
- added H3: M3, MountingHole:MountingHole_3.2mm_M3_Pad_Via, symbol Mechanical:MountingHole_Pad
- renumbered H3 to H4, H4 to H5
Connections:
- net GND: now also H3.1
Other:
- sheet SD+EEPROM renamed SD
- sheet SD ports: added none; removed {I^{2}C}
