File: io.kicad_sch (KiCad schematic)
At the start: 30 parts

Commit message: lots changed
Parts:
- removed D10, D11, D12, D13, D6, D7, D8, D9: 3.3V, Diode_SMD:D_SOD-123, symbol Device:D_Zener
- removed JP10, JP13, JP14, JP17, JP18, JP9: LowZ, Jumper:SolderJumper-2_P1.3mm_Open_TrianglePad1.0x1.5mm, symbol Jumper:Jumper_2_Open
- removed JP11, JP12, JP15, JP16, JP19, JP20: Vdiv, Jumper:SolderJumper-2_P1.3mm_Open_TrianglePad1.0x1.5mm, symbol Jumper:Jumper_2_Open
- removed RN3, RN5: 330, Resistor_SMD:R_Array_Convex_4x0603, symbol Device:R_Pack04_Split
- removed RN4, RN6: 10k, Resistor_SMD:R_Array_Convex_4x0603, symbol Device:R_Pack04_Split
- removed RN7, RN8: 1k, Resistor_SMD:R_Array_Convex_4x0603, symbol Device:R_Pack04_Split
- added D10, D11, D12, D13, D14, D15, D16, D17, D6, D7, D8, D9: BAS40-04, Package_TO_SOT_SMD:SOT-23, symbol Device:D_Schottky_Dual_Series_AKC_Split
- added D18: 33V, Diode_SMD:D_SMB, symbol Device:D_TVS
- added Q10, Q11, Q4, Q5, Q6, Q7, Q8, Q9: 2N7002K, Package_TO_SOT_SMD:SOT-23, symbol Transistor_FET:2N7002K
- added R16, R17, R18, R19, R21, R22, R23, R24, R26, R27, R28, R29, R31, R32, R33, R34: 10k, Resistor_SMD:R_0603_1608Metric, symbol Device:R
- added R20, R25, R30, R35: 100, Resistor_SMD:R_0603_1608Metric, symbol Device:R
- JP7, JP8: value Vdiv -> LowZ
Connections:
- net GND: now also D10.1 (A), D11.1 (A), D12.1 (A), D13.1 (A), D14.1 (A), D15.1 (A), D16.1 (A), D17.1 (A), D18.1 (A1), D6.1 (A), D7.1 (A), D8.1 (A), D9.1 (A); no longer JP7.2 (B), JP8.2 (B)
- net RP0: now also Q4.2 (S), R16.2
- net RP1: now also Q6.2 (S), R21.2
- net RP2: now also Q8.2 (S), R26.2
- net RP3: now also Q10.2 (S), R31.2
- net RP4: now also Q5.2 (S), R18.2
- net RP5: now also Q7.2 (S), R23.2
- net RP6: now also Q9.2 (S), R28.2
- net RP7: now also Q11.2 (S), R33.2
- net RP11: now reaches JP8.1 (A)
- net RP11: now also D17.3 (K), R35.1
- net RP9: now reaches JP6.1 (A)
- net RP9: now also D11.3 (K), R25.1
- net RP8: now reaches JP5.1 (A)
- net RP8: now also D8.3 (K), R20.1
- net RP10: now reaches JP7.1 (A)
- net RP10: now also D14.3 (K), R30.1
- net IO0.0 renamed IO8
- net IO8: now also R20.2
- net IO0.4 renamed IO9
- net IO9: now also R25.2
- new net +3V3: D11.2 (K), D14.2 (K), D17.2 (K), D8.2 (K), Q10.1 (G), Q11.1 (G), Q4.1 (G), Q5.1 (G), Q6.1 (G), Q7.1 (G), Q8.1 (G), Q9.1 (G), R16.1, R18.1, R21.1, R23.1, R26.1, R28.1, R31.1, R33.1
- new net IO0: D6.3 (K), Q4.3 (D), R17.2
- new net IO1: D9.3 (K), Q6.3 (D), R22.2
- new net IO10: JP7.2 (B), R30.2
- new net IO11: JP8.2 (B), R35.2
- new net IO2: D12.3 (K), Q8.3 (D), R27.2
- new net IO3: D15.3 (K), Q10.3 (D), R32.2
- new net IO4: D7.3 (K), Q5.3 (D), R19.2
- new net IO5: D10.3 (K), Q7.3 (D), R24.2
- new net IO6: D13.3 (K), Q9.3 (D), R29.2
- new net IO7: D16.3 (K), Q11.3 (D), R34.2
- new net VIO: D10.2 (K), D12.2 (K), D13.2 (K), D15.2 (K), D16.2 (K), D18.2 (A2), D6.2 (K), D7.2 (K), D9.2 (K), R17.1, R19.1, R22.1, R24.1, R27.1, R29.1, R32.1, R34.1
Other:
- note added: "Digital I/O + ADC"
- note added: "Digital I/O only"

Commit message: things changed
Parts:
- removed JP5, JP6, JP7, JP8: LowZ, Jumper:SolderJumper-2_P1.3mm_Open_TrianglePad1.0x1.5mm, symbol Jumper:Jumper_2_Open
- added C29, C30, C31, C32: 10n, Capacitor_SMD:C_0603_1608Metric, symbol Device:C
- added D17: 3.3V, Diode_SMD:D_SOD-123, symbol Device:D_Zener
- added R23, R24, R30, R31, R37, R38, R44, R45: 10, Resistor_SMD:R_0603_1608Metric, symbol Device:R
- renumbered D12 to D10, D13 to D11, D14 to D12, D15 to D13, D16 to D14, D17 to D15, D18 to D16, D6 to D4, D7 to D5, D8 to D6, D9 to D7, D10 to D8, D11 to D9, Q4 to Q12, Q5 to Q13, Q6 to Q14, Q7 to Q15, Q8 to Q16, Q9 to Q17, Q10 to Q18, Q11 to Q19, R16 to R19, R17 to R20, R18 to R21, R19 to R22, R20 to R25, R21 to R26, R22 to R27, R23 to R28, R24 to R29, R25 to R32, R26 to R33, R27 to R34, R28 to R35, R29 to R36, R30 to R39, R31 to R40, R32 to R41, R33 to R42, R34 to R43, R35 to R46
Connections:
- net +3V3: now also D17.1 (K)
- net GND: now also C29.2, C30.2, C31.2, C32.2, D17.2 (A)
- net IO0: now also R23.2; no longer D4.3 (K), Q12.3 (D), R20.2
- net IO1: now also R30.2; no longer D7.3 (K), Q14.3 (D), R27.2
- net IO2: now also R37.2; no longer D10.3 (K), Q16.3 (D), R34.2
- net IO3: now also R44.2; no longer D13.3 (K), Q18.3 (D), R41.2
- net IO4: now also R24.2; no longer D5.3 (K), Q13.3 (D), R22.2
- net IO5: now also R31.2; no longer D8.3 (K), Q15.3 (D), R29.2
- net IO6: now also R38.2; no longer D11.3 (K), Q17.3 (D), R36.2
- net IO7: now also R45.2; no longer D14.3 (K), Q19.3 (D), R43.2
- net RP10: now also C31.1
- net RP11: now also C32.1
- net RP8: now also C29.1
- net RP9: now also C30.1
- new net: D7.3 (K), Q14.3 (D), R27.2, R30.1
- new net: D8.3 (K), Q15.3 (D), R29.2, R31.1
- new net: D11.3 (K), Q17.3 (D), R36.2, R38.1
- new net: D14.3 (K), Q19.3 (D), R43.2, R45.1
- new net: D10.3 (K), Q16.3 (D), R34.2, R37.1
- new net: D4.3 (K), Q12.3 (D), R20.2, R23.1
- new net: D13.3 (K), Q18.3 (D), R41.2, R44.1
- new net: D5.3 (K), Q13.3 (D), R22.2, R24.1
Other:
- moved on the sheet: D10A, D10B, D11A, D11B, D12A, D12B, D13A, D13B, D14A, D14B, D15A, D15B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

Commit message: isolate and other stuff
Parts:
- D17: footprint Diode_SMD:D_SOD-123 -> Diode_SMD:D_MiniMELF
- renumbered C29 to C28, C30 to C29, C31 to C30, C32 to C31, R19 to R23, R20 to R24, R21 to R25, R22 to R26, R23 to R27, R24 to R28, R25 to R29, R26 to R30, R27 to R31, R28 to R32, R29 to R33, R30 to R34, R31 to R35, R32 to R36, R33 to R37, R34 to R38, R35 to R39, R36 to R40, R37 to R41, R38 to R42, R39 to R43, R40 to R44, R41 to R45, R42 to R46, R43 to R47, R44 to R48, R45 to R49, R46 to R50
Other:
- title: [canbrd] CAN/RS485 IO board -> [canbrd] CAN IO board

Commit message: things changed
Parts:
- removed C28, C29, C30, C31: 10n, Capacitor_SMD:C_0603_1608Metric, symbol Device:C
- removed D12, D15, D6, D9: BAS40-04, Package_TO_SOT_SMD:SOT-23, symbol Device:D_Schottky_Dual_Series_AKC_Split
- removed D17: 3.3V, Diode_SMD:D_MiniMELF, symbol Device:D_Zener
- removed R29, R36, R43, R50: 100, Resistor_SMD:R_0603_1608Metric, symbol Device:R
- D9: renamed from D16; value 33V -> 30V
- renumbered D4 to D1, D5 to D2, D7 to D3, D8 to D4, D10 to D5, D11 to D6, D13 to D7, D14 to D8, Q12 to Q1, Q13 to Q2, Q14 to Q3, Q15 to Q4, Q16 to Q5, Q17 to Q6, Q18 to Q7, Q19 to Q8, R23 to R12, R24 to R13, R25 to R14, R26 to R15, R27 to R16, R28 to R17, R30 to R18, R31 to R19, R32 to R20, R33 to R21, R34 to R22, R35 to R23, R37 to R24, R38 to R25, R39 to R26, R40 to R27, R41 to R28, R42 to R29, R44 to R30, R45 to R31, R46 to R32, R47 to R33, R48 to R34, R49 to R35
Connections:
- net +3V3 renamed +3.3V
Other:
- note removed: "Digital I/O + ADC"
