File: io_expander.kicad_sch (KiCad schematic)
At the start: 9 parts, among them J601 UPDI, U601 ATtiny427

Commit message: started routing
Parts:
- removed C605: 10n, symbol Device:C
- C20: renamed from C?; footprint (none) -> Capacitor_SMD:C_0603_1608Metric
- C21: renamed from C606; footprint (none) -> Capacitor_SMD:C_0603_1608Metric
- C22: renamed from C?; value 2.2u -> 1u
- J2: renamed from J601; footprint (none) -> Connector_PinHeader_1.27mm:PinHeader_2x03_P1.27mm_Vertical_SMD
- JP19: renamed from JP?; footprint (none) -> Jumper:SolderJumper-2_P1.3mm_Open_TrianglePad1.0x1.5mm
- R16: renamed from R?; footprint (none) -> Resistor_SMD:R_0603_1608Metric
- gave numbers to parts that had none: 1
- renumbered U601 to U8
Connections:
- net AIN1 renamed AT1.0
- net AIN12 renamed AT2.0
- net AIN13 renamed AT2.1
- net AIN14 renamed AT2.2
- net AIN15 renamed AT2.3
- net AIN2 renamed AT1.1
- net AIN3 renamed AT1.2
- net AIN4 renamed AT1.3
- net AIN6 renamed AT1.4
- net AIN7 renamed AT1.5
- net AIN8 renamed AT1.7
- net AIN9 renamed AT1.6
- net PB2 renamed AT2.4
- net PB3 renamed AT2.5
- net PB6 renamed AT2.6
- net PB7 renamed AT2.7
Other:
- sheet IO Expander Power IO ports: added AT2.[4..7], IO2.[4..7]; removed AT2.4, AT2.5, AT2.6, AT2.7, IO2.4, IO2.5, IO2.6, IO2.7
- sheet IO Expander Protection ports: added AT1.[0..7], AT2.[0..3], IO1.[0..7], IO2.[0..3]; removed AT1.0, AT1.1, AT1.2, AT1.3, AT1.4, AT1.5, AT1.6, AT1.7, AT2.0, AT2.1, AT2.2, AT2.3, IO1.0, IO1.1, IO1.2, IO1.3, IO1.4, IO1.5, IO1.6, IO1.7, IO2.0, IO2.1, IO2.2, IO2.3
- title: (none) -> [canbrd] CAN/RS485 IO board
- moved on the sheet: C22, C23, J2, R16

Commit message: Done?
Parts:
- renumbered C20 to C21, C21 to C22, C22 to C23, C23 to C24, JP19 to JP21, R16 to R15
Connections:
- net AT1.6: now also U8.11 (PB5); no longer U8.12 (PB4)
- net AT1.7: now also U8.12 (PB4); no longer U8.11 (PB5)
- net AT2.4: now also U8.21 (PC4); no longer U8.14 (PB2)
- net AT2.5: now also U8.22 (PC5); no longer U8.13 (PB3)
- net AT_ADDR: now also U8.13 (PB3); no longer U8.22 (PC5)
- net AT_~{INT}: now also U8.14 (PB2); no longer U8.21 (PC4)
Other:
- sheet IO Expander Power IO ports: added AT2.[0..7], IO2.[0..7]; removed AT2.[4..7], IO2.[4..7]
- sheet IO Expander Protection ports: added none; removed AT2.[0..3], IO2.[0..3]
- moved on the sheet: JP21
