File: mcu.kicad_sch (KiCad schematic)
At the start: 28 parts, among them J201 RP_DEBUG, SW201 BOOTSEL, SW202 RESET, U201 W25Q16JVSNIQ, U202 RP2040, Y201 12MHz

Commit message: started routing
Parts:
- removed C211: 100n, Capacitor_SMD:C_0603_1608Metric, symbol Device:C
- C11: renamed from C212; value 2.2u -> 1u
- U2: renamed from U202; footprint Package_DFN_QFN:QFN-56-1EP_7x7mm_P0.4mm_EP5.6x5.6mm_ThermalVias -> RP2040:RP2040-QFN-56
- renumbered C201 to C1, C210 to C10, C213 to C12, C214 to C13, C215 to C14, C216 to C15, C202 to C2, C203 to C3, C204 to C4, C205 to C5, C206 to C6, C207 to C7, C208 to C8, C209 to C9, J201 to J1, R201 to R1, R202 to R2, R203 to R3, R204 to R4, R205 to R5, R206 to R6, SW201 to SW1, SW202 to SW2, U201 to U1, Y201 to Y1
Connections:
- net EXT.0: now reaches U2.31 (GPIO20)
- net EXT.1: now reaches U2.32 (GPIO21)
Other:
- title: (none) -> [canbrd] CAN/RS485 IO board

Commit message: Done?
Connections:
- net CAN_~{CS}: now also U2.3 (GPIO1); no longer U2.16 (GPIO13)
- net CAN_~{INT}: now also U2.7 (GPIO5); no longer U2.13 (GPIO10)
- net CAN_~{RX1}: now also U2.8 (GPIO6); no longer U2.14 (GPIO11)
- net Dig: now also U2.27 (GPIO16); no longer U2.12 (GPIO9)
- net IO_~{INT}: now also U2.28 (GPIO17); no longer U2.30 (GPIO19)
- net MISO: now also U2.6 (GPIO4); no longer U2.15 (GPIO12)
- net MOSI: now also U2.5 (GPIO3); no longer U2.18 (GPIO15)
- net SCK: now also U2.4 (GPIO2); no longer U2.17 (GPIO14)
- net SCL: now also U2.30 (GPIO19); no longer U2.28 (GPIO17)
- net SDA: now also U2.29 (GPIO18); no longer U2.27 (GPIO16)
- net SD_~{CS}: now also U2.2 (GPIO0); no longer U2.29 (GPIO18)
- net Seg.0: now also U2.18 (GPIO15); no longer U2.2 (GPIO0)
- net Seg.1: now also U2.17 (GPIO14); no longer U2.3 (GPIO1)
- net Seg.2: now also U2.16 (GPIO13); no longer U2.4 (GPIO2)
- net Seg.3: now also U2.15 (GPIO12); no longer U2.5 (GPIO3)
- net Seg.4: now also U2.14 (GPIO11); no longer U2.6 (GPIO4)
- net Seg.5: now also U2.13 (GPIO10); no longer U2.7 (GPIO5)
- net Seg.6: now also U2.12 (GPIO9); no longer U2.8 (GPIO6)
- net Seg.7: now also U2.11 (GPIO8); no longer U2.9 (GPIO7)
- net Seg.8: now also U2.9 (GPIO7); no longer U2.11 (GPIO8)
