File: memory.kicad_sch (KiCad schematic)
At the start: 4 parts

Commit message: started routing
Parts:
- removed J?: Micro_SD_Card_Det, symbol Connector:Micro_SD_Card_Det
- removed R?: 1k, symbol Device:R
- added J3: Micro_SD_Card, GTFH081x1YHR:GTFH081x1YHR, symbol Connector:Micro_SD_Card
- C24: renamed from C?; footprint (none) -> Capacitor_SMD:C_0603_1608Metric
- gave numbers to parts that had none: 1
Connections:
- net +3V3: now also J3.4 (VDD)
- net GND: now also J3.6 (VSS), J3.9 (SHIELD)
- net MISO: now also J3.7 (DAT0)
- net MOSI: now also J3.3 (CMD)
- net SCK: now also J3.5 (CLK)
- net SD_~{CS}: now also J3.2 (DAT3/CD)
Other:
- note removed: "TODO"
- title: (none) -> [canbrd] CAN/RS485 IO board
Changed lines of the file:
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@@
 (kicad_sch (version 20211123) (generator eeschema)
   (paper "A4")
-  (junction (at 104.14 119.38) (diameter 0) (color 0 0 0 0)
+  (title_block
+    (title "[canbrd] CAN/RS485 IO board")
+    (date "2022-01-23")
+    (rev "Indev")
   )
   (junction (at 127 53.34) (diameter 0) (color 0 0 0 0)
@@
     (stroke (width 0) (type default) (color 0 0 0 0))
   )
-  (wire (pts (xy 114.3 137.16) (xy 116.84 137.16))
-    (stroke (width 0) (type default) (color 0 0 0 0))
-  )
   (bus (pts (xy 88.9 27.94) (xy 88.9 119.38))
     (stroke (width 0) (type default) (color 0 0 0 0))
@@
     (stroke (width 0) (type default) (color 0 0 0 0))
   )
-  (wire (pts (xy 104.14 119.38) (xy 116.84 119.38))
+  (wire (pts (xy 91.44 119.38) (xy 116.84 119.38))
     (stroke (width 0) (type default) (color 0 0 0 0))
   )
@@
     (stroke (width 0) (type default) (color 0 0 0 0))
   )
-  (wire (pts (xy 162.56 139.7) (xy 160.02 139.7))
-    (stroke (width 0) (type default) (color 0 0 0 0))
-  )
   (bus (pts (xy 88.9 124.46) (xy 88.9 129.54))
     (stroke (width 0) (type default) (color 0 0 0 0))
@@
     (stroke (width 0) (type default) (color 0 0 0 0))
   )
-  (wire (pts (xy 91.44 119.38) (xy 104.14 119.38))
-    (stroke (width 0) (type default) (color 0 0 0 0))
-  )
   (wire (pts (xy 129.54 50.8) (xy 127 50.8))
     (stroke (width 0) (type default) (color 0 0 0 0))
@@
     (stroke (width 0) (type default) (color 0 0 0 0))
   )
-  (wire (pts (xy 106.68 137.16) (xy 104.14 137.16))
-    (stroke (width 0) (type default) (color 0 0 0 0))
-  )
   (wire (pts (xy 127 48.26) (xy 127 50.8))
     (stroke (width 0) (type default) (color 0 0 0 0))
@@
     (stroke (width 0) (type default) (color 0 0 0 0))
   )
-  (wire (pts (xy 104.14 137.16) (xy 104.14 119.38))
-    (stroke (width 0) (type default) (color 0 0 0 0))
-  )
   (wire (pts (xy 127 53.34) (xy 127 58.42))
     (stroke (width 0) (type default) (color 0 0 0 0))
@@
     (stroke (width 0) (type default) (color 0 0 0 0))
   )
-  (text "TODO" (at 177.8 127 0)
-    (effects (font (size 5 5)) (justify left bottom))
+  (wire (pts (xy 160.02 139.7) (xy 162.56 139.7))
+    (stroke (width 0) (type default) (color 0 0 0 0))
   )
   (label "SDA" (at 149.86 48.26 0)
@@
     (effects (font (size 1 1)) (justify right))
   )
-  (hierarchical_label "{MOSI MISO SCK}" (shape bidirectional) (at 38.1 27.94 180)
+  (hierarchical_label "{SPI}" (shape bidirectional) (at 38.1 27.94 180)
     (effects (font (size 1 1)) (justify right))
   )
-  (hierarchical_label "{SDA SCL}" (shape bidirectional) (at 38.1 22.86 180)
+  (hierarchical_label "{I^{2}C}" (shape bidirectional) (at 38.1 22.86 180)
     (effects (font (size 1 1)) (justify right))
   )
   (symbol (lib_id "Device:C") (at 114.3 50.8 0) (unit 1)
     (in_bom yes) (on_board yes) (fields_autoplaced)
-    (property "Reference" "C?" (id 0) (at 117.221 49.8915 0)
+    (property "Reference" "C24" (id 0) (at 117.221 49.8915 0)
       (effects (font (size 1.27 1.27)) (justify left))
     )
@@
       (effects (font (size 1.27 1.27)) (justify left))
     )
-    (property "Footprint" "" (id 2) (at 115.2652 54.61 0)
+    (property "Footprint" "Capacitor_SMD:C_0603_1608Metric" (id 2) (at 115.2652 54.61 0)
       (effects (font (size 1.27 1.27)) hide)
     )
@@
   (symbol (lib_id "power:+3.3V") (at 139.7 43.18 0) (unit 1)
     (in_bom yes) (on_board yes)
-    (property "Reference" "#PWR?" (id 0) (at 139.7 46.99 0)
+    (property "Reference" "#PWR0114" (id 0) (at 139.7 46.99 0)
       (effects (font (size 1.27 1.27)) hide)
     )
@@
   (symbol (lib_id "power:GND") (at 162.56 143.51 0) (unit 1)
     (in_bom yes) (on_board yes)
-    (property "Reference" "#PWR?" (id 0) (at 162.56 149.86 0)
+    (property "Reference" "#PWR0121" (id 0) (at 162.56 149.86 0)
       (effects (font (size 1.27 1.27)) hide)
     )
@@
   (symbol (lib_id "power:+3.3V") (at 114.3 46.99 0) (unit 1)
     (in_bom yes) (on_board yes)
-    (property "Reference" "#PWR?" (id 0) (at 114.3 50.8 0)
+    (property "Reference" "#PWR0115" (id 0) (at 114.3 50.8 0)
       (effects (font (size 1.27 1.27)) hide)
     )
@@
   (symbol (lib_id "power:+3.3V") (at 101.6 110.49 0) (unit 1)
     (in_bom yes) (on_board yes)
-    (property "Reference" "#PWR?" (id 0) (at 101.6 114.3 0)
+    (property "Reference" "#PWR0119" (id 0) (at 101.6 114.3 0)
       (effects (font (size 1.27 1.27)) hide)
     )
@@
   (symbol (lib_id "power:GND") (at 101.6 143.51 0) (unit 1)
     (in_bom yes) (on_board yes)
-    (property "Reference" "#PWR?" (id 0) (at 101.6 149.86 0)
+    (property "Reference" "#PWR0120" (id 0) (at 101.6 149.86 0)
       (effects (font (size 1.27 1.27)) hide)
     )
@@
   (symbol (lib_id "power:GND") (at 114.3 54.61 0) (unit 1)
     (in_bom yes) (on_board yes)
-    (property "Reference" "#PWR?" (id 0) (at 114.3 60.96 0)
+    (property "Reference" "#PWR0116" (id 0) (at 114.3 60.96 0)
       (effects (font (size 1.27 1.27)) hide)
     )
@@
   (symbol (lib_id "Memory_EEPROM:M24C02-WMN") (at 139.7 50.8 0) (unit 1)
     (in_bom yes) (on_board yes)
-    (property "Reference" "U?" (id 0) (at 144.78 41.91 0)
+    (property "Reference" "U9" (id 0) (at 144.78 41.91 0)
       (effects (font (size 1.27 1.27)) (justify left))
     )
@@
   (symbol (lib_id "power:GND") (at 139.7 58.42 0) (unit 1)
     (in_bom yes) (on_board yes)
-    (property "Reference" "#PWR?" (id 0) (at 139.7 64.77 0)
+    (property "Reference" "#PWR0118" (id 0) (at 139.7 64.77 0)
       (effects (font (size 1.27 1.27)) hide)
     )
@@
     (pin "1")
   )
-  (symbol (lib_id "Device:R") (at 110.49 137.16 90) (unit 1)
-    (in_bom yes) (on_board yes)
-    (property "Reference" "R?" (id 0) (at 110.49 134.62 90))
-    (property "Value" "1k" (id 1) (at 110.49 137.16 90))
-    (property "Footprint" "" (id 2) (at 110.49 138.938 90)
-      (effects (font (size 1.27 1.27)) hide)
-    )
-    (property "Datasheet" "~" (id 3) (at 110.49 137.16 0)
-      (effects (font (size 1.27 1.27)) hide)
-    )
-    (pin "1")
-    (pin "2")
-  )
-  (symbol (lib_id "Connector:Micro_SD_Card_Det") (at 139.7 127 0) (unit 1)
+  (symbol (lib_id "Connector:Micro_SD_Card") (at 139.7 124.46 0) (unit 1)
     (in_bom yes) (on_board yes) (fields_autoplaced)
-    (property "Reference" "J?" (id 0) (at 140.335 106.5235 0))
-    (property "Value" "Micro_SD_Card_Det" (id 1) (at 140.335 109.2986 0))
-    (property "Footprint" "" (id 2) (at 191.77 109.22 0)
-      (effects (font (size 1.27 1.27)) hide)
-    )
-    (property "Datasheet" "https://www.hirose.com/product/en/download_file/key_name/DM3/category/Catalog/doc_file_id/49662/?file_category_id=4&item_id=195&is_series=1" (id 3) (at 139.7 124.46 0)
-      (effects (font (size 1.27 1.27)) hide)
-    )
-    (pin "1")
-    (pin "10")
-    (pin "11")
+    (property "Reference" "J3" (id 0) (at 140.335 105.41 0))
+    (property "Value" "Micro_SD_Card" (id 1) (at 140.335 107.95 0))
+    (property "Footprint" "GTFH081x1YHR:GTFH081x1YHR" (id 2) (at 168.91 116.84 0)
+      (effects (font (size 1.27 1.27)) hide)
+    )
+    (property "Datasheet" "http://katalog.we-online.de/em/datasheet/693072010801.pdf" (id 3) (at 139.7 124.46 0)
+      (effects (font (size 1.27 1.27)) hide)
+    )
+    (pin "1")
     (pin "2")
     (pin "3")
@@
   (symbol (lib_id "power:GND") (at 127 58.42 0) (unit 1)
     (in_bom yes) (on_board yes)
-    (property "Reference" "#PWR?" (id 0) (at 127 64.77 0)
-      (effects (font (size 1.27 1.27)) hide)
-    )
+    (property "Reference" "#PWR0117" (id 0) (at 127 64.77 0)
+      (effects (font (size 1.27 1.27)) hide)
+    )

Commit message: Done?
Parts:
- removed C24: 100n, Capacitor_SMD:C_0603_1608Metric, symbol Device:C
- removed U9: M24C04-WMN, Package_SO:SOIC-8_3.9x4.9mm_P1.27mm, symbol Memory_EEPROM:M24C02-WMN
Connections:
- no-connect marks 3 -> 2
Changed lines of the file:
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@@
     (rev "Indev")
   )
-  (junction (at 127 53.34) (diameter 0) (color 0 0 0 0)
-  )
-  (junction (at 127 50.8) (diameter 0) (color 0 0 0 0)
-  )
   (no_connect (at 116.84 134.62))
-  (no_connect (at 149.86 53.34))
   (no_connect (at 116.84 116.84))
-  (bus_entry (at 165.1 48.26) (size -2.54 2.54)
-    (stroke (width 0) (type default) (color 0 0 0 0))
-  )
-  (bus_entry (at 165.1 45.72) (size -2.54 2.54)
-    (stroke (width 0) (type default) (color 0 0 0 0))
-  )
   (bus_entry (at 88.9 119.38) (size 2.54 2.54)
     (stroke (width 0) (type default) (color 0 0 0 0))
@@
   )
   (bus_entry (at 88.9 129.54) (size 2.54 2.54)
-    (stroke (width 0) (type default) (color 0 0 0 0))
-  )
-  (bus (pts (xy 38.1 22.86) (xy 165.1 22.86))
     (stroke (width 0) (type default) (color 0 0 0 0))
   )
@@
     (stroke (width 0) (type default) (color 0 0 0 0))
   )
-  (wire (pts (xy 129.54 53.34) (xy 127 53.34))
-    (stroke (width 0) (type default) (color 0 0 0 0))
-  )
-  (wire (pts (xy 149.86 48.26) (xy 162.56 48.26))
-    (stroke (width 0) (type default) (color 0 0 0 0))
-  )
-  (wire (pts (xy 127 50.8) (xy 127 53.34))
-    (stroke (width 0) (type default) (color 0 0 0 0))
-  )
-  (bus (pts (xy 165.1 45.72) (xy 165.1 48.26))
-    (stroke (width 0) (type default) (color 0 0 0 0))
-  )
   (bus (pts (xy 88.9 124.46) (xy 88.9 129.54))
     (stroke (width 0) (type default) (color 0 0 0 0))
@@
     (stroke (width 0) (type default) (color 0 0 0 0))
   )
-  (wire (pts (xy 129.54 48.26) (xy 127 48.26))
-    (stroke (width 0) (type default) (color 0 0 0 0))
-  )
-  (wire (pts (xy 129.54 50.8) (xy 127 50.8))
-    (stroke (width 0) (type default) (color 0 0 0 0))
-  )
   (wire (pts (xy 91.44 127) (xy 116.84 127))
     (stroke (width 0) (type default) (color 0 0 0 0))
   )
-  (wire (pts (xy 127 48.26) (xy 127 50.8))
-    (stroke (width 0) (type default) (color 0 0 0 0))
-  )
   (wire (pts (xy 101.6 124.46) (xy 101.6 110.49))
-    (stroke (width 0) (type default) (color 0 0 0 0))
-  )
-  (wire (pts (xy 149.86 50.8) (xy 162.56 50.8))
     (stroke (width 0) (type default) (color 0 0 0 0))
   )
@@
     (stroke (width 0) (type default) (color 0 0 0 0))
   )
-  (wire (pts (xy 127 53.34) (xy 127 58.42))
-    (stroke (width 0) (type default) (color 0 0 0 0))
-  )
-  (bus (pts (xy 165.1 22.86) (xy 165.1 45.72))
-    (stroke (width 0) (type default) (color 0 0 0 0))
-  )
   (wire (pts (xy 91.44 132.08) (xy 116.84 132.08))
     (stroke (width 0) (type default) (color 0 0 0 0))
@@
   (wire (pts (xy 160.02 139.7) (xy 162.56 139.7))
     (stroke (width 0) (type default) (color 0 0 0 0))
-  )
-  (label "SDA" (at 149.86 48.26 0)
-    (effects (font (size 1.27 1.27)) (justify left bottom))
   )
   (label "SCK" (at 111.76 127 0)
@@
     (effects (font (size 1.27 1.27)) (justify left bottom))
   )
-  (label "SCL" (at 149.86 50.8 0)
-    (effects (font (size 1.27 1.27)) (justify left bottom))
-  )
   (hierarchical_label "SD_~{CS}" (shape input) (at 38.1 25.4 180)
     (effects (font (size 1 1)) (justify right))
@@
     (effects (font (size 1 1)) (justify right))
   )
-  (hierarchical_label "{I^{2}C}" (shape bidirectional) (at 38.1 22.86 180)
-    (effects (font (size 1 1)) (justify right))
-  )
-  (symbol (lib_id "Device:C") (at 114.3 50.8 0) (unit 1)
-    (in_bom yes) (on_board yes) (fields_autoplaced)
-    (property "Reference" "C24" (id 0) (at 117.221 49.8915 0)
-      (effects (font (size 1.27 1.27)) (justify left))
-    )
-    (property "Value" "100n" (id 1) (at 117.221 52.6666 0)
-      (effects (font (size 1.27 1.27)) (justify left))
-    )
-    (property "Footprint" "Capacitor_SMD:C_0603_1608Metric" (id 2) (at 115.2652 54.61 0)
-      (effects (font (size 1.27 1.27)) hide)
-    )
-    (property "Datasheet" "~" (id 3) (at 114.3 50.8 0)
-      (effects (font (size 1.27 1.27)) hide)
-    )
-    (pin "1")
-    (pin "2")
-  )
-  (symbol (lib_id "power:+3.3V") (at 139.7 43.18 0) (unit 1)
-    (in_bom yes) (on_board yes)
-    (property "Reference" "#PWR0114" (id 0) (at 139.7 46.99 0)
-      (effects (font (size 1.27 1.27)) hide)
-    )
-    (property "Value" "+3.3V" (id 1) (at 139.7 39.37 0))
-    (property "Footprint" "" (id 2) (at 139.7 43.18 0)
-      (effects (font (size 1.27 1.27)) hide)
-    )
-    (property "Datasheet" "" (id 3) (at 139.7 43.18 0)
-      (effects (font (size 1.27 1.27)) hide)
-    )
-    (pin "1")
-  )
   (symbol (lib_id "power:GND") (at 162.56 143.51 0) (unit 1)
     (in_bom yes) (on_board yes)
-    (property "Reference" "#PWR0121" (id 0) (at 162.56 149.86 0)
+    (property "Reference" "#PWR0103" (id 0) (at 162.56 149.86 0)
       (effects (font (size 1.27 1.27)) hide)
     )
@@
     (pin "1")
   )
-  (symbol (lib_id "power:+3.3V") (at 114.3 46.99 0) (unit 1)
-    (in_bom yes) (on_board yes)
-    (property "Reference" "#PWR0115" (id 0) (at 114.3 50.8 0)
-      (effects (font (size 1.27 1.27)) hide)
-    )
-    (property "Value" "+3.3V" (id 1) (at 114.3 43.18 0))
-    (property "Footprint" "" (id 2) (at 114.3 46.99 0)
-      (effects (font (size 1.27 1.27)) hide)
-    )
-    (property "Datasheet" "" (id 3) (at 114.3 46.99 0)
-      (effects (font (size 1.27 1.27)) hide)
-    )
-    (pin "1")
-  )
   (symbol (lib_id "power:+3.3V") (at 101.6 110.49 0) (unit 1)
     (in_bom yes) (on_board yes)
-    (property "Reference" "#PWR0119" (id 0) (at 101.6 114.3 0)
+    (property "Reference" "#PWR0101" (id 0) (at 101.6 114.3 0)
       (effects (font (size 1.27 1.27)) hide)
     )
@@
   (symbol (lib_id "power:GND") (at 101.6 143.51 0) (unit 1)
     (in_bom yes) (on_board yes)
-    (property "Reference" "#PWR0120" (id 0) (at 101.6 149.86 0)
+    (property "Reference" "#PWR0102" (id 0) (at 101.6 149.86 0)
       (effects (font (size 1.27 1.27)) hide)
     )
@@
     )
     (property "Datasheet" "" (id 3) (at 101.6 143.51 0)
-      (effects (font (size 1.27 1.27)) hide)
-    )
-    (pin "1")
-  )
-  (symbol (lib_id "power:GND") (at 114.3 54.61 0) (unit 1)
-    (in_bom yes) (on_board yes)
-    (property "Reference" "#PWR0116" (id 0) (at 114.3 60.96 0)
-      (effects (font (size 1.27 1.27)) hide)
-    )
-    (property "Value" "GND" (id 1) (at 114.3 58.42 0))
-    (property "Footprint" "" (id 2) (at 114.3 54.61 0)
-      (effects (font (size 1.27 1.27)) hide)
-    )
-    (property "Datasheet" "" (id 3) (at 114.3 54.61 0)
-      (effects (font (size 1.27 1.27)) hide)
-    )
-    (pin "1")
-  )
-  (symbol (lib_id "Memory_EEPROM:M24C02-WMN") (at 139.7 50.8 0) (unit 1)
-    (in_bom yes) (on_board yes)
-    (property "Reference" "U9" (id 0) (at 144.78 41.91 0)
-      (effects (font (size 1.27 1.27)) (justify left))
-    )
-    (property "Value" "M24C04-WMN" (id 1) (at 144.78 44.45 0)
-      (effects (font (size 1.27 1.27)) (justify left))
-    )
-    (property "Footprint" "Package_SO:SOIC-8_3.9x4.9mm_P1.27mm" (id 2) (at 139.7 41.91 0)
-      (effects (font (size 1.27 1.27)) hide)
-    )
-    (property "Datasheet" "http://www.st.com/content/ccc/resource/technical/document/datasheet/b0/d8/50/40/5a/85/49/6f/DM00071904.pdf/files/DM00071904.pdf/jcr:content/translations/en.DM00071904.pdf" (id 3) (at 140.97 63.5 0)
-      (effects (font (size 1.27 1.27)) hide)
-    )
-    (pin "1")
-    (pin "2")
-    (pin "3")
-    (pin "4")
-    (pin "5")
-    (pin "6")
-    (pin "7")
-    (pin "8")
-  )
-  (symbol (lib_id "power:GND") (at 139.7 58.42 0) (unit 1)
-    (in_bom yes) (on_board yes)
-    (property "Reference" "#PWR0118" (id 0) (at 139.7 64.77 0)
-      (effects (font (size 1.27 1.27)) hide)
-    )
-    (property "Value" "GND" (id 1) (at 139.7 62.23 0))
-    (property "Footprint" "" (id 2) (at 139.7 58.42 0)
-      (effects (font (size 1.27 1.27)) hide)
-    )
-    (property "Datasheet" "" (id 3) (at 139.7 58.42 0)
       (effects (font (size 1.27 1.27)) hide)
     )
@@
     (pin "9")
   )
-  (symbol (lib_id "power:GND") (at 127 58.42 0) (unit 1)
-    (in_bom yes) (on_board yes)
-    (property "Reference" "#PWR0117" (id 0) (at 127 64.77 0)
-      (effects (font (size 1.27 1.27)) hide)
-    )
-    (property "Value" "GND" (id 1) (at 127 62.23 0))
-    (property "Footprint" "" (id 2) (at 127 58.42 0)
-      (effects (font (size 1.27 1.27)) hide)
-    )
-    (property "Datasheet" "" (id 3) (at 127 58.42 0)
-      (effects (font (size 1.27 1.27)) hide)
-    )
-    (pin "1")
-  )
 )
