File: memory.kicad_sch (KiCad schematic)
At the start: 1 part, among them J3 Micro_SD_Card

Commit message: lots changed
Parts:
- renumbered J3 to J2
Changed lines of the file:
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@@
   (title_block
     (title "[canbrd] CAN/RS485 IO board")
-    (date "2022-03-18")
-    (rev "1.1")
+    (date "2022-04-03")
+    (rev "2.0")
   )
   (no_connect (at 116.84 134.62))
@@
   (symbol (lib_id "power:GND") (at 162.56 143.51 0) (unit 1)
     (in_bom yes) (on_board yes)
-    (property "Reference" "#PWR0105" (id 0) (at 162.56 149.86 0)
+    (property "Reference" "#PWR0115" (id 0) (at 162.56 149.86 0)
       (effects (font (size 1.27 1.27)) hide)
     )
@@
   (symbol (lib_id "power:+3.3V") (at 101.6 110.49 0) (unit 1)
     (in_bom yes) (on_board yes)
-    (property "Reference" "#PWR0103" (id 0) (at 101.6 114.3 0)
+    (property "Reference" "#PWR0113" (id 0) (at 101.6 114.3 0)
       (effects (font (size 1.27 1.27)) hide)
     )
@@
   (symbol (lib_id "power:GND") (at 101.6 143.51 0) (unit 1)
     (in_bom yes) (on_board yes)
-    (property "Reference" "#PWR0104" (id 0) (at 101.6 149.86 0)
+    (property "Reference" "#PWR0114" (id 0) (at 101.6 149.86 0)
       (effects (font (size 1.27 1.27)) hide)
     )
@@
   (symbol (lib_id "Connector:Micro_SD_Card") (at 139.7 124.46 0) (unit 1)
     (in_bom yes) (on_board yes) (fields_autoplaced)
-    (property "Reference" "J3" (id 0) (at 140.335 105.41 0))
+    (property "Reference" "J2" (id 0) (at 140.335 105.41 0))
     (property "Value" "Micro_SD_Card" (id 1) (at 140.335 107.95 0))
     (property "Footprint" "GTFH081x1YHR:GTFH081x1YHR" (id 2) (at 168.91 116.84 0)

Commit message: things changed
Parts:
- added R47: 130, Resistor_SMD:R_0603_1608Metric, symbol Device:R
Connections:
- net MISO: now also R47.1; no longer J2.7 (DAT0)
- new net xMISO: J2.7 (DAT0), R47.2
Changed lines of the file:
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@@
   (title_block
     (title "[canbrd] CAN/RS485 IO board")
-    (date "2022-04-03")
-    (rev "2.0")
+    (date "2022-05-22")
+    (rev "2.1")
   )
   (no_connect (at 116.84 134.62))
@@
     (stroke (width 0) (type default) (color 0 0 0 0))
   )
+  (wire (pts (xy 109.22 132.08) (xy 116.84 132.08))
+    (stroke (width 0) (type default) (color 0 0 0 0))
+  )
   (bus (pts (xy 88.9 124.46) (xy 88.9 129.54))
     (stroke (width 0) (type default) (color 0 0 0 0))
   )
-  (wire (pts (xy 101.6 129.54) (xy 101.6 143.51))
+  (wire (pts (xy 97.79 129.54) (xy 97.79 143.51))
     (stroke (width 0) (type default) (color 0 0 0 0))
   )
-  (wire (pts (xy 116.84 124.46) (xy 101.6 124.46))
+  (wire (pts (xy 116.84 124.46) (xy 97.79 124.46))
     (stroke (width 0) (type default) (color 0 0 0 0))
   )
@@
     (stroke (width 0) (type default) (color 0 0 0 0))
   )
-  (wire (pts (xy 101.6 124.46) (xy 101.6 110.49))
+  (wire (pts (xy 97.79 124.46) (xy 97.79 110.49))
     (stroke (width 0) (type default) (color 0 0 0 0))
   )
@@
     (stroke (width 0) (type default) (color 0 0 0 0))
   )
-  (wire (pts (xy 91.44 132.08) (xy 116.84 132.08))
+  (wire (pts (xy 91.44 132.08) (xy 101.6 132.08))
     (stroke (width 0) (type default) (color 0 0 0 0))
   )
-  (wire (pts (xy 116.84 129.54) (xy 101.6 129.54))
+  (wire (pts (xy 116.84 129.54) (xy 97.79 129.54))
     (stroke (width 0) (type default) (color 0 0 0 0))
   )
@@
     (effects (font (size 1.27 1.27)) (justify left bottom))
   )
-  (label "MISO" (at 111.76 132.08 0)
+  (label "MISO" (at 91.44 132.08 0)
+    (effects (font (size 1.27 1.27)) (justify left bottom))
+  )
+  (label "xMISO" (at 110.49 132.08 0)
     (effects (font (size 1.27 1.27)) (justify left bottom))
   )
@@
   (symbol (lib_id "power:GND") (at 162.56 143.51 0) (unit 1)
     (in_bom yes) (on_board yes)
-    (property "Reference" "#PWR0115" (id 0) (at 162.56 149.86 0)
+    (property "Reference" "#PWR0132" (id 0) (at 162.56 149.86 0)
       (effects (font (size 1.27 1.27)) hide)
     )
@@
     (pin "1")
   )
-  (symbol (lib_id "power:+3.3V") (at 101.6 110.49 0) (unit 1)
+  (symbol (lib_id "power:+3.3V") (at 97.79 110.49 0) (unit 1)
     (in_bom yes) (on_board yes)
-    (property "Reference" "#PWR0113" (id 0) (at 101.6 114.3 0)
+    (property "Reference" "#PWR0130" (id 0) (at 97.79 114.3 0)
       (effects (font (size 1.27 1.27)) hide)
     )
-    (property "Value" "+3.3V" (id 1) (at 101.6 106.68 0))
-    (property "Footprint" "" (id 2) (at 101.6 110.49 0)
+    (property "Value" "+3.3V" (id 1) (at 97.79 106.68 0))
+    (property "Footprint" "" (id 2) (at 97.79 110.49 0)
       (effects (font (size 1.27 1.27)) hide)
     )
-    (property "Datasheet" "" (id 3) (at 101.6 110.49 0)
+    (property "Datasheet" "" (id 3) (at 97.79 110.49 0)
       (effects (font (size 1.27 1.27)) hide)
     )
     (pin "1")
   )
-  (symbol (lib_id "power:GND") (at 101.6 143.51 0) (unit 1)
+  (symbol (lib_id "power:GND") (at 97.79 143.51 0) (unit 1)
     (in_bom yes) (on_board yes)
-    (property "Reference" "#PWR0114" (id 0) (at 101.6 149.86 0)
+    (property "Reference" "#PWR0131" (id 0) (at 97.79 149.86 0)
       (effects (font (size 1.27 1.27)) hide)
     )
-    (property "Value" "GND" (id 1) (at 101.6 147.32 0))
-    (property "Footprint" "" (id 2) (at 101.6 143.51 0)
+    (property "Value" "GND" (id 1) (at 97.79 147.32 0))
+    (property "Footprint" "" (id 2) (at 97.79 143.51 0)
       (effects (font (size 1.27 1.27)) hide)
     )
-    (property "Datasheet" "" (id 3) (at 101.6 143.51 0)
+    (property "Datasheet" "" (id 3) (at 97.79 143.51 0)
       (effects (font (size 1.27 1.27)) hide)
     )
     (pin "1")
   )
+  (symbol (lib_id "Device:R") (at 105.41 132.08 90) (unit 1)
+    (in_bom yes) (on_board yes)
+    (property "Reference" "R47" (id 0) (at 101.6 132.08 90)
+      (effects (font (size 1 1)) (justify left top))
+    )
+    (property "Value" "130" (id 1) (at 105.41 132.08 90))
+    (property "Footprint" "Resistor_SMD:R_0603_1608Metric" (id 2) (at 105.41 133.858 90)
+      (effects (font (size 1.27 1.27)) hide)
+    )
+    (property "Datasheet" "~" (id 3) (at 105.41 132.08 0)
+      (effects (font (size 1.27 1.27)) hide)
+    )
+    (pin "1")
+    (pin "2")
+  )
   (symbol (lib_id "Connector:Micro_SD_Card") (at 139.7 124.46 0) (unit 1)

Commit message: isolate and other stuff
Parts:
- R52: renamed from R47; value 130 -> 100
Other:
- title: [canbrd] CAN/RS485 IO board -> [canbrd] CAN IO board
Changed lines of the file:
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@@
   (paper "A4")
   (title_block
-    (title "[canbrd] CAN/RS485 IO board")
-    (date "2022-05-22")
-    (rev "2.1")
+    (title "[canbrd] CAN IO board")
+    (date "2022-05-30")
+    (rev "2.2")
   )
   (no_connect (at 116.84 134.62))
@@
   (symbol (lib_id "power:GND") (at 162.56 143.51 0) (unit 1)
     (in_bom yes) (on_board yes)
-    (property "Reference" "#PWR0132" (id 0) (at 162.56 149.86 0)
+    (property "Reference" "#PWR0135" (id 0) (at 162.56 149.86 0)
       (effects (font (size 1.27 1.27)) hide)
     )
@@
   (symbol (lib_id "power:+3.3V") (at 97.79 110.49 0) (unit 1)
     (in_bom yes) (on_board yes)
-    (property "Reference" "#PWR0130" (id 0) (at 97.79 114.3 0)
+    (property "Reference" "#PWR0133" (id 0) (at 97.79 114.3 0)
       (effects (font (size 1.27 1.27)) hide)
     )
@@
   (symbol (lib_id "power:GND") (at 97.79 143.51 0) (unit 1)
     (in_bom yes) (on_board yes)
-    (property "Reference" "#PWR0131" (id 0) (at 97.79 149.86 0)
+    (property "Reference" "#PWR0134" (id 0) (at 97.79 149.86 0)
       (effects (font (size 1.27 1.27)) hide)
     )
@@
   (symbol (lib_id "Device:R") (at 105.41 132.08 90) (unit 1)
     (in_bom yes) (on_board yes)
-    (property "Reference" "R47" (id 0) (at 101.6 132.08 90)
+    (property "Reference" "R52" (id 0) (at 101.6 132.08 90)
       (effects (font (size 1 1)) (justify left top))
     )
-    (property "Value" "130" (id 1) (at 105.41 132.08 90))
+    (property "Value" "100" (id 1) (at 105.41 132.08 90))
     (property "Footprint" "Resistor_SMD:R_0603_1608Metric" (id 2) (at 105.41 133.858 90)
       (effects (font (size 1.27 1.27)) hide)

Commit message: things changed
Parts:
- added C30: 100n, Capacitor_SMD:C_0603_1608Metric, symbol Device:C
- added U6: AT24CS01-STUM, Package_TO_SOT_SMD:SOT-23-5, symbol Memory_EEPROM:AT24CS01-STUM
- renumbered R52 to R47
Connections:
- net GND: now also C30.2, U6.2 (GND), U6.5 (WP)
- net +3V3 renamed +3.3V
- net +3.3V: now also C30.1, U6.4 (VCC)
- new net SCL: U6.1 (SCL)
- new net SDA: U6.3 (SDA)
Changed lines of the file:
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@@
   (title_block
     (title "[canbrd] CAN IO board")
-    (date "2022-05-30")
-    (rev "2.2")
+    (date "2022-10-08")
+    (rev "3.2")
   )
   (no_connect (at 116.84 134.62))
   (no_connect (at 116.84 116.84))
+  (bus_entry (at 93.98 71.12) (size 2.54 2.54)
+    (stroke (width 0) (type default) (color 0 0 0 0))
+  )
   (bus_entry (at 88.9 119.38) (size 2.54 2.54)
     (stroke (width 0) (type default) (color 0 0 0 0))
   )
+  (bus_entry (at 93.98 73.66) (size 2.54 2.54)
+    (stroke (width 0) (type default) (color 0 0 0 0))
+  )
   (bus_entry (at 88.9 124.46) (size 2.54 2.54)
     (stroke (width 0) (type default) (color 0 0 0 0))
@@
     (stroke (width 0) (type default) (color 0 0 0 0))
   )
+  (wire (pts (xy 96.52 73.66) (xy 129.54 73.66))
+    (stroke (width 0) (type default) (color 0 0 0 0))
+  )
   (wire (pts (xy 38.1 25.4) (xy 91.44 25.4))
     (stroke (width 0) (type default) (color 0 0 0 0))
   )
+  (wire (pts (xy 127 78.74) (xy 127 83.82))
+    (stroke (width 0) (type default) (color 0 0 0 0))
+  )
   (bus (pts (xy 88.9 27.94) (xy 88.9 119.38))
     (stroke (width 0) (type default) (color 0 0 0 0))
   )
+  (bus (pts (xy 93.98 22.86) (xy 93.98 71.12))
+    (stroke (width 0) (type default) (color 0 0 0 0))
+  )
+  (wire (pts (xy 129.54 78.74) (xy 127 78.74))
+    (stroke (width 0) (type default) (color 0 0 0 0))
+  )
   (wire (pts (xy 162.56 143.51) (xy 162.56 139.7))
     (stroke (width 0) (type default) (color 0 0 0 0))
@@
     (stroke (width 0) (type default) (color 0 0 0 0))
   )
+  (bus (pts (xy 38.1 22.86) (xy 93.98 22.86))
+    (stroke (width 0) (type default) (color 0 0 0 0))
+  )
   (bus (pts (xy 38.1 27.94) (xy 88.9 27.94))
     (stroke (width 0) (type default) (color 0 0 0 0))
@@
     (stroke (width 0) (type default) (color 0 0 0 0))
   )
+  (bus (pts (xy 93.98 71.12) (xy 93.98 73.66))
+    (stroke (width 0) (type default) (color 0 0 0 0))
+  )
   (wire (pts (xy 91.44 132.08) (xy 101.6 132.08))
     (stroke (width 0) (type default) (color 0 0 0 0))
@@
     (stroke (width 0) (type default) (color 0 0 0 0))
   )
+  (wire (pts (xy 96.52 76.2) (xy 129.54 76.2))
+    (stroke (width 0) (type default) (color 0 0 0 0))
+  )
   (wire (pts (xy 160.02 139.7) (xy 162.56 139.7))
     (stroke (width 0) (type default) (color 0 0 0 0))
@@
   )
   (label "xMISO" (at 110.49 132.08 0)
+    (effects (font (size 1.27 1.27)) (justify left bottom))
+  )
+  (label "SDA" (at 123.19 73.66 0)
+    (effects (font (size 1.27 1.27)) (justify left bottom))
+  )
+  (label "SCL" (at 123.19 76.2 0)
     (effects (font (size 1.27 1.27)) (justify left bottom))
   )
@@
     (effects (font (size 1 1)) (justify right))
   )
+  (hierarchical_label "{I^{2}C}" (shape bidirectional) (at 38.1 22.86 180)
+    (effects (font (size 1 1)) (justify right))
+  )
+  (symbol (lib_id "Device:C") (at 171.45 76.2 0) (unit 1)
+    (in_bom yes) (on_board yes) (fields_autoplaced)
+    (property "Reference" "C30" (id 0) (at 174.371 75.3653 0)
+      (effects (font (size 1.27 1.27)) (justify left))
+    )
+    (property "Value" "100n" (id 1) (at 174.371 77.9022 0)
+      (effects (font (size 1.27 1.27)) (justify left))
+    )
+    (property "Footprint" "Capacitor_SMD:C_0603_1608Metric" (id 2) (at 172.4152 80.01 0)
+      (effects (font (size 1.27 1.27)) hide)
+    )
+    (property "Datasheet" "~" (id 3) (at 171.45 76.2 0)
+      (effects (font (size 1.27 1.27)) hide)
+    )
+    (pin "1")
+    (pin "2")
+  )
   (symbol (lib_id "power:GND") (at 162.56 143.51 0) (unit 1)
     (in_bom yes) (on_board yes)
-    (property "Reference" "#PWR0135" (id 0) (at 162.56 149.86 0)
+    (property "Reference" "#PWR0128" (id 0) (at 162.56 149.86 0)
       (effects (font (size 1.27 1.27)) hide)
     )
@@
   (symbol (lib_id "power:+3.3V") (at 97.79 110.49 0) (unit 1)
     (in_bom yes) (on_board yes)
-    (property "Reference" "#PWR0133" (id 0) (at 97.79 114.3 0)
+    (property "Reference" "#PWR0126" (id 0) (at 97.79 114.3 0)
       (effects (font (size 1.27 1.27)) hide)
     )
@@
     (pin "1")
   )
+  (symbol (lib_id "power:GND") (at 171.45 80.01 0) (unit 1)
+    (in_bom yes) (on_board yes) (fields_autoplaced)
+    (property "Reference" "#PWR0123" (id 0) (at 171.45 86.36 0)
+      (effects (font (size 1.27 1.27)) hide)
+    )
+    (property "Value" "GND" (id 1) (at 171.45 84.4534 0))
+    (property "Footprint" "" (id 2) (at 171.45 80.01 0)
+      (effects (font (size 1.27 1.27)) hide)
+    )
+    (property "Datasheet" "" (id 3) (at 171.45 80.01 0)
+      (effects (font (size 1.27 1.27)) hide)
+    )
+    (pin "1")
+  )
   (symbol (lib_id "power:GND") (at 97.79 143.51 0) (unit 1)
     (in_bom yes) (on_board yes)
-    (property "Reference" "#PWR0134" (id 0) (at 97.79 149.86 0)
+    (property "Reference" "#PWR0127" (id 0) (at 97.79 149.86 0)
       (effects (font (size 1.27 1.27)) hide)
     )
@@
     (pin "1")
   )
+  (symbol (lib_id "power:GND") (at 139.7 83.82 0) (unit 1)
+    (in_bom yes) (on_board yes)
+    (property "Reference" "#PWR0125" (id 0) (at 139.7 90.17 0)
+      (effects (font (size 1.27 1.27)) hide)
+    )
+    (property "Value" "GND" (id 1) (at 139.7 87.63 0))
+    (property "Footprint" "" (id 2) (at 139.7 83.82 0)
+      (effects (font (size 1.27 1.27)) hide)
+    )
+    (property "Datasheet" "" (id 3) (at 139.7 83.82 0)
+      (effects (font (size 1.27 1.27)) hide)
+    )
+    (pin "1")
+  )
+  (symbol (lib_id "power:+3.3V") (at 171.45 72.39 0) (unit 1)
+    (in_bom yes) (on_board yes) (fields_autoplaced)
+    (property "Reference" "#PWR0122" (id 0) (at 171.45 76.2 0)
+      (effects (font (size 1.27 1.27)) hide)
+    )
+    (property "Value" "+3.3V" (id 1) (at 171.45 68.8142 0))
+    (property "Footprint" "" (id 2) (at 171.45 72.39 0)
+      (effects (font (size 1.27 1.27)) hide)
+    )
+    (property "Datasheet" "" (id 3) (at 171.45 72.39 0)
+      (effects (font (size 1.27 1.27)) hide)
+    )
+    (pin "1")
+  )
+  (symbol (lib_id "Memory_EEPROM:AT24CS01-STUM") (at 139.7 76.2 0) (mirror y) (unit 1)
+    (in_bom yes) (on_board yes) (fields_autoplaced)
+    (property "Reference" "U6" (id 0) (at 148.59 74.9299 0)
+      (effects (font (size 1.27 1.27)) (justify right))
+    )
+    (property "Value" "AT24CS01-STUM" (id 1) (at 148.59 77.4699 0)
+      (effects (font (size 1.27 1.27)) (justify right))
+    )
+    (property "Footprint" "Package_TO_SOT_SMD:SOT-23-5" (id 2) (at 139.7 76.2 0)
+      (effects (font (size 1.27 1.27)) hide)
+    )
+    (property "Datasheet" "http://ww1.microchip.com/downloads/en/DeviceDoc/Atmel-8815-SEEPROM-AT24CS01-02-Datasheet.pdf" (id 3) (at 139.7 76.2 0)
+      (effects (font (size 1.27 1.27)) hide)
+    )
+    (pin "1")
+    (pin "2")
+    (pin "3")
+    (pin "4")
+    (pin "5")
+  )
   (symbol (lib_id "Device:R") (at 105.41 132.08 90) (unit 1)
     (in_bom yes) (on_board yes)
-    (property "Reference" "R52" (id 0) (at 101.6 132.08 90)
+    (property "Reference" "R47" (id 0) (at 101.6 132.08 90)
       (effects (font (size 1 1)) (justify left top))
     )
@@
     (pin "1")
     (pin "2")
+  )
+  (symbol (lib_id "power:+3.3V") (at 139.7 68.58 0) (unit 1)
+    (in_bom yes) (on_board yes)
+    (property "Reference" "#PWR0121" (id 0) (at 139.7 72.39 0)
+      (effects (font (size 1.27 1.27)) hide)
+    )
+    (property "Value" "+3.3V" (id 1) (at 139.7 64.77 0))
+    (property "Footprint" "" (id 2) (at 139.7 68.58 0)
+      (effects (font (size 1.27 1.27)) hide)
+    )
+    (property "Datasheet" "" (id 3) (at 139.7 68.58 0)
+      (effects (font (size 1.27 1.27)) hide)
+    )
+    (pin "1")
   )
   (symbol (lib_id "Connector:Micro_SD_Card") (at 139.7 124.46 0) (unit 1)
@@
     (pin "9")
   )
+  (symbol (lib_id "power:GND") (at 127 83.82 0) (unit 1)
+    (in_bom yes) (on_board yes)
+    (property "Reference" "#PWR0124" (id 0) (at 127 90.17 0)
+      (effects (font (size 1.27 1.27)) hide)
+    )
+    (property "Value" "GND" (id 1) (at 127 87.63 0))
+    (property "Footprint" "" (id 2) (at 127 83.82 0)
+      (effects (font (size 1.27 1.27)) hide)
+    )
+    (property "Datasheet" "" (id 3) (at 127 83.82 0)
+      (effects (font (size 1.27 1.27)) hide)
+    )
+    (pin "1")
+  )
 )
