File: onboard.kicad_sch (KiCad schematic)
At the start: 13 parts, among them Q2 BSS83P, Q3 BSS83P, SW3 SW_DIP_x08, SW4 User, U6 157119S12801, U7 157119S12801

Commit message: lots changed
Parts:
- removed Q2, Q3: BSS83P, Package_TO_SOT_SMD:SOT-23, symbol Transistor_FET:BSS83P
- removed R14: 470, Resistor_SMD:R_0603_1608Metric, symbol Device:R
- removed U6, U7: 157119S12801, Display_7Segment:Sx39-1xxxxx, symbol Display_Character:SA39-11EWA
- added Q2, Q3: 2N7002K, Package_TO_SOT_SMD:SOT-23, symbol Transistor_FET:2N7002K
- added R12, R15: R, Resistor_SMD:R_0603_1608Metric, symbol Device:R
- added U6: HDSM-293L, HDSM-293L:HDSM-293L, symbol HDSM-293L:HDSM-293L
- RN1, RN2: value 470 -> 330
- renumbered R15 to R13, R16 to R14
Connections:
- net +3V3: now also R13.1, R14.1
- net Dig: now also Q3.1 (G)
- net GND: now also Q2.2 (S), Q3.2 (S); no longer R13.2, R14.2
- net Seg.8: now also R12.1, R15.1
- net SegR.0: now also U6.6 (d)
- net SegR.1: now also U6.4 (f)
- net SegR.2: now also U6.3 (a)
- net SegR.3: now also U6.2 (DP2)
- net SegR.4: now also U6.1 (g)
- net SegR.5: now also U6.9 (b)
- net SegR.6: now also U6.8 (c)
- net SegR.7: now also U6.7 (e)
- net nDig: now also D4.1 (K), R14.2, Q2.1 (G), Q3.3 (D), U6.10 (CC_D1); no longer D4.2 (A), R14.1
- net ~{nDig}: now also D5.1 (K), R13.2, Q2.3 (D), U6.5 (CC_D2); no longer D5.2 (A), R13.1
- removed net SegR.8: D4.1 (K), D5.1 (K)
- new net: D4.2 (A), R12.2
- new net: D5.2 (A), R15.2
- no-connect marks 0 -> 1
Other:
- moved on the sheet: D4, D5, R13, R14, SW3, SW4

Commit message: things changed
Parts:
- removed U6: HDSM-293L, HDSM-293L:HDSM-293L, symbol HDSM-293L:HDSM-293L
- added LD1: DC56-11CGKWA, LB-402:LB-402, symbol Display_Character:DC56-11CGKWA
- added Q1, Q10, Q11, Q2, Q3, Q4, Q5, Q6, Q7: FJV4101, Package_TO_SOT_SMD:SOT-23, symbol Transistor_BJT:DTA143E
- renumbered D4 to LD2, D5 to LD3, Q2 to Q8, Q3 to Q9, R12 to R15, R13 to R16, R14 to R17, R15 to R18
Connections:
- net +3V3: now also Q1.2 (E), Q10.2 (E), Q11.2 (E), Q2.2 (E), Q3.2 (E), Q4.2 (E), Q5.2 (E), Q6.2 (E), Q7.2 (E)
- net Seg.0: now also Q1.1 (B); no longer RN1.1 (R1.1)
- net Seg.1: now also Q2.1 (B); no longer RN1.2 (R2.1)
- net Seg.2: now also Q3.1 (B); no longer RN1.3 (R3.1)
- net Seg.3: now also Q4.1 (B); no longer RN1.4 (R4.1)
- net Seg.4: now also Q5.1 (B); no longer RN2.1 (R1.1)
- net Seg.5: now also Q6.1 (B); no longer RN2.2 (R2.1)
- net Seg.6: now also Q7.1 (B); no longer RN2.3 (R3.1)
- net Seg.7: now also Q10.1 (B); no longer RN2.4 (R4.1)
- net Seg.8: now also Q11.1 (B)
- net SegR.0: now also LD1.2 (DIG1_D), LD1.6 (DIG2_D)
- net SegR.1: now also LD1.12 (DIG2_F), LD1.18 (DIG1_F)
- net SegR.2: now also LD1.11 (DIG2_A), LD1.16 (DIG1_A)
- net SegR.3: now also LD1.4 (DP1), LD1.9 (DP2)
- net SegR.4: now also LD1.17 (DIG1_G), LD1.7 (DIG2_G)
- net SegR.5: now also LD1.10 (DIG2_B), LD1.15 (DIG1_B)
- net SegR.6: now also LD1.3 (DIG1_C), LD1.8 (DIG2_C)
- net SegR.7: now also LD1.1 (DIG1_E), LD1.5 (DIG2_E)
- net nDig: now also LD1.13 (DIG2_CC)
- net ~{nDig}: now also LD1.14 (DIG1_CC)
- new net: Q4.3 (C), RN1.4 (R4.1)
- new net: Q5.3 (C), RN2.1 (R1.1)
- new net: Q6.3 (C), RN2.2 (R2.1)
- new net: Q2.3 (C), RN1.2 (R2.1)
- new net: Q1.3 (C), RN1.1 (R1.1)
- new net: Q7.3 (C), RN2.3 (R3.1)
- new net: Q3.3 (C), RN1.3 (R3.1)
- new net: Q10.3 (C), RN2.4 (R4.1)
- new net SegR.8: Q11.3 (C)
- no-connect marks 1 -> 0
Other:
- note removed: "max 5mA per segment!"
- moved on the sheet: LD2, LD3, Q8, Q9, R15, R16, R17, R18, RN1A, RN1B, RN1C, RN1D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

Commit message: isolate and other stuff
Parts:
- RN1, RN2: value 330 -> 220
- renumbered R15 to R19, R16 to R20, R17 to R21, R18 to R22
Connections:
- net Seg.8: no longer R19.1, R22.1
- net SegR.0: now also LD1.4 (DP1), LD1.9 (DP2); no longer LD1.2 (DIG1_D), LD1.6 (DIG2_D)
- net SegR.1: now also LD1.3 (DIG1_C), LD1.8 (DIG2_C); no longer LD1.12 (DIG2_F), LD1.18 (DIG1_F)
- net SegR.2: now also LD1.2 (DIG1_D), LD1.6 (DIG2_D); no longer LD1.11 (DIG2_A), LD1.16 (DIG1_A)
- net SegR.3: now also LD1.1 (DIG1_E), LD1.5 (DIG2_E); no longer LD1.4 (DP1), LD1.9 (DP2)
- net SegR.5: now also LD1.12 (DIG2_F), LD1.18 (DIG1_F); no longer LD1.10 (DIG2_B), LD1.15 (DIG1_B)
- net SegR.6: now also LD1.11 (DIG2_A), LD1.16 (DIG1_A); no longer LD1.3 (DIG1_C), LD1.8 (DIG2_C)
- net SegR.7: now also LD1.10 (DIG2_B), LD1.15 (DIG1_B); no longer LD1.1 (DIG1_E), LD1.5 (DIG2_E)
- net SegR.8: now also R19.1, R22.1
Other:
- title: [canbrd] CAN/RS485 IO board -> [canbrd] CAN IO board

Commit message: things changed
Parts:
- added D25, D26, D27, D28: BAS40TW, Package_TO_SOT_SMD:SOT-363_SC-70-6, symbol BAS40TW:BAS40TW
- added LD4: Power, LED_SMD:LED_0805_2012Metric, symbol Device:LED
- added Q17: 2N7002K, Package_TO_SOT_SMD:SOT-23, symbol Transistor_FET:2N7002K
- added R53, R54: 10k, Resistor_SMD:R_0603_1608Metric, symbol Device:R
- added R57: R, Resistor_SMD:R_0603_1608Metric, symbol Device:R
- R51: renamed from R20; value 1k -> 10k
- R56: renamed from R21; value 1k -> 10k
- renumbered Q1 to Q10, Q2 to Q11, Q3 to Q12, Q4 to Q13, Q5 to Q14, Q6 to Q15, Q8 to Q16, Q7 to Q18, Q10 to Q19, Q9 to Q20, Q11 to Q21, R19 to R52, R22 to R55
Connections:
- net GND: now also LD4.1 (K), Q17.2 (S)
- net +3V3 renamed +3.3V
- net +3.3V: now also R53.1, R54.1
- removed net Dig: Q20.1 (G), SW3.1, SW3.2, SW3.3, SW3.4, SW3.5, SW3.6, SW3.7, SW3.8
- removed net nDig: LD1.13 (DIG2_CC), LD2.1 (K), Q16.1 (G), Q20.3 (D), R56.2
- removed net ~{nDig}: LD1.14 (DIG1_CC), LD3.1 (K), Q16.3 (D), R51.2, SW4.1
- new net: LD4.2 (A), R57.2
- new net: D28.1 (A), D28.2 (A), D28.3 (A), Q17.1 (G), R54.2
- new net: D27.1 (A), SW4.1
- new net: D27.2 (A), SW3.8
- new net: D27.3 (A), SW3.7
- new net: D26.1 (A), SW3.6
- new net: D26.2 (A), SW3.5
- new net: D26.3 (A), SW3.4
- new net: D25.3 (A), SW3.1
- new net: D25.2 (A), SW3.2
- new net: D25.1 (A), SW3.3
- new net +5V: R57.1
- new net Dig0: Q20.1 (G)
- new net Dig1: Q16.1 (G)
- new net nDig0: D28.6 (K), LD1.14 (DIG1_CC), LD3.1 (K), Q20.3 (D), R56.2
- new net nDig1: D28.4 (K), LD1.13 (DIG2_CC), LD2.1 (K), Q16.3 (D), R51.2
- new net sw_en: D25.4 (K), D25.5 (K), D25.6 (K), D26.4 (K), D26.5 (K), D26.6 (K), D27.4 (K), D27.5 (K), D27.6 (K), Q17.3 (D), R53.2
- no-connect marks 0 -> 1
Other:
- moved on the sheet: Q16, Q20, R51, R56
