File: canbrd.kicad_pcb (KiCad board)
At the start: 2 copper layers, 100 x 100 mm, 221 parts, among them J1 RP_DEBUG, J10 PwrOut, J11 IO2, J12 I^{2}C, J13 USB_C_Receptacle, J14 IO1, J15 IO0, J2 UPDI, J3 Micro_SD_Card, J4 GND, J5 Field24V, J6 Amphenol RJHSE5380, J7 Amphenol RJHSE5380, J8 CAN, J9 CAN, Q1 2N7002K, Q2 BSS83P, Q3 BSS83P, Q4 Q_PMOS_GDS, Q5 BC856, SW1 BOOTSEL, SW2 RESET, SW3 SW_DIP_x08, SW4 User, U1 W25Q16JVSNIQ, U10 ULN2003A, U11 MAX17634BATP+, U12 AP62250WU, U2 RP2040, U3 TJA1051T-3, U4 MCP2510-x/SO, U5 MAX3485CSA, U6 157119S12801, U7 157119S12801, U8 ATtiny427, U9 ULN2003A, Y1 12MHz, Y2 16MHz

Commit message: lots changed
Parts:
- removed the C22 at (138.4, 123.0)
- removed the C23 at (136.9, 126.1)
- removed the C24 at (138.4, 126.1)
- removed the D20 at (136.2, 133.5)
- removed the D21 at (150.2, 133.5)
- removed the D22 at (121.2, 120.2)
- removed D23: 33V, Diode_SMD:D_SMB
- removed the F8 at (113.8, 107.8)
- removed the J12 at (158.0, 124.0)
- removed the J2 at (129.0, 123.0)
- removed the J8 at (149.0, 56.0)
- removed the J9 at (129.0, 56.0)
- removed the JP10 at (175.2, 140.0)
- removed the JP11 at (161.2, 130.5)
- removed JP12, JP15, JP16, JP19, JP20, JP24, JP25, JP28, JP29, JP32, JP33, JP36, JP37: Vdiv, Jumper:SolderJumper-2_P1.3mm_Open_TrianglePad1.0x1.5mm
- removed JP13, JP14, JP17, JP18, JP22, JP23, JP26, JP27, JP30, JP31, JP34, JP35: LowZ, Jumper:SolderJumper-2_P1.3mm_Open_TrianglePad1.0x1.5mm
- removed JP21: Addr, Jumper:SolderJumper-2_P1.3mm_Open_TrianglePad1.0x1.5mm
- removed the R14 at (116.0, 61.0)
- removed the R6 at (147.5, 122.5)
- removed the R7 at (149.5, 122.5)
- removed RN10, RN12, RN4, RN6: 10k, Resistor_SMD:R_Array_Convex_4x0603
- removed RN11, RN9: 68, Resistor_SMD:R_Array_Convex_4x0603
- removed RN13, RN14, RN7, RN8: 1k, Resistor_SMD:R_Array_Convex_4x0603
- removed RN3, RN5: 330, Resistor_SMD:R_Array_Convex_4x0603
- removed the U10 at (121.2, 112.5)
- removed the U9 at (121.2, 128.0)
- removed kibuzzard-62179F8F: G***, kibuzzard-62179F8F
- removed kibuzzard-62179F9F: G***, kibuzzard-62179F9F
- removed kibuzzard-62179FB2: G***, kibuzzard-62179FB2
- removed kibuzzard-6217A003: G***, kibuzzard-6217A003
- removed kibuzzard-6217A022: G***, kibuzzard-6217A022
- removed kibuzzard-6217A03E: G***, kibuzzard-6217A03E
- removed kibuzzard-6217A08D: G***, kibuzzard-6217A08D
- removed kibuzzard-6217A0B8: G***, kibuzzard-6217A0B8
- removed kibuzzard-6217A0C8: G***, kibuzzard-6217A0C8
- removed kibuzzard-6217A0EA: G***, kibuzzard-6217A0EA
- removed kibuzzard-6234FB7E: G***, kibuzzard-6234FB7E
- added J5: RJ45_LED_Shielded_x2, canbrd_conn:RJ45_Amphenol_RJHSE5380-02, F.Cu at (126.6, 59.1)
- added Q10: 2N7002K, Package_TO_SOT_SMD:SOT-23, F.Cu at (138.2, 129.8)
- added Q11: 2N7002K, Package_TO_SOT_SMD:SOT-23, F.Cu at (152.2, 129.8)
- added Q12: TPCP8110, TPCP8110:PS-8, F.Cu at (185.5, 68.8)
- added Q5: 2N7002K, Package_TO_SOT_SMD:SOT-23, F.Cu at (141.8, 129.8)
- added Q6: 2N7002K, Package_TO_SOT_SMD:SOT-23, F.Cu at (131.2, 129.8)
- added Q7: 2N7002K, Package_TO_SOT_SMD:SOT-23, F.Cu at (145.2, 129.8)
- added Q8: 2N7002K, Package_TO_SOT_SMD:SOT-23, F.Cu at (134.8, 129.8)
- added Q9: 2N7002K, Package_TO_SOT_SMD:SOT-23, F.Cu at (148.8, 129.8)
- added R12: R, Resistor_SMD:R_0603_1608Metric, F.Cu at (117.4, 61.0)
- added R15: R, Resistor_SMD:R_0603_1608Metric, F.Cu at (119.0, 61.0)
- added R16: 10k, Resistor_SMD:R_0603_1608Metric, F.Cu at (127.8, 126.8)
- added R18: 10k, Resistor_SMD:R_0603_1608Metric, F.Cu at (141.8, 126.8)
- added R19: 10k, Resistor_SMD:R_0603_1608Metric, F.Cu at (141.8, 136.8)
- added R20: 100, Resistor_SMD:R_0603_1608Metric, F.Cu at (165.0, 135.0)
- added R21: 10k, Resistor_SMD:R_0603_1608Metric, F.Cu at (131.2, 126.8)
- added R22: 10k, Resistor_SMD:R_0603_1608Metric, F.Cu at (131.2, 136.8)
- added R23: 10k, Resistor_SMD:R_0603_1608Metric, F.Cu at (145.2, 126.8)
- added R24: 10k, Resistor_SMD:R_0603_1608Metric, F.Cu at (145.2, 136.8)
- added R25: 100, Resistor_SMD:R_0603_1608Metric, F.Cu at (168.0, 135.0)
- added R26: 10k, Resistor_SMD:R_0603_1608Metric, F.Cu at (134.8, 126.8)
- added R27: 10k, Resistor_SMD:R_0603_1608Metric, F.Cu at (134.8, 136.8)
- added R28: 10k, Resistor_SMD:R_0603_1608Metric, F.Cu at (148.8, 126.8)
- added R29: 10k, Resistor_SMD:R_0603_1608Metric, F.Cu at (148.8, 136.8)
- added R30: 100, Resistor_SMD:R_0603_1608Metric, F.Cu at (175.5, 135.0)
- added R31: 10k, Resistor_SMD:R_0603_1608Metric, F.Cu at (138.2, 126.8)
- added R32: 10k, Resistor_SMD:R_0603_1608Metric, F.Cu at (138.2, 136.8)
- added R33: 10k, Resistor_SMD:R_0603_1608Metric, F.Cu at (152.2, 126.8)
- added R34: 10k, Resistor_SMD:R_0603_1608Metric, F.Cu at (152.2, 136.8)
- added R35: 100, Resistor_SMD:R_0603_1608Metric, F.Cu at (178.5, 135.0)
- added kibuzzard-624B71BB: G***, kibuzzard-624B71BB, F.Cu at (127.8, 138.5)
- added kibuzzard-624B71D2: G***, kibuzzard-624B71D2, F.Cu at (131.2, 138.5)
- added kibuzzard-624B71E6: G***, kibuzzard-624B71E6, F.Cu at (134.8, 138.5)
- added kibuzzard-624B71F2: G***, kibuzzard-624B71F2, F.Cu at (138.2, 138.5)
- added kibuzzard-624B71FA: G***, kibuzzard-624B71FA, F.Cu at (141.8, 138.5)
- added kibuzzard-624B7201: G***, kibuzzard-624B7201, F.Cu at (145.2, 138.5)
- added kibuzzard-624B720A: G***, kibuzzard-624B720A, F.Cu at (148.8, 138.5)
- added kibuzzard-624B7210: G***, kibuzzard-624B7210, F.Cu at (152.2, 138.5)
- added kibuzzard-624B7220: G***, kibuzzard-624B7220, F.Cu at (164.8, 138.5)
- added kibuzzard-624B7229: G***, kibuzzard-624B7229, F.Cu at (168.2, 138.5)
- added kibuzzard-624B7230: G***, kibuzzard-624B7230, F.Cu at (175.2, 138.5)
- added kibuzzard-624B7237: G***, kibuzzard-624B7237, F.Cu at (178.8, 138.5)
- added kibuzzard-624B7242: G***, kibuzzard-624B7242, F.Cu at (171.8, 138.5)
- added kibuzzard-624B7247: G***, kibuzzard-624B7247, F.Cu at (161.2, 138.5)
- added kibuzzard-624B724B: G***, kibuzzard-624B724B, F.Cu at (182.2, 138.5)
- added kibuzzard-624B7255: G***, kibuzzard-624B7255, F.Cu at (157.8, 138.5)
- added kibuzzard-624B7539: G***, kibuzzard-624B7539, F.Cu at (111.5, 111.2)
- added kibuzzard-624B7544: G***, kibuzzard-624B7544, F.Cu at (111.5, 107.8)
- added kibuzzard-624B7558: G***, kibuzzard-624B7558, F.Cu at (111.5, 114.8)
- added kibuzzard-624B7567: G***, kibuzzard-624B7567, F.Cu at (111.5, 118.2)
- added kibuzzard-624B7585: G***, kibuzzard-624B7585, F.Cu at (111.5, 121.8)
- added kibuzzard-624B75E6: G***, kibuzzard-624B75E6, F.Cu at (111.5, 125.2)
- added kibuzzard-624B75EF: G***, kibuzzard-624B75EF, F.Cu at (111.5, 128.8)
- added kibuzzard-624B75FB: G***, kibuzzard-624B75FB, F.Cu at (111.5, 132.2)
- added kibuzzard-624B766D: G***, kibuzzard-624B766D, F.Cu at (117.2, 146.2)
- added kibuzzard-624B7E7C: G***, kibuzzard-624B7E7C, F.Cu at (145.0, 105.7)
- C21: value 1u -> 100n
- D10, D11, D12, D13, D14, D15, D16, D17, D6, D7, D8, D9: value 3.3V -> BAS40-04; footprint Diode_SMD:D_SOD-123 -> Package_TO_SOT_SMD:SOT-23
- D18, D19: value 3.3V -> 33V; footprint Diode_SMD:D_SOD-123 -> Diode_SMD:D_SMB
- F1, F2, F3, F5, F6, F7: value 1A -> 500mA
- F8: renamed from F9; footprint Littelfuse-154:Littelfuse-154 -> Littelfuse-154:Littelfuse-154-2920
- J11: renamed from J14; value IO1 -> DIO
- J12: renamed from J15; value IO0 -> AIO
- J6, J7: value Amphenol RJHSE5380 -> CAN; footprint Connector_RJ:RJ45_Amphenol_RJHSE5380 -> canbrd_conn:NH0210x0xxxxG
- J9: renamed from J11; value IO2 -> OUT
- JP7, JP8: value Vdiv -> LowZ
- JP9: value LowZ -> Jumper_2_Open; moved to F.Cu
- Q2, Q3: value BSS83P -> 2N7002K
- Q4: value Q_PMOS_GDS -> 2N7002K; footprint Package_TO_SOT_SMD:TO-252-2 -> Package_TO_SOT_SMD:SOT-23
- R17: value 220 -> 10k
- RN1, RN2: value 470 -> 330
- U6: value 157119S12801 -> HDSM-293L; footprint Display_7Segment:Sx39-1xxxxx -> HDSM-293L:HDSM-293L
- U7: value 157119S12801 -> 74HC595; footprint Display_7Segment:Sx39-1xxxxx -> Package_SO:SOIC-16_3.9x9.9mm_P1.27mm
- U8: value ATtiny427 -> ULN2003A; footprint Package_DFN_QFN:QFN-24-1EP_4x4mm_P0.5mm_EP2.6x2.6mm -> Package_SO:SOIC-16_3.9x9.9mm_P1.27mm
- moved Q4 83.6 mm to (127.8, 129.8), turned to -90 degrees
- moved U7 49.6 mm to (130.1, 119.0), turned to 0 degrees
- moved JP9 46.9 mm to (115.0, 132.2)
- moved D14 45.3 mm to (175.0, 131.5), turned to 90 degrees
- moved D9 40.0 mm to (131.2, 133.8)
- moved D19 39.1 mm to (122.5, 108.8), turned to 0 degrees
- moved D17 37.8 mm to (179.0, 131.5)
- moved D6 32.0 mm to (127.8, 133.8)
- moved D7 32.0 mm to (141.8, 133.8)
- moved D12 31.5 mm to (134.8, 133.8)
- moved D13 31.5 mm to (148.8, 133.8)
- moved D16 25.0 mm to (152.2, 133.8)
- moved F1 24.5 mm to (115.0, 107.8)
- moved D10 23.5 mm to (145.2, 133.8)
- moved U8 21.2 mm to (122.5, 116.5), turned to 180 degrees
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- renumbered C25 to C22, C26 to C23, C27 to C24, C28 to C25, C29 to C26, C30 to C27, C31 to C28, C32 to C29, C33 to C30, C34 to C31, C35 to C32, C36 to C33, C37 to C34, C38 to C35, C39 to C36, C40 to C37, D24 to D20, D25 to D21, D26 to D22, J13 to J10, J3 to J2, J4 to J3, J5 to J4, J10 to J8, JP38 to JP10, JP39 to JP11, Q5 to Q13, R12 to R10, R13 to R11, R15 to R13, R16 to R14, R18 to R36, R19 to R37, R20 to R38, R21 to R39, R22 to R40, R23 to R41, R24 to R42, R8 to R6, R9 to R7, R10 to R8, R11 to R9, U12 to U10, U11 to U9
Connections:
- D10 pad 1: /IO/RP2 -> GND
- D10 pad 2: GND -> VIO
- D11 pad 1: /IO/RP6 -> GND
- D11 pad 2: GND -> +3V3
- D12 pad 1: /IO/RP3 -> GND
- D12 pad 2: GND -> VIO
- D13 pad 1: /IO/RP7 -> GND
- D13 pad 2: GND -> VIO
- D14 pad 1: /IO Expander/IO Expander Protection/AT1.0 -> GND
- D14 pad 2: GND -> +3V3
- D15 pad 1: /IO Expander/IO Expander Protection/AT1.4 -> GND
- D15 pad 2: GND -> VIO
- D16 pad 1: /IO Expander/IO Expander Protection/AT1.1 -> GND
- D16 pad 2: GND -> VIO
- D17 pad 1: /IO Expander/IO Expander Protection/AT1.5 -> GND
- D17 pad 2: GND -> +3V3
- D18 pad 1: /IO Expander/IO Expander Protection/AT1.2 -> GND
- D18 pad 2: GND -> VIO
- D19 pad 1: /IO Expander/IO Expander Protection/AT1.6 -> /IO Expander/O_TVS
- D4 pad 1: /DISP+SW/SegR.8 -> /DISP+SW/nDig
- D4 pad 2: /DISP+SW/nDig -> Net-(D4-Pad2)
- D5 pad 1: /DISP+SW/SegR.8 -> /DISP+SW/~{nDig}
- D5 pad 2: /DISP+SW/~{nDig} -> Net-(D5-Pad2)
- D6 pad 1: /IO/RP0 -> GND
- D6 pad 2: GND -> VIO
- D7 pad 1: /IO/RP4 -> GND
- D7 pad 2: GND -> VIO
- D8 pad 1: /IO/RP1 -> GND
- D8 pad 2: GND -> +3V3
- D9 pad 1: /IO/RP5 -> GND
- D9 pad 2: GND -> VIO
- F1 pad 1: /IO Expander/IO Expander Power IO/HC0 -> Net-(F1-Pad1)
- F1 pad 2: /Connectors/IO2.7 -> /Connectors/OUT0
- F2 pad 1: /IO Expander/IO Expander Power IO/HC1 -> Net-(F2-Pad1)
- F2 pad 2: /Connectors/IO2.6 -> /Connectors/OUT1
- F3 pad 1: /IO Expander/IO Expander Power IO/HC2 -> Net-(F3-Pad1)
- F3 pad 2: /Connectors/IO2.5 -> /Connectors/OUT2
- F4 pad 1: /IO Expander/IO Expander Power IO/HC3 -> Net-(F4-Pad1)
- F4 pad 2: /Connectors/IO2.4 -> /Connectors/OUT3
- F5 pad 1: /IO Expander/IO Expander Power IO/HC4 -> Net-(F5-Pad1)
- F5 pad 2: /Connectors/IO2.3 -> /Connectors/OUT4
- F6 pad 1: /IO Expander/IO Expander Power IO/HC5 -> Net-(F6-Pad1)
- F6 pad 2: /Connectors/IO2.2 -> /Connectors/OUT5
- F7 pad 1: /IO Expander/IO Expander Power IO/HC6 -> Net-(F7-Pad1)
- F7 pad 2: /Connectors/IO2.1 -> /Connectors/OUT6
- J11 pad 1: /Connectors/IO1.0 -> /Connectors/IO0
- J11 pad 2: /Connectors/IO1.1 -> /Connectors/IO1
- J11 pad 3: /Connectors/IO1.2 -> /Connectors/IO2
- J11 pad 4: /Connectors/IO1.3 -> /Connectors/IO3
- J11 pad 5: /Connectors/IO1.4 -> /Connectors/IO4
- J11 pad 6: /Connectors/IO1.5 -> /Connectors/IO5
- J11 pad 7: /Connectors/IO1.6 -> /Connectors/IO6
- J11 pad 8: /Connectors/IO1.7 -> /Connectors/IO7
- J12 pad 1: /Connectors/IO0.0 -> VIO
- J12 pad 2: /Connectors/IO0.1 -> GND
- J12 pad 3: /Connectors/IO0.2 -> /Connectors/IO8
- J12 pad 4: /Connectors/IO0.3 -> /Connectors/IO9
- J12 pad 5: /Connectors/IO0.4 -> GND
- J12 pad 6: /Connectors/IO0.5 -> /Connectors/IO10
- J12 pad 7: /Connectors/IO0.6 -> /Connectors/IO11
- J12 pad 8: /Connectors/IO0.7 -> GND
- J6 pad 1: /CAN/CANH -> /CAN/CANL
- J6 pad 2: /CAN/CANL -> /CAN/CANH
- J7 pad 1: /CAN/CANH -> /CAN/CANL
- J7 pad 2: /CAN/CANL -> /CAN/CANH
- J9 pad 1: /Connectors/IO2.0 -> /Connectors/OUT0
- J9 pad 2: /Connectors/IO2.1 -> /Connectors/OUT1
- J9 pad 3: /Connectors/IO2.2 -> /Connectors/OUT2
- J9 pad 4: /Connectors/IO2.3 -> /Connectors/OUT3
- J9 pad 5: /Connectors/IO2.4 -> /Connectors/OUT4
- J9 pad 6: /Connectors/IO2.5 -> /Connectors/OUT5
- J9 pad 7: /Connectors/IO2.6 -> /Connectors/OUT6
- J9 pad 8: /Connectors/IO2.7 -> /Connectors/OUT7
- JP5 pad 1: Net-(JP5-Pad1) -> /IO/RP8
- JP5 pad 2: /Connectors/IO0.0 -> /Connectors/IO8
- JP6 pad 1: Net-(JP6-Pad1) -> /IO/RP9
- JP6 pad 2: /Connectors/IO0.4 -> /Connectors/IO9
- JP7 pad 1: Net-(JP7-Pad1) -> /IO/RP10
- JP7 pad 2: GND -> /Connectors/IO10
- JP8 pad 1: Net-(JP8-Pad1) -> /IO/RP11
- JP8 pad 2: GND -> /Connectors/IO11
- JP9 pad 2: /Connectors/IO0.1 -> /Connectors/OUT7
- Q2 pad 1: /DISP+SW/Dig -> /DISP+SW/nDig
- Q2 pad 2: +3V3 -> GND
- Q2 pad 3: /DISP+SW/nDig -> /DISP+SW/~{nDig}
- Q3 pad 1: /DISP+SW/nDig -> /DISP+SW/Dig
- Q3 pad 2: +3V3 -> GND
- Q3 pad 3: /DISP+SW/~{nDig} -> /DISP+SW/nDig
- Q4 pad 1: /Power/revprot_gate -> +3V3
- Q4 pad 2: /Power/Fused24V -> /IO/RP0
- Q4 pad 3: +24V -> /Connectors/IO0
- R13 pad 1: /DISP+SW/~{nDig} -> +3V3
- R13 pad 2: GND -> /DISP+SW/~{nDig}
- R14 pad 1: /DISP+SW/nDig -> +3V3
- R14 pad 2: GND -> /DISP+SW/nDig
- R17 pad 1: +3V3 -> VIO
- R17 pad 2: +3.3VA2 -> /Connectors/IO0
- U2 pad 28: /IO Expander/AT_~{INT} -> /IO Expander/595_~{CS}
- U2 pad 29: /Connectors/SDA -> /IO/RP0
- U2 pad 30: /Connectors/SCL -> /IO/RP1
- U2 pad 31: /Connectors/EXT.0 -> /IO/RP2
- U2 pad 32: /Connectors/EXT.1 -> /IO/RP3
- U2 pad 34: /IO/RP0 -> /IO/RP4
- U2 pad 35: /IO/RP1 -> /IO/RP5
- U2 pad 36: /IO/RP2 -> /IO/RP6
- U2 pad 37: /IO/RP3 -> /IO/RP7
- U2 pad 38: /IO/RP4 -> /IO/RP8
- U2 pad 39: /IO/RP5 -> /IO/RP9
- U2 pad 40: /IO/RP6 -> /IO/RP10
- U2 pad 41: /IO/RP7 -> /IO/RP11
- U6 pad 1: /DISP+SW/SegR.7 -> /DISP+SW/SegR.4
- U6 pad 10: /DISP+SW/SegR.6 -> /DISP+SW/nDig
- U6 pad 2: /DISP+SW/SegR.5 -> /DISP+SW/SegR.3
- U6 pad 3: /DISP+SW/nDig -> /DISP+SW/SegR.2
- U6 pad 4: /DISP+SW/SegR.3 -> /DISP+SW/SegR.1
- U6 pad 5: /DISP+SW/SegR.1 -> /DISP+SW/~{nDig}
- U6 pad 7: /DISP+SW/SegR.2 -> /DISP+SW/SegR.7
- U6 pad 8: /DISP+SW/nDig -> /DISP+SW/SegR.6
- U6 pad 9: /DISP+SW/SegR.4 -> /DISP+SW/SegR.5
- U7 pad 1: /DISP+SW/SegR.7 -> Net-(U7-Pad1)
- U7 pad 10: /DISP+SW/SegR.6 -> +3V3
- U7 pad 2: /DISP+SW/SegR.5 -> Net-(U7-Pad2)
- U7 pad 3: /DISP+SW/~{nDig} -> Net-(U7-Pad3)
- U7 pad 4: /DISP+SW/SegR.3 -> Net-(U7-Pad4)
- U7 pad 5: /DISP+SW/SegR.1 -> Net-(U7-Pad5)
- U7 pad 6: /DISP+SW/SegR.0 -> Net-(U7-Pad6)
- U7 pad 7: /DISP+SW/SegR.2 -> Net-(JP9-Pad1)
- U7 pad 8: /DISP+SW/~{nDig} -> GND
- U7 pad 9: /DISP+SW/SegR.4 -> unconnected-(U7-Pad9)
- U8 pad 1: /IO Expander/IO Expander Protection/AT1.1 -> Net-(U7-Pad6)
- U8 pad 10: /IO Expander/IO Expander Power IO/AT2.6 -> Net-(F1-Pad1)
- U8 pad 11: /IO Expander/IO Expander Protection/AT1.6 -> Net-(F2-Pad1)
- U8 pad 12: /IO Expander/IO Expander Protection/AT1.7 -> Net-(F3-Pad1)
- U8 pad 13: /IO Expander/AT_ADDR -> Net-(F4-Pad1)
- U8 pad 14: /IO Expander/AT_~{INT} -> Net-(F5-Pad1)
- U8 pad 15: /Connectors/SDA -> Net-(F6-Pad1)
- U8 pad 16: /Connectors/SCL -> Net-(F7-Pad1)
- U8 pad 2: /IO Expander/IO Expander Protection/AT1.2 -> Net-(U7-Pad5)
- U8 pad 3: GND -> Net-(U7-Pad4)
- U8 pad 4: +3V3 -> Net-(U7-Pad3)
- U8 pad 5: /IO Expander/IO Expander Protection/AT1.3 -> Net-(U7-Pad2)
- U8 pad 6: +3.3VA2 -> Net-(U7-Pad1)
- U8 pad 7: /IO Expander/IO Expander Protection/AT1.4 -> Net-(U7-Pad15)
- U8 pad 8: /IO Expander/IO Expander Protection/AT1.5 -> GND
- U8 pad 9: /IO Expander/IO Expander Power IO/AT2.7 -> /IO Expander/O_TVS
Routing:
- net +3V3: track 479.0 -> 553.0 mm, vias 25 -> 32
- net VIO: track 0.00 -> 73.7 mm, vias 0 -> 10
- net /IO Expander/595_~{CS}: track 0.00 -> 39.1 mm
- net /IO Expander/IO Expander Power IO/AT2.0: track 31.7 -> 0.00 mm
- net /Connectors/SCL: track 31.0 -> 0.00 mm
- net /Connectors/SDA: track 30.3 -> 0.00 mm, vias 2 -> 0
- net /IO Expander/IO Expander Power IO/AT2.1: track 29.2 -> 0.00 mm
- net /IO Expander/IO Expander Protection/AT1.1: track 28.6 -> 0.00 mm
- net /IO Expander/IO Expander Power IO/AT2.5: track 28.5 -> 0.00 mm
- net /IO Expander/IO Expander Protection/AT1.2: track 27.8 -> 0.00 mm
- net /IO Expander/IO Expander Power IO/AT2.4: track 27.3 -> 0.00 mm
- net /IO Expander/IO Expander Power IO/AT2.7: track 26.1 -> 0.00 mm, vias 2 -> 0
- net /IO/RP11: track 0.00 -> 25.8 mm, vias 0 -> 1
- net /IO Expander/IO Expander Power IO/AT2.2: track 25.6 -> 0.00 mm
- net /IO Expander/AT_~{INT}: track 25.5 -> 0.00 mm, vias 2 -> 0
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- added copper zone on F.Cu, net /IO Expander/O_TVS
- added copper zone on F.Cu, net VIO
- removed copper zone on F.Cu, net +3.3VA2
- removed copper zone on F.Cu, net /IO Expander/IO Expander Power IO/COM0
- removed copper zone on F.Cu, net /IO Expander/IO Expander Power IO/COM1
- removed copper zone on F.Cu, net /IO Expander/IO Expander Power IO/HC0
- removed copper zone on F.Cu, net /IO Expander/IO Expander Power IO/HC1
- removed copper zone on F.Cu, net /IO Expander/IO Expander Power IO/HC2
- removed copper zone on F.Cu, net /IO Expander/IO Expander Power IO/HC3
- removed copper zone on F.Cu, net /IO Expander/IO Expander Power IO/HC4
- removed copper zone on F.Cu, net /IO Expander/IO Expander Power IO/HC5
- removed copper zone on F.Cu, net /IO Expander/IO Expander Power IO/HC6
- removed copper zone on F.Cu, net /IO Expander/IO Expander Power IO/HC7

Commit message: things changed
Routing:
- net /CAN/~{INT}: track 61.1 -> 57.3 mm
- net GND: vias 439 -> 431

Commit message: Update gerber
Other:
- board text added: "Changelog: rev1.1: Add I2C pullups rev2.0: Simplify"
- board text removed: "Changelog: rev1.1: Add I2C pullups."
Changed lines of the file:
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@@
   (gr_line (start 105 149.992152) (end 195 149.992152) (layer "Edge.Cuts") (width 0.1))
   (gr_line (start 195 49.992152) (end 105 49.992152) (layer "Edge.Cuts") (width 0.1))
-  (gr_text "Changelog:\nrev1.1: Add I2C pullups." (at 14.7 185.1) (layer "Cmts.User")
+  (gr_text "Changelog:\nrev1.1: Add I2C pullups\nrev2.0: Simplify" (at 14.7 185.1) (layer "Cmts.User")
     (effects (font (size 2 2) (thickness 0.3)) (justify left))
   )
@@
   (segment (start 129.27 99.15) (end 129.27 98.58) (width 0.3) (layer "F.Cu") (net 73))
   (segment (start 168.999511 104.700489) (end 169.8 105.500978) (width 0.2) (layer "F.Cu") (net 73))
+  (segment (start 149.5 80.5) (end 149.8 80.5) (width 0.3) (layer "F.Cu") (net 73))
   (segment (start 150.2 80.1) (end 150.2 79) (width 0.3) (layer "F.Cu") (net 73))
   (segment (start 129.6 103) (end 136 103) (width 0.2) (layer "F.Cu") (net 73))
@@
   (segment (start 129.2 99.22) (end 129.2 102.6) (width 0.2) (layer "F.Cu") (net 73))
   (segment (start 164.500489 104.700489) (end 168.999511 104.700489) (width 0.2) (layer "F.Cu") (net 73))
-  (segment (start 149.5 80.5) (end 149.8 80.5) (width 0.3) (layer "F.Cu") (net 73))
   (segment (start 129.27 99.15) (end 129.2 99.22) (width 0.2) (layer "F.Cu") (net 73))
   (via (at 144.105 80.395) (size 0.8) (drill 0.4) (layers "F.Cu" "B.Cu") (net 73))

Commit message: things changed
Parts:
- removed the D3 at (127.4, 77.7)
- removed the JP5 at (165.0, 135.0)
- removed the JP6 at (168.0, 135.0)
- removed the JP7 at (175.5, 135.0)
- removed JP8: LowZ, Jumper:SolderJumper-2_P1.3mm_Open_TrianglePad1.0x1.5mm
- removed the R7 at (133.6, 86.2)
- removed the R9 at (136.8, 83.4)
- removed kibuzzard-62179E98: G***, kibuzzard-62179E98
- removed kibuzzard-62179EAF: G***, kibuzzard-62179EAF
- added C14: 100n, Capacitor_SMD:C_0603_1608Metric, F.Cu at (193.9, 122.0)
- added C17: 100n, Capacitor_SMD:C_0603_1608Metric, F.Cu at (140.0, 119.0)
- added C20: 47p, Capacitor_SMD:C_0603_1608Metric, F.Cu at (83.4, 86.6)
- added C21: 47p, Capacitor_SMD:C_0603_1608Metric, F.Cu at (86.0, 87.4)
- added C22: 47p, Capacitor_SMD:C_0603_1608Metric, F.Cu at (88.6, 86.6)
- added C26: 10u, Capacitor_SMD:C_0805_2012Metric, F.Cu at (5.04, 121.0)
- added C27: 10u, Capacitor_SMD:C_0805_2012Metric, F.Cu at (-0.97, 124.3)
- added C28: 1n, Capacitor_SMD:C_1206_3216Metric_Pad1.33x1.80mm_HandSolder, F.Cu at (-0.19, 121.2)
- added C29: 10n, Capacitor_SMD:C_0603_1608Metric, F.Cu at (164.5, 136.0)
- added C30: 10n, Capacitor_SMD:C_0603_1608Metric, F.Cu at (168.5, 136.0)
- added C31: 10n, Capacitor_SMD:C_0603_1608Metric, F.Cu at (175.0, 136.0)
- added C32: 10n, Capacitor_SMD:C_0603_1608Metric, F.Cu at (179.0, 136.0)
- added D17: 3.3V, Diode_SMD:D_SOD-123, F.Cu at (171.8, 136.0)
- added D2: NUP2105L, Package_TO_SOT_SMD:SOT-23, F.Cu at (86.0, 83.6)
- added FB1: 220, Inductor_SMD:L_1206_3216Metric, F.Cu at (223.0, 72.5)
- added FB2: 220, Inductor_SMD:L_1206_3216Metric, F.Cu at (223.0, 69.0)
- added J7: CANGND, canbrd_conn:NH0210x0xxxxG, F.Cu at (138.0, 51.0)
- added LD1: DC56-11CGKWA, LB-402:LB-402, F.Cu at (56.0, 59.0)
- added PS1: RFM-0505S, RFM-0505S:CONV_RFM-0505S, F.Cu at (-8.54, 111.5)
- added Q10: FJV4101, Package_TO_SOT_SMD:SOT-23, F.Cu at (21.0, 87.4)
- added Q11: FJV4101, Package_TO_SOT_SMD:SOT-23, F.Cu at (11.2, 87.4)
- added Q2: FJV4101, Package_TO_SOT_SMD:SOT-23, F.Cu at (16.1, 87.4)
- added Q3: FJV4101, Package_TO_SOT_SMD:SOT-23, F.Cu at (11.2, 96.3)
- added Q4: FJV4101, Package_TO_SOT_SMD:SOT-23, F.Cu at (11.2, 82.9)
- added Q5: FJV4101, Package_TO_SOT_SMD:SOT-23, F.Cu at (16.1, 82.9)
- added Q6: FJV4101, Package_TO_SOT_SMD:SOT-23, F.Cu at (11.2, 91.8)
- added Q7: FJV4101, Package_TO_SOT_SMD:SOT-23, F.Cu at (16.1, 91.8)
- added R12: DNP, Resistor_SMD:R_0603_1608Metric, F.Cu at (47.9, 107.1)
- added R13: 680, Resistor_SMD:R_0603_1608Metric, F.Cu at (3.26, 124.1)
- added R14: 680, Resistor_SMD:R_0603_1608Metric, F.Cu at (9.27, 120.8)
- added R23: 10, Resistor_SMD:R_0603_1608Metric, F.Cu at (127.8, 141.0)
- added R24: 10, Resistor_SMD:R_0603_1608Metric, F.Cu at (141.8, 141.0)
- added R30: 10, Resistor_SMD:R_0603_1608Metric, F.Cu at (131.2, 141.0)
- added R31: 10, Resistor_SMD:R_0603_1608Metric, F.Cu at (145.2, 141.0)
- added R37: 10, Resistor_SMD:R_0603_1608Metric, F.Cu at (134.8, 141.0)
- added R38: 10, Resistor_SMD:R_0603_1608Metric, F.Cu at (148.8, 141.0)
- added R44: 10, Resistor_SMD:R_0603_1608Metric, F.Cu at (138.2, 141.0)
- added R45: 10, Resistor_SMD:R_0603_1608Metric, F.Cu at (152.2, 141.0)
- added R47: 130, Resistor_SMD:R_0603_1608Metric, F.Cu at (143.9, 85.2)
- added R5: 130, Resistor_SMD:R_0603_1608Metric, F.Cu at (168.0, 102.0)
- added R51: 56k, Resistor_SMD:R_0603_1608Metric, F.Cu at (227.9, 71.0)
- added R52: 10k, Resistor_SMD:R_0603_1608Metric, F.Cu at (227.9, 68.5)
- added R6: 130, Resistor_SMD:R_0603_1608Metric, F.Cu at (168.0, 103.5)
- added U7: 6N137S, Package_DIP:SMDIP-8_W9.53mm, F.Cu at (4.56, 113.6)
- Q1: value 2N7002K -> FJV4101
- R10: value 10k -> 130
- R8: value 1k -> DNP
- U10: renamed from U9; value MAX17634BATP+ -> MAX17633BATP+
- U6: value HDSM-293L -> 6N137S; footprint HDSM-293L:HDSM-293L -> Package_DIP:SMDIP-8_W9.53mm
- moved U6 130.1 mm to (-9.77, 121.2), turned to 0 degrees
- moved Q1 112.6 mm to (21.0, 82.9), turned to 0 degrees
- moved R10 85.2 mm to (54.7, 109.0)
- moved U5 80.3 mm to (62.8, 88.0)
- moved C25 80.2 mm to (60.1, 83.6)
- moved JP1 54.8 mm to (90.1, 90.0), turned to -90 degrees
- moved JP3 54.8 mm to (87.4, 90.0)
- moved C19 53.3 mm to (86.0, 96.6), turned to 180 degrees
- moved U3 51.7 mm to (86.0, 92.0)
- moved JP2 49.1 mm to (81.9, 90.0), turned to 90 degrees
- moved JP4 49.0 mm to (84.6, 90.0)
- moved D20 46.1 mm to (224.0, 80.0)
- moved R8 40.9 mm to (158.4, 113.2), turned to -90 degrees
- moved D3 40.8 mm to (88.6, 77.8)
- moved D1 40.8 mm to (83.4, 77.8)
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- renumbered C14 to C15, C15 to C16, C16 to C23, C17 to C24, C20 to C25, C21 to C33, C22 to C34, C23 to C35, C24 to C36, C25 to C37, C26 to C38, C27 to C39, C28 to C40, C29 to C41, C30 to C42, C31 to C43, C32 to C44, C33 to C45, C34 to C46, C35 to C47, C36 to C48, C37 to C49, D12 to D10, D13 to D11, D14 to D12, D15 to D13, D16 to D14, D17 to D15, D18 to D16, D19 to D18, D20 to D19, D21 to D20, D22 to D21, D2 to D3, D6 to D4, D7 to D5, D8 to D6, D9 to D7, D10 to D8, D11 to D9, J9 to J10, J10 to J11, J11 to J12, J12 to J13, J7 to J8, J8 to J9, JP9 to JP5, JP10 to JP6, JP11 to JP7, D4 to LD2, D5 to LD3, Q4 to Q12, Q5 to Q13, Q6 to Q14, Q7 to Q15, Q8 to Q16, Q9 to Q17, Q10 to Q18, Q11 to Q19, Q12 to Q20, Q13 to Q21, Q2 to Q8, Q3 to Q9, R12 to R15, R13 to R16, R14 to R17, R15 to R18, R16 to R19, R17 to R20, R18 to R21, R19 to R22, R20 to R25, R21 to R26, R22 to R27, R23 to R28, R24 to R29, R25 to R32, R26 to R33, R27 to R34, R28 to R35, R29 to R36, R30 to R39, R31 to R40, R32 to R41, R33 to R42, R34 to R43, R35 to R46, R36 to R48, R37 to R49, R38 to R50, R39 to R53, R40 to R54, R41 to R55, R42 to R56, R5 to R7, R6 to R9, U10 to U11, U7 to U8, U8 to U9
Connections:
- net /CAN/CAN_OSC1 renamed /CAN/OSC1
- net /CAN/CAN_OSC2 renamed /CAN/OSC2
- net /MCU/RP_SWCLK renamed /MCU/SWCLK
- net /MCU/RP_SWDIO renamed /MCU/SWDIO
- net /MCU/USB_XDM renamed /MCU/xUSB_DM
- net /MCU/USB_XDP renamed /MCU/xUSB_DP
- C15 pad 2: /MCU/RP_XIN -> /MCU/XIN
- C16 pad 2: /MCU/RP_XOUT -> /MCU/XOUT
- C19 pad 1: +5V -> +5VISO
- C19 pad 2: GND -> GNDISO
- C34 pad 1: /Power/Fused24V -> Net-(C34-Pad1)
- D10 pad 3: /Connectors/IO2 -> Net-(D10-Pad3)
- D11 pad 3: /Connectors/IO6 -> Net-(D11-Pad3)
- D13 pad 3: /Connectors/IO3 -> Net-(D13-Pad3)
- D14 pad 3: /Connectors/IO7 -> Net-(D14-Pad3)
- D20 pad 2: /Power/Fused24V -> Net-(D20-Pad2)
- D4 pad 3: /Connectors/IO0 -> Net-(D4-Pad3)
- D5 pad 3: /Connectors/IO4 -> Net-(D5-Pad3)
- D7 pad 3: /Connectors/IO1 -> Net-(D7-Pad3)
- D8 pad 3: /Connectors/IO5 -> Net-(D8-Pad3)
- J2 pad 7: /CAN/MISO -> /SD/xMISO
- J5 pad 15: GND -> GNDISO
- J5 pad 16: unconnected-(J5-Pad16) -> /Connectors/Field24V
- J5 pad 17: unconnected-(J5-Pad17) -> GND
- J5 pad 18: GND -> unconnected-(J5-Pad18)
- J5 pad 3: GND -> GNDISO
- J5 pad 4: unconnected-(J5-Pad4) -> /Connectors/Field24V
- J5 pad 5: unconnected-(J5-Pad5) -> GND
- J5 pad 6: GND -> unconnected-(J5-Pad6)
- J5 pad SH: GND -> unconnected-(J5-PadSH)
- JP1 pad 2: +5V -> +5VISO
- JP2 pad 1: +5V -> +5VISO
- JP3 pad 1: GND -> GNDISO
- JP4 pad 2: GND -> GNDISO
- Q1 pad 1: +3V3 -> /DISP+SW/Seg.0
- Q1 pad 2: /CAN/CAN_Tx_LV -> +3V3
- Q1 pad 3: /CAN/CAN_Tx_HV -> Net-(Q1-Pad3)
- Q12 pad 3: /Connectors/IO0 -> Net-(D4-Pad3)
- Q13 pad 3: /Connectors/IO4 -> Net-(D5-Pad3)
- Q14 pad 3: /Connectors/IO1 -> Net-(D7-Pad3)
- Q15 pad 3: /Connectors/IO5 -> Net-(D8-Pad3)
- Q16 pad 3: /Connectors/IO2 -> Net-(D10-Pad3)
- Q17 pad 3: /Connectors/IO6 -> Net-(D11-Pad3)
- Q18 pad 3: /Connectors/IO3 -> Net-(D13-Pad3)
- Q19 pad 3: /Connectors/IO7 -> Net-(D14-Pad3)
- Q20 pad 5: /Power/Fused24V -> Net-(C34-Pad1)
- Q20 pad 6: /Power/Fused24V -> Net-(C34-Pad1)
- Q20 pad 7: /Power/Fused24V -> Net-(C34-Pad1)
- Q20 pad 8: /Power/Fused24V -> Net-(C34-Pad1)
- Q21 pad 2: /Power/Fused24V -> Net-(C34-Pad1)
- R10 pad 1: /CAN/CAN_Rx_LV -> /CAN/MISO
- R10 pad 2: GND -> /CAN/xMISO
- R20 pad 2: /Connectors/IO0 -> Net-(D4-Pad3)
- R22 pad 2: /Connectors/IO4 -> Net-(D5-Pad3)
- R27 pad 2: /Connectors/IO1 -> Net-(D7-Pad3)
- R29 pad 2: /Connectors/IO5 -> Net-(D8-Pad3)
- R34 pad 2: /Connectors/IO2 -> Net-(D10-Pad3)
- R36 pad 2: /Connectors/IO6 -> Net-(D11-Pad3)
- R41 pad 2: /Connectors/IO3 -> Net-(D13-Pad3)
- R43 pad 2: /Connectors/IO7 -> Net-(D14-Pad3)
- R8 pad 1: +5V -> /MCU/XIN
- R8 pad 2: /CAN/CAN_Tx_HV -> /MCU/XOUT
- R9 pad 1: /MCU/RP_XOUT -> /MCU/XOUT
- RN1 pad 1: /DISP+SW/Seg.0 -> Net-(Q1-Pad3)
- RN1 pad 2: /DISP+SW/Seg.1 -> Net-(Q2-Pad3)
- RN1 pad 3: /DISP+SW/Seg.2 -> Net-(Q3-Pad3)
- RN1 pad 4: /DISP+SW/Seg.3 -> Net-(Q4-Pad3)
- RN2 pad 1: /DISP+SW/Seg.4 -> Net-(Q5-Pad3)
- RN2 pad 2: /DISP+SW/Seg.5 -> Net-(Q6-Pad3)
- RN2 pad 3: /DISP+SW/Seg.6 -> Net-(Q7-Pad3)
- RN2 pad 4: /DISP+SW/Seg.7 -> Net-(Q10-Pad3)
- U10 pad 4: +24V -> /Power/MAX_EN
- U10 pad 5: unconnected-(U9-Pad5) -> /Power/MAX_~{RST}
- U11 pad 5: +5V -> /Power/MAX_~{RST}
- U2 pad 20: /MCU/RP_XIN -> /MCU/XIN
- U2 pad 4: /CAN/SCK -> /MCU/xSCK
- U2 pad 5: /CAN/MOSI -> /MCU/xMOSI
- U3 pad 1: /CAN/CAN_Tx_HV -> /CAN/CAN_Tx_ISO
- U3 pad 2: GND -> GNDISO
- U3 pad 3: +5V -> +5VISO
- U3 pad 4: /CAN/CAN_Rx_HV -> /CAN/CAN_Rx_ISO
- U4 pad 1: /CAN/CAN_Tx_LV -> /CAN/CAN_Tx
- U4 pad 15: /CAN/MISO -> /CAN/xMISO
- U4 pad 2: /CAN/CAN_Rx_LV -> /CAN/CAN_Rx
- U6 pad 1: /DISP+SW/SegR.4 -> unconnected-(U6-Pad1)
- U6 pad 2: /DISP+SW/SegR.3 -> Net-(R13-Pad2)
- U6 pad 3: /DISP+SW/SegR.2 -> /CAN/CAN_Tx
- U6 pad 4: /DISP+SW/SegR.1 -> (no net)
- U6 pad 5: /DISP+SW/~{nDig} -> GNDISO
- U6 pad 6: /DISP+SW/SegR.0 -> /CAN/CAN_Tx_ISO
- U6 pad 7: /DISP+SW/SegR.7 -> +5VISO
- U6 pad 8: /DISP+SW/SegR.6 -> +5VISO
- Y1 pad 1: /MCU/RP_XOUT -> /MCU/XOUT
- Y1 pad 3: /MCU/RP_XIN -> /MCU/XIN
Routing:
- net +5V: track 115.0 -> 61.4 mm, vias 9 -> 8
- net GNDISO: track 0.00 -> 44.5 mm, vias 0 -> 5
- net +3V3: track 553.0 -> 586.4 mm, vias 32 -> 35
- net /Connectors/Field24V: track 58.4 -> 25.3 mm
- net /DISP+SW/~{nDig}: track 39.2 -> 11.7 mm
- net Net-(C20-Pad1): track 39.2 -> 13.0 mm
- net /DISP+SW/nDig: track 33.8 -> 10.1 mm
- net GND: track 0.00 -> 23.3 mm, vias 431 -> 398
- net /DISP+SW/SegR.4: track 21.2 -> 0.00 mm, vias 2 -> 0
- net /DISP+SW/Seg.8: track 117.6 -> 99.8 mm
- net /DISP+SW/SegR.0: track 4.83 -> 21.2 mm
- net +5VISO: track 0.00 -> 16.0 mm, vias 0 -> 1
- net /DISP+SW/SegR.6: track 8.67 -> 23.8 mm
- net /DISP+SW/SegR.1: track 12.7 -> 26.9 mm, vias 2 -> 0
- net /MCU/XIN: track 0.00 -> 14.0 mm
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- removed copper zone on F.Cu, net /Connectors/Field24V
- removed copper zone on F.Cu, net /Power/Fused24V
- removed copper zone on F.Cu, net /Power/revprot_gate
Other:
- board size 100 x 100 mm -> 100 x 110 mm
