File: canbrd.kicad_pcb (KiCad board)
At the start: 2 copper layers, 100 x 110 mm, 244 parts, among them J1 RP_DEBUG, J10 OUT, J11 USB_C_Receptacle, J12 DIO, J13 AIO, J2 Micro_SD_Card, J3 GND, J4 Field24V, J5 RJ45_LED_Shielded_x2, J6 CAN, J7 CANGND, J8 CAN, J9 PwrOut, Q1 FJV4101, Q10 FJV4101, Q11 FJV4101, Q12 2N7002K, Q13 2N7002K, Q14 2N7002K, Q15 2N7002K, Q16 2N7002K, Q17 2N7002K, Q18 2N7002K, Q19 2N7002K, Q2 FJV4101, Q20 TPCP8110, Q21 BC856, Q3 FJV4101, Q4 FJV4101, Q5 FJV4101, Q6 FJV4101, Q7 FJV4101, Q8 2N7002K, Q9 2N7002K, SW1 BOOTSEL, SW2 RESET, SW3 SW_DIP_x08, SW4 User, U1 W25Q16JVSNIQ, U10 MAX17633BATP+, U11 AP62250WU, U2 RP2040, U3 TJA1051T-3, U4 MCP2510-x/SO, U5 MAX3485CSA, U6 6N137S, U7 6N137S, U8 74HC595, U9 ULN2003A, Y1 12MHz, Y2 16MHz

Commit message: isolate and other stuff
Parts:
- removed the C25 at (60.1, 83.6)
- removed the H3 at (145.0, 95.0)
- removed the J6 at (129.0, 51.0)
- removed the JP5 at (115.0, 132.2)
- removed the U5 at (62.8, 88.0)
- removed kibuzzard-62179C2A: G***, kibuzzard-62179C2A
- removed kibuzzard-62179E31: G***, kibuzzard-62179E31
- removed kibuzzard-621B6EAC: G***, kibuzzard-621B6EAC
- removed kibuzzard-621B6EB9: G***, kibuzzard-621B6EB9
- removed kibuzzard-621B6EDA: G***, kibuzzard-621B6EDA
- removed kibuzzard-624B7E7C: G***, kibuzzard-624B7E7C
- added D18: D, Diode_SMD:D_SMB, F.Cu at (114.4, 140.3)
- added D19: 60v, Diode_SMD:D_SMB, F.Cu at (114.4, 135.3)
- added F8: 2A, Littelfuse-154:Littelfuse-154-2920, F.Cu at (121.4, 141.0)
- added G***: LOGO, sbt_logo:logo_outline, F.Cu at (172.0, 57.0)
- added J10: VIO2, canbrd_conn:NH0210x0xxxxG, F.Cu at (106.0, 141.0)
- added Q20: AO4266E, Package_SO:SOIC-8_3.9x4.9mm_P1.27mm, F.Cu at (121.4, 131.2)
- added R13: 680, Resistor_SMD:R_0603_1608Metric, F.Cu at (147.5, 68.1)
- added R15: 680, Resistor_SMD:R_0603_1608Metric, F.Cu at (136.0, 82.0)
- added R16: 5.1k, Resistor_SMD:R_0603_1608Metric, F.Cu at (133.6, 82.8)
- added R18: 10k, Resistor_SMD:R_0603_1608Metric, F.Cu at (132.8, 85.2)
- added R51: 10k, Resistor_SMD:R_0603_1608Metric, F.Cu at (121.4, 126.5)
- added TP1: TestPoint, TestPoint:TestPoint_THTPad_D2.0mm_Drill1.0mm, F.Cu at (138.5, 116.5)
- added TP2: TestPoint, TestPoint:TestPoint_THTPad_D2.0mm_Drill1.0mm, F.Cu at (141.5, 114.5)
- added TP3: TestPoint, TestPoint:TestPoint_THTPad_D2.0mm_Drill1.0mm, F.Cu at (141.5, 118.5)
- added kibuzzard-629153AB: G***, kibuzzard-629153AB, F.Cu at (144.9, 105.7)
- added kibuzzard-62915456: G***, kibuzzard-62915456, F.Cu at (175.0, 46.5)
- added kibuzzard-62915475: G***, kibuzzard-62915475, F.Cu at (188.5, 89.5)
- added kibuzzard-62915589: G***, kibuzzard-62915589, F.Cu at (108.4, 136.1)
- added kibuzzard-629155A8: G***, kibuzzard-629155A8, F.Cu at (108.7, 145.9)
- added kibuzzard-629155F9: G***, kibuzzard-629155F9, F.Cu at (118.0, 40.0)
- added kibuzzard-62991FA5: G***, kibuzzard-62991FA5, F.Cu at (135.0, 48.0)
- added kibuzzard-62991FA5: G***, kibuzzard-62991FA5, F.Cu at (147.0, 48.0)
- added kibuzzard-62992008: G***, kibuzzard-62992008, F.Cu at (141.0, 50.5)
- added kibuzzard-629930A8: G***, kibuzzard-629930A8, F.Cu at (145.0, 109.8)
- added kibuzzard-629930D0: G***, kibuzzard-629930D0, F.Cu at (118.0, 37.0)
- added kibuzzard-629930D0: G***, kibuzzard-629930D0, F.Cu at (118.0, 42.5)
- C15, C16, C23, C24: value ??? -> 10p
- C33: renamed from C34; footprint Capacitor_SMD:C_0805_2012Metric -> Capacitor_SMD:C_1206_3216Metric
- C37: renamed from C38; footprint Capacitor_SMD:C_0805_2012Metric -> Capacitor_SMD:C_1206_3216Metric
- D17: footprint Diode_SMD:D_SOD-123 -> Diode_SMD:D_MiniMELF
- FB1, FB2: value 220 -> 100
- J7: value CANGND -> CAN; footprint canbrd_conn:NH0210x0xxxxG -> canbrd_conn:NH0310x0xxxxG
- J8: footprint canbrd_conn:NH0210x0xxxxG -> canbrd_conn:NH0310x0xxxxG
- R10, R5, R6: value 130 -> 100
- R14: renamed from R13; value 680 -> 330
- R52: renamed from R47; value 130 -> 100
- RN1, RN2: value 330 -> 220
- moved PS1 174.1 mm to (160.0, 68.0), turned to 180 degrees
- moved C26 169.7 mm to (157.5, 63.6)
- moved C25 167.7 mm to (162.6, 63.6)
- moved U5 163.4 mm to (147.0, 75.0), turned to 90 degrees
- moved C27 161.9 mm to (155.0, 75.0), turned to 90 degrees
- moved R14 151.0 mm to (148.3, 82.0), turned to 180 degrees
- moved R17 140.8 mm to (139.9, 68.1)
- moved U6 137.0 mm to (136.0, 75.0), turned to -90 degrees
- moved Q11 114.7 mm to (118.0, 45.6), turned to -90 degrees
- moved Q6 101.8 mm to (113.0, 92.5), turned to 90 degrees
- moved Q7 99.4 mm to (115.5, 88.5), turned to 90 degrees
- moved Q4 98.2 mm to (109.0, 92.5), turned to 90 degrees
- moved Q3 96.6 mm to (107.5, 88.5), turned to 90 degrees
- moved Q10 96.1 mm to (117.0, 92.5), turned to 90 degrees
- moved Q5 95.6 mm to (111.5, 88.5), turned to 90 degrees
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- renumbered C26 to C25, C27 to C26, C28 to C27, C29 to C28, C30 to C29, C31 to C30, C32 to C31, C33 to C32, C35 to C34, C36 to C35, C37 to C36, C39 to C38, C40 to C39, C41 to C40, C42 to C41, C43 to C42, C44 to C43, C45 to C44, C46 to C45, C47 to C46, C48 to C47, C49 to C48, D18 to D20, D19 to D21, D20 to D22, D21 to D23, F8 to F9, H4 to H3, H5 to H4, J9 to J6, J10 to J9, JP6 to JP5, JP7 to JP6, Q20 to Q21, Q21 to Q22, R14 to R17, R15 to R19, R16 to R20, R17 to R21, R18 to R22, R19 to R23, R20 to R24, R21 to R25, R22 to R26, R23 to R27, R24 to R28, R25 to R29, R26 to R30, R27 to R31, R28 to R32, R29 to R33, R30 to R34, R31 to R35, R32 to R36, R33 to R37, R34 to R38, R35 to R39, R36 to R40, R37 to R41, R38 to R42, R39 to R43, R40 to R44, R41 to R45, R42 to R46, R43 to R47, R44 to R48, R45 to R49, R46 to R50, R48 to R53, R49 to R54, R50 to R55, R51 to R56, R52 to R57, R53 to R58, R54 to R59, R55 to R60, R56 to R61, U11 to U10, U6 to U5, U7 to U6, U8 to U7, U9 to U8, U10 to U9
Connections:
- D20 pad 1: /IO Expander/O_TVS -> GND
- D20 pad 2: GND -> VIO2
- J7 pad 1: GNDISO -> /CAN/CANL
- J8 pad 2: /CAN/CANH -> GNDISO
- LD1 pad 1: /DISP+SW/SegR.7 -> /DISP+SW/SegR.3
- LD1 pad 10: /DISP+SW/SegR.5 -> /DISP+SW/SegR.7
- LD1 pad 11: /DISP+SW/SegR.2 -> /DISP+SW/SegR.6
- LD1 pad 12: /DISP+SW/SegR.1 -> /DISP+SW/SegR.5
- LD1 pad 15: /DISP+SW/SegR.5 -> /DISP+SW/SegR.7
- LD1 pad 16: /DISP+SW/SegR.2 -> /DISP+SW/SegR.6
- LD1 pad 18: /DISP+SW/SegR.1 -> /DISP+SW/SegR.5
- LD1 pad 2: /DISP+SW/SegR.0 -> /DISP+SW/SegR.2
- LD1 pad 3: /DISP+SW/SegR.6 -> /DISP+SW/SegR.1
- LD1 pad 4: /DISP+SW/SegR.3 -> /DISP+SW/SegR.0
- LD1 pad 5: /DISP+SW/SegR.7 -> /DISP+SW/SegR.3
- LD1 pad 6: /DISP+SW/SegR.0 -> /DISP+SW/SegR.2
- LD1 pad 8: /DISP+SW/SegR.6 -> /DISP+SW/SegR.1
- LD1 pad 9: /DISP+SW/SegR.3 -> /DISP+SW/SegR.0
- R14 pad 1: +5V -> +3V3
- R19 pad 1: /DISP+SW/Seg.8 -> /DISP+SW/SegR.8
- R22 pad 1: /DISP+SW/Seg.8 -> /DISP+SW/SegR.8
- U4 pad 17: unconnected-(U4-Pad17) -> +3V3
- U6 pad 6: /CAN/CAN_Rx -> Net-(R15-Pad2)
- U8 pad 9: /IO Expander/O_TVS -> VIO2
Routing:
- net GND: track 23.3 -> 85.7 mm, vias 398 -> 321
- net +3V3: track 586.4 -> 634.2 mm, vias 35 -> 41
- net /DISP+SW/nDig: track 10.1 -> 57.1 mm
- net +5V: track 61.4 -> 106.3 mm, vias 8 -> 10
- net VIO2: track 0.00 -> 43.3 mm, vias 0 -> 4
- net /DISP+SW/~{nDig}: track 11.7 -> 53.7 mm
- net /Connectors/Field24V: track 25.3 -> 64.5 mm
- net /CAN/MOSI: track 108.8 -> 72.2 mm
- net /DISP+SW/SegR.4: track 0.00 -> 35.5 mm, vias 0 -> 1
- net +5VISO: track 16.0 -> 51.2 mm, vias 1 -> 2
- net /CAN/~{CS}: track 80.4 -> 47.9 mm
- net /CAN/SCK: track 108.3 -> 75.9 mm
- net /Power/MAX_~{RST}: track 2.59 -> 34.1 mm, vias 0 -> 2
- net GNDISO: track 44.5 -> 73.5 mm, vias 5 -> 8
- net /DISP+SW/Seg.8: track 99.8 -> 127.3 mm
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- added copper zone on F.Cu, net /IO Expander/xOUT7
- added copper zone on B.Cu, net GNDISO
- added copper zone on F.Cu, net GNDISO
- added copper zone on F.Cu, net VIO2
- removed copper zone on F.Cu, net /IO Expander/O_TVS
Other:
- board size 100 x 110 mm -> 100 x 120 mm
- board text added: "Changelog: rev1.1: Add I2C pullups rev2.0: Simplify rev2.1: Isolate CAN, CAN filter, PSU ferrit, UVLO rev2.2: Remove RS485"
- board text added: "MZ 2022"
- board text removed: "Changelog: rev1.1: Add I2C pullups rev2.0: Simplify"
