File: canbrd.kicad_sch (KiCad schematic)
At the start: 5 parts

Commit message: lots changed
Other:
- sheet Connectors ports: added IO[0..11], OUT[0..7]; removed EXT.[0..1], IO0.[0..7], IO1.[0..7], IO2.[0..7], {I^{2}C}
- sheet IO ports: added IO[0..11], RP[0..11]; removed IO0.[0..7], RP[0..7]
- sheet IO Expander ports: added 595_~{CS}, OUT[0..7], {SPI}; removed AT_~{INT}, IO1.[0..7], IO2.[0..7], {I^{2}C}
- sheet MCU ports: added IO_~{CS}, RP[0..11]; removed EXT.[0..1], IO_~{INT}, RP[0..7], {I^{2}C}
- note added: "Changelog: rev1.1: Add I^{2}C pullups rev2.0: Simplify"
- note removed: "Changelog: rev1.1: Add I^{2}C pullups"

Commit message: things changed
Other:
- note added: "Changelog: rev1.1: Add I^{2}C pullups rev2.0: Simplify rev2.1: Isolate CAN, CAN filter, PSU ferrit, UVLO"
- note removed: "Changelog: rev1.1: Add I^{2}C pullups rev2.0: Simplify"

Commit message: isolate and other stuff
Parts:
- removed H3: M3, MountingHole:MountingHole_3.2mm_M3_Pad_Via, symbol Mechanical:MountingHole_Pad
- renumbered H4 to H3, H5 to H4
Other:
- note added: "Changelog: rev1.1: Add I^{2}C pullups rev2.0: Simplify rev2.1: Isolate CAN, CAN filter, PSU ferrit, UVLO rev2.2: Remove RS485"
- note removed: "Changelog: rev1.1: Add I^{2}C pullups rev2.0: Simplify rev2.1: Isolate CAN, CAN filter, PSU ferrit, UVLO"
- title: [canbrd] CAN/RS485 IO board -> [canbrd] CAN IO board

Commit message: things changed
Parts:
- removed H1, H3, H4: M3, MountingHole:MountingHole_3.2mm_M3_Pad_Via, symbol Mechanical:MountingHole_Pad
- added FID1, FID2, FID3: Fiducial, Fiducial:Fiducial_0.5mm_Mask1.5mm, symbol Mechanical:Fiducial
- added H1, H3, H4, H5, H6: M3, canbrd_hole:MountingHole_3.2mm_M3, symbol Mechanical:MountingHole
Other:
- sheet SD renamed SD+EEPROM
- added sheet ADC+Temp (adc.kicad_sch)
- sheet CAN ports: added none; removed ~{RX1}
- sheet Connectors ports: added AIN[0..7], IO[0..7]; removed IO[0..11]
- sheet DISP+SW ports: added Dig[0..1]; removed Dig
- sheet IO ports: added IO[0..7], RP[0..7]; removed IO[0..11], RP[0..11]
- sheet MCU ports: added Dig[0..1], I_meas, RP[0..7], U_meas, {I^{2}C}; removed CAN_~{RX1}, Dig, RP[0..11]
- sheet Power ports: added I_meas, U_meas; removed none
- sheet SD+EEPROM ports: added {I^{2}C}; removed none
- note added: "Changelog: rev1.1: Add I^{2}C pullups rev2.0: Simplify rev2.1: Isolate CAN, CAN filter, PSU ferrit, UVLO rev2.2: Remove RS485 rev2.3: Change PMOS, change screw holes, flip out7 TVS, update USB-C footprint rev2.4: Add power LED (5V), add IDC IO connector, add input voltage+current meas, change fuses, fix out7 fuse placement, add more mounting holes rev3.0: Add ADC, change IDC pinout and size, add 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"
- note removed: "Changelog: rev1.1: Add I^{2}C pullups rev2.0: Simplify rev2.1: Isolate CAN, CAN filter, PSU ferrit, UVLO rev2.2: Remove RS485"
