File: isolation.kicad_sch (KiCad schematic)
At the start: 8 parts, among them U6 6N137S, U7 6N137S

Commit message: isolate and other stuff
Parts:
- added R13, R15: 680, Resistor_SMD:R_0603_1608Metric, symbol Device:R_Small
- added R16: 5.1k, Resistor_SMD:R_0603_1608Metric, symbol Device:R
- added R18: 10k, Resistor_SMD:R_0603_1608Metric, symbol Device:R_Small
- R14: renamed from R13; value 680 -> 330
- renumbered C26 to C25, C27 to C26, C28 to C27, R14 to R17, U6 to U5, U7 to U6
Connections:
- net 5V: now also R15.1; no longer R14.1
- net 5VISO: now also R13.1
- net GND: now also R18.2
- net RX: now also R16.1, R18.1; no longer U6.6 (VO)
- net TX_ISO: now also R13.2
- new net: R15.2, R16.2, U6.6 (VO)
- new net 3.3V: R14.1
Other:
- title: [canbrd] CAN/RS485 IO board -> [canbrd] CAN IO board

Commit message: things changed
Parts:
- removed R13, R15: 680, Resistor_SMD:R_0603_1608Metric, symbol Device:R_Small
- removed R14: 330, Resistor_SMD:R_0603_1608Metric, symbol Device:R
- removed R16: 5.1k, Resistor_SMD:R_0603_1608Metric, symbol Device:R
- removed R17: 680, Resistor_SMD:R_0603_1608Metric, symbol Device:R
- removed R18: 10k, Resistor_SMD:R_0603_1608Metric, symbol Device:R_Small
- removed U5, U6: 6N137S, Package_DIP:SMDIP-8_W9.53mm, symbol Isolator:6N137
- added C41, C42: 100n, Capacitor_SMD:C_0603_1608Metric, symbol Device:C
- added U9: ISO6721Q1, Package_SO:SOIC-8_7.5x5.85mm_P1.27mm, symbol ISO6721Q1:ISO6721Q1
- PS1: MANUFACTURER (none) -> Recom; MAXIMUM_PACKAGE_HEIGHT (none) -> 10mm; PARTREV (none) -> 0; STANDARD (none) -> Manufacturer Recommendations
- renumbered C25 to C38, C26 to C39, C27 to C40
Connections:
- net 3.3V: now also C41.1, U9.1 (VCC1)
- net 5VISO: now also C42.1, U9.8 (VCC2)
- net GND: now also C41.2, U9.4 (GND1)
- net GNDISO: now also C42.2, U9.5 (GND2)
- net RX: now also U9.2 (OUTA)
- net RX_ISO: now also U9.7 (INA)
- net TX: now also U9.3 (INB)
- net TX_ISO: now also U9.6 (OUTB)
