File: adc.kicad_sch (KiCad schematic)
At the start: 34 parts, among them U5 MAX11603

Commit message: Minimal design for testing
Parts:
- removed C19, C20, C23: 100n, Capacitor_SMD:C_0603_1608Metric, symbol Device:C
- removed C21, C22, C24, C25, C26, C27, C28, C29: 10n, Capacitor_SMD:C_0603_1608Metric, symbol Device:C
- removed D13, D14, D15, D16, D17, D18, D20, D21: BAS40-04, Package_TO_SOT_SMD:SOT-23, symbol Device:D_Schottky_Dual_Series_AKC_Split
- removed D19: 3.3V, Diode_SMD:D_MiniMELF, symbol Device:D_Zener
- removed JP1: Temp7, Jumper:SolderJumper-2_P1.3mm_Open_TrianglePad1.0x1.5mm, symbol Jumper:Jumper_2_Open
- removed JP2: Temp8, Jumper:SolderJumper-2_P1.3mm_Bridged_Pad1.0x1.5mm, symbol Jumper:Jumper_2_Bridged
- removed R37: 10, Resistor_SMD:R_0603_1608Metric, symbol Device:R
- removed R38, R39, R40, R41, R42, R43, R44, R45: 100, Resistor_SMD:R_0603_1608Metric, symbol Device:R
- removed R46: 10k, Resistor_SMD:R_0603_1608Metric, symbol Device:R
- removed TH1: NTC 10k, Resistor_SMD:R_0805_2012Metric, symbol Device:Thermistor_NTC
- removed U5: MAX11603, Package_SO:QSOP-16_3.9x4.9mm_P0.635mm, symbol max11604:MAX11604
Other:
- note removed: "I didn't want to make a proper symbol, so I reused this. AIN0-7 ARE NUMBERED IN OPPOSITE ORDER!"
